File: Models/MainBoard/MainBoard.kicad_pcb (KiCad board)
At the start: 2 copper layers, 0 parts

Commit message: Added PA95 footprint draft
Parts:
- added IC**: PA95, PA95:PA95, F.Cu at (130.0, 83.9)
- added REF**: TSSOP-16, IC:TSSOP-16, F.Cu at (151.6, 95.3)
- added REF**: PA95, IC:PA95, F.Cu at (144.0, 73.0)
- added REF**: TO-220, ThreeTerminal:TO-220, F.Cu at (134.9, 95.6)
