File: Models/MainBoard/CPU.kicad_sch (KiCad schematic)
At the start: 0 parts

Commit message: Save progress
Other:
- sheet DAC renamed DAC1
- added sheet DAC2 (DAC.kicad_sch)
- note added: "Print the 2nd DAC, but don't buy the number of spare QFNs needed for this This is a de-risking step to avoid the design cost of revising the PCB (and possibly save money by using spare boards)"
Changed lines of the file:
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@@
 	(generator_version "9.0")
 	(paper "A4")
-	(sheet
-		(at 127 76.2)
+	(text "Print the 2nd DAC, but don't buy the\nnumber of spare QFNs needed for this\n\nThis is a de-risking step to avoid the\ndesign cost of revising the PCB (and\npossibly save money by using spare boards)"
+		(exclude_from_sim no)
+		(at 72.39 69.85 0)
+		(effects
+			(font
+				(size 1.27 1.27)
+			)
+			(justify left top)
+		)
+	)
+	(sheet
+		(at 127 101.6)
 		(size 25.4 25.4)
 		(exclude_from_sim no)
@@
 		)
 		(property "Sheetname" "ADC"
-			(at 127 75.4884 0)
+			(at 127 100.8884 0)
 			(effects
 				(font
@@
 		)
 		(property "Sheetfile" "ADC.kicad_sch"
-			(at 127 102.1846 0)
+			(at 127 127.5846 0)
 			(effects
 				(font
@@
 	)
 	(sheet
-		(at 127 114.3)
+		(at 127 139.7)
 		(size 25.4 25.4)
 		(exclude_from_sim no)
@@
 		)
 		(property "Sheetname" "CDC"
-			(at 127 113.5884 0)
+			(at 127 138.9884 0)
 			(effects
 				(font
@@
 		)
 		(property "Sheetfile" "CDC.kicad_sch"
-			(at 127 140.2846 0)
+			(at 127 165.6846 0)
 			(effects
 				(font
@@
 	)
 	(sheet
-		(at 127 38.1)
-		(size 25.4 25.4)
-		(exclude_from_sim no)
-		(in_bom yes)
-		(on_board yes)
-		(dnp no)
-		(fields_autoplaced yes)
-		(stroke
-			(width 0.1524)
-			(type solid)
-		)
-		(fill
-			(color 0 0 0 0.0000)
-		)
-		(property "Sheetname" "DAC"
-			(at 127 37.3884 0)
+		(at 127 25.4)
+		(size 25.4 25.4)
+		(exclude_from_sim no)
+		(in_bom yes)
+		(on_board yes)
+		(dnp no)
+		(fields_autoplaced yes)
+		(stroke
+			(width 0.1524)
+			(type solid)
+		)
+		(fill
+			(color 0 0 0 0.0000)
+		)
+		(property "Sheetname" "DAC1"
+			(at 127 24.6884 0)
 			(effects
 				(font
@@
 		)
 		(property "Sheetfile" "DAC.kicad_sch"
-			(at 127 64.0846 0)
+			(at 127 51.3846 0)
 			(effects
 				(font
@@
 				)
 			)
+		)
+	)
+	(sheet
+		(at 127 63.5)
+		(size 25.4 25.4)
+		(exclude_from_sim no)
+		(in_bom yes)
+		(on_board yes)
+		(dnp no)
+		(fields_autoplaced yes)
+		(stroke
+			(width 0.1524)
+			(type solid)
+		)
+		(fill
+			(color 0 0 0 0.0000)
+		)
+		(property "Sheetname" "DAC2"
+			(at 127 62.7884 0)
+			(effects
+				(font
+					(size 1.27 1.27)
+				)
+				(justify left bottom)
+			)
+		)
+		(property "Sheetfile" "DAC.kicad_sch"
+			(at 127 89.4846 0)
+			(effects
+				(font
+					(size 1.27 1.27)
+				)
+				(justify left top)
+			)
+		)
+		(instances
+			(project "MainBoard"
+				(path "/600cc1cc-74ca-4bfc-97a0-b230eb3afbcd/dcbaa67c-e094-4d47-92d5-6abf5c7cf167"
+					(page "12")
+				)
+			)
