File: Models/MainBoard/MainBoard.kicad_sch (KiCad schematic)
At the start: 0 parts

Commit message: Added PA95 footprint draft
Parts:
- added IC1: PA95, PA95, symbol PA95:PA95
Changed lines of the file:
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@@
 	(generator_version "9.0")
 	(paper "A4")
+	(symbol
+		(lib_id "PA95:PA95")
+		(at 127 76.2 0)
+		(unit 1)
+		(exclude_from_sim no)
+		(in_bom yes)
+		(on_board yes)
+		(dnp no)
+		(fields_autoplaced yes)
+		(property "Reference" "IC1"
+			(at 146.05 83.8199 0)
+			(effects
+				(font
+					(size 1.27 1.27)
+				)
+				(justify left)
+			)
+		)
+		(property "Value" "PA95"
+			(at 146.05 86.3599 0)
+			(effects
+				(font
+					(size 1.27 1.27)
+				)
+				(justify left)
+			)
+		)
+		(property "Footprint" "PA95"
+			(at 146.05 171.12 0)
+			(effects
+				(font
+					(size 1.27 1.27)
+				)
+				(justify left top)
+				(hide yes)
+			)
+		)
+		(property "Datasheet" "https://www.apexanalog.com/resources/products/pa95u.pdf"
+			(at 146.05 271.12 0)
+			(effects
+				(font
+					(size 1.27 1.27)
+				)
+				(justify left top)
+				(hide yes)
+			)
+		)
+		(property "Description" "900V, 1.6mA Power Amplifier with Low Standby Current, High voltage  900V (+/-450V), Low quiescent current  1.6mA, High output current  100mA continuous, 200mA PEAK."
+			(at 127 76.2 0)
+			(effects
+				(font
+					(size 1.27 1.27)
+				)
+				(hide yes)
+			)
+		)
+		(property "Height" "22.73"
+			(at 146.05 471.12 0)
+			(effects
+				(font
+					(size 1.27 1.27)
+				)
+				(justify left top)
+				(hide yes)
+			)
+		)
+		(property "Manufacturer_Name" "Apex Microtechnology"
+			(at 146.05 571.12 0)
+			(effects
+				(font
+					(size 1.27 1.27)
+				)
+				(justify left top)
+				(hide yes)
+			)
+		)
+		(property "Manufacturer_Part_Number" "PA95"
+			(at 146.05 671.12 0)
+			(effects
+				(font
+					(size 1.27 1.27)
+				)
+				(justify left top)
+				(hide yes)
+			)
+		)
+		(property "Mouser Part Number" "137-PA95"
+			(at 146.05 771.12 0)
+			(effects
+				(font
+					(size 1.27 1.27)
+				)
+				(justify left top)
+				(hide yes)
+			)
+		)
+		(property "Mouser Price/Stock" "https://www.mouser.co.uk/ProductDetail/Apex-Microtechnology/PA95?qs=TiOZkKH1s2T5rE6vjqqrxw%3D%3D"
+			(at 146.05 871.12 0)
+			(effects
+				(font
+					(size 1.27 1.27)
+				)
+				(justify left top)
+				(hide yes)
+			)
+		)
+		(property "Arrow Part Number" ""
+			(at 146.05 971.12 0)
+			(effects
+				(font
+					(size 1.27 1.27)
+				)
+				(justify left top)
+				(hide yes)
+			)
+		)
+		(property "Arrow Price/Stock" ""
+			(at 146.05 1071.12 0)
+			(effects
+				(font
+					(size 1.27 1.27)
+				)
+				(justify left top)
+				(hide yes)
+			)
+		)
+		(pin "4"
+		)
+		(pin "2"
+		)
+		(pin "1"
+		)
+		(pin "6"
+		)
+		(pin "7"
+		)
+		(pin "8"
+		)
+		(pin "10"
+		)
+		(pin "12"
+		)
+		(instances
+			(project ""
+				(path "/600cc1cc-74ca-4bfc-97a0-b230eb3afbcd"
+					(reference "IC1")
+					(unit 1)
+				)
+			)
+		)
+	)
 	(sheet_instances
 		(path "/"

Commit message: Save progress
Parts:
- added U1: DAC81404RHBR, RHB0032E-IPC_A, symbol DAC81404:DAC81404RHBR
Changed lines of the file:
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@@
+		)
+	)
+	(symbol
+		(lib_id "DAC81404:DAC81404RHBR")
+		(at 185.42 54.61 0)
+		(unit 1)
+		(exclude_from_sim no)
+		(in_bom yes)
+		(on_board yes)
+		(dnp no)
+		(fields_autoplaced yes)
+		(property "Reference" "U1"
+			(at 210.82 45.72 0)
+			(effects
+				(font
+					(size 1.524 1.524)
+				)
+			)
+		)
+		(property "Value" "DAC81404RHBR"
+			(at 210.82 48.26 0)
+			(effects
+				(font
+					(size 1.524 1.524)
+				)
+			)
+		)
+		(property "Footprint" "RHB0032E-IPC_A"
+			(at 185.42 54.61 0)
+			(effects
+				(font
+					(size 1.27 1.27)
+					(italic yes)
+				)
+				(hide yes)
+			)
+		)
+		(property "Datasheet" "https://www.ti.com/lit/gpn/dac81404"
+			(at 185.42 54.61 0)
+			(effects
+				(font
+					(size 1.27 1.27)
+					(italic yes)
+				)
+				(hide yes)
+			)
+		)
+		(property "Description" ""
+			(at 185.42 54.61 0)
+			(effects
+				(font
+					(size 1.27 1.27)
+				)
+				(hide yes)
+			)
+		)
+		(pin "28"
+		)
+		(pin "30"
+		)
+		(pin "25"
+		)
+		(pin "15"
+		)
+		(pin "10"
+		)
+		(pin "11"
+		)
+		(pin "9"
+		)
+		(pin "12"
+		)
+		(pin "13"
+		)
+		(pin "16"
+		)
+		(pin "31"
+		)
+		(pin "32"
+		)
+		(pin "26"
+		)
+		(pin "1"
+		)
+		(pin "3"
+		)
+		(pin "4"
+		)
+		(pin "2"
+		)
+		(pin "8"
+		)
+		(pin "6"
+		)
+		(pin "5"
+		)
+		(pin "7"
+		)
+		(pin "17"
+		)
+		(pin "19"
+		)
+		(pin "20"
+		)
+		(pin "18"
+		)
+		(pin "24"
+		)
+		(pin "22"
+		)
+		(pin "21"
+		)
+		(pin "23"
+		)
+		(pin "29"
+		)
+		(pin "14"
+		)
+		(pin "27"
+		)
+		(pin "33"
+		)
+		(instances
+			(project ""
+				(path "/600cc1cc-74ca-4bfc-97a0-b230eb3afbcd"
+					(reference "U1")
+					(unit 1)
+				)
+			)
 		)
 	)

Commit message: Save progress
Parts:
- added U2: ISO1641DWR, SOIC16-DW_TEX, symbol ISO1641DW:ISO1641DWR
- added U3: ISO7761DW, DW0016B_N, symbol ISO7761DW:ISO7761DW
Changed lines of the file:
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@@
 	(paper "A4")
 	(symbol
+		(lib_id "ISO1641DW:ISO1641DWR")
+		(at 97.79 135.89 0)
+		(unit 1)
+		(exclude_from_sim no)
+		(in_bom yes)
+		(on_board yes)
+		(dnp no)
+		(fields_autoplaced yes)
+		(property "Reference" "U2"
+			(at 118.11 125.73 0)
+			(effects
+				(font
+					(size 1.524 1.524)
+				)
+			)
+		)
+		(property "Value" "ISO1641DWR"
+			(at 118.11 128.27 0)
+			(effects
+				(font
+					(size 1.524 1.524)
+				)
+			)
+		)
+		(property "Footprint" "SOIC16-DW_TEX"
+			(at 97.79 135.89 0)
+			(effects
+				(font
+					(size 1.27 1.27)
+					(italic yes)
+				)
+				(hide yes)
+			)
+		)
+		(property "Datasheet" "https://www.ti.com/lit/gpn/iso1641"
+			(at 97.79 135.89 0)
+			(effects
+				(font
+					(size 1.27 1.27)
+					(italic yes)
+				)
+				(hide yes)
+			)
+		)
+		(property "Description" ""
+			(at 97.79 135.89 0)
+			(effects
+				(font
+					(size 1.27 1.27)
+				)
+				(hide yes)
+			)
+		)
+		(pin "1"
+		)
+		(pin "2"
+		)
+		(pin "3"
+		)
+		(pin "4"
+		)
+		(pin "5"
+		)
+		(pin "6"
+		)
+		(pin "7"
+		)
+		(pin "8"
+		)
+		(pin "16"
+		)
+		(pin "15"
+		)
+		(pin "14"
+		)
+		(pin "13"
+		)
+		(pin "12"
+		)
+		(pin "11"
+		)
+		(pin "10"
+		)
+		(pin "9"
+		)
+		(instances
+			(project ""
+				(path "/600cc1cc-74ca-4bfc-97a0-b230eb3afbcd"
+					(reference "U2")
+					(unit 1)
+				)
+			)
+		)
+	)
+	(symbol
 		(lib_id "PA95:PA95")
-		(at 127 76.2 0)
+		(at 123.19 77.47 0)
 		(unit 1)
 		(exclude_from_sim no)
@@
 		(fields_autoplaced yes)
 		(property "Reference" "IC1"
-			(at 146.05 83.8199 0)
+			(at 142.24 85.0899 0)
 			(effects
 				(font
@@
 		)
 		(property "Value" "PA95"
-			(at 146.05 86.3599 0)
+			(at 142.24 87.6299 0)
 			(effects
 				(font
@@
 		)
 		(property "Footprint" "PA95"
-			(at 146.05 171.12 0)
+			(at 142.24 172.39 0)
 			(effects
 				(font
@@
 		)
 		(property "Datasheet" "https://www.apexanalog.com/resources/products/pa95u.pdf"
-			(at 146.05 271.12 0)
+			(at 142.24 272.39 0)
 			(effects
 				(font
@@
 		)
 		(property "Description" "900V, 1.6mA Power Amplifier with Low Standby Current, High voltage  900V (+/-450V), Low quiescent current  1.6mA, High output current  100mA continuous, 200mA PEAK."
-			(at 127 76.2 0)
+			(at 123.19 77.47 0)
 			(effects
 				(font
@@
 		)
 		(property "Height" "22.73"
-			(at 146.05 471.12 0)
+			(at 142.24 472.39 0)
 			(effects
 				(font
@@
 		)
 		(property "Manufacturer_Name" "Apex Microtechnology"
-			(at 146.05 571.12 0)
+			(at 142.24 572.39 0)
 			(effects
 				(font
@@
 		)
 		(property "Manufacturer_Part_Number" "PA95"
-			(at 146.05 671.12 0)
+			(at 142.24 672.39 0)
 			(effects
 				(font
@@
 		)
 		(property "Mouser Part Number" "137-PA95"
-			(at 146.05 771.12 0)
+			(at 142.24 772.39 0)
 			(effects
 				(font
@@
 		)
 		(property "Mouser Price/Stock" "https://www.mouser.co.uk/ProductDetail/Apex-Microtechnology/PA95?qs=TiOZkKH1s2T5rE6vjqqrxw%3D%3D"
-			(at 146.05 871.12 0)
+			(at 142.24 872.39 0)
 			(effects
 				(font
@@
 		)
 		(property "Arrow Part Number" ""
-			(at 146.05 971.12 0)
+			(at 142.24 972.39 0)
 			(effects
 				(font
@@
 		)
 		(property "Arrow Price/Stock" ""
-			(at 146.05 1071.12 0)
+			(at 142.24 1072.39 0)
 			(effects
 				(font
@@
 		(pin "1"
 		)
+		(pin "10"
+		)
+		(pin "12"
+		)
+		(pin "8"
+		)
 		(pin "6"
 		)
 		(pin "7"
-		)
-		(pin "8"
-		)
-		(pin "10"
-		)
-		(pin "12"
 		)
 		(instances
@@
 					(unit 1)
 				)
+			)
+		)
+	)
+	(symbol
+		(lib_id "ISO7761DW:ISO7761DW")
+		(at 69.85 99.06 0)
+		(unit 1)
+		(exclude_from_sim no)
+		(in_bom yes)
+		(on_board yes)
+		(dnp no)
+		(fields_autoplaced yes)
+		(property "Reference" "U3"
+			(at 69.85 71.12 0)
+			(effects
+				(font
+					(size 1.524 1.524)
+				)
+			)
+		)
+		(property "Value" "ISO7761DW"
+			(at 69.85 73.66 0)
+			(effects
+				(font
+					(size 1.524 1.524)
+				)
+			)
+		)
+		(property "Footprint" "DW0016B_N"
+			(at 69.85 99.06 0)
+			(effects
+				(font
+					(size 1.27 1.27)
+					(italic yes)
+				)
+				(hide yes)
+			)
+		)
+		(property "Datasheet" "https://www.ti.com/lit/gpn/iso7761"
+			(at 69.85 99.06 0)
+			(effects
+				(font
+					(size 1.27 1.27)
+					(italic yes)
+				)
+				(hide yes)
+			)
+		)
+		(property "Description" ""
+			(at 69.85 99.06 0)
+			(effects
+				(font
+					(size 1.27 1.27)
+				)
+				(hide yes)
+			)
+		)
+		(pin "11"
+		)
+		(pin "8"
+		)
+		(pin "14"
+		)
+		(pin "16"
+		)
+		(pin "6"
+		)
+		(pin "3"
+		)
+		(pin "12"
+		)
+		(pin "15"
+		)
+		(pin "7"
+		)
+		(pin "13"
+		)
+		(pin "9"
+		)
+		(pin "10"
+		)
+		(pin "4"
+		)
+		(pin "5"
+		)
+		(pin "1"
+		)
+		(pin "2"
+		)
+		(instances
+			(project ""
+				(path "/600cc1cc-74ca-4bfc-97a0-b230eb3afbcd"
+					(reference "U3")
+					(unit 1)
+				)

Commit message: Save progress
Parts:
- removed IC1: PA95, PA95, symbol PA95:PA95
- removed U1: DAC81404RHBR, RHB0032E-IPC_A, symbol DAC81404:DAC81404RHBR
- removed U2: ISO1641DWR, SOIC16-DW_TEX, symbol ISO1641DW:ISO1641DWR
- removed U3: ISO7761DW, DW0016B_N, symbol ISO7761DW:ISO7761DW
Other:
- added sheet CPU (CPU.kicad_sch)
- added sheet Power (Power.kicad_sch)

Commit message: Save progress
Other:
- removed sheet CPU
- removed sheet Power
- added sheet ADC (ADC.kicad_sch)
- added sheet CDC (CDC.kicad_sch)
- added sheet DAC1 (DAC.kicad_sch)
- added sheet DAC2 (DAC.kicad_sch)
- added sheet Isolation (Isolation.kicad_sch)
- added sheet Teensy (Teensy.kicad_sch)
- note added: "Print the 2nd DAC, but don't buy the number of spare QFNs needed for this This is a de-risking step to avoid the design cost of revising the PCB (and possibly save money by using spare boards)"
Changed lines of the file:
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@@
 	(generator_version "9.0")
 	(paper "A4")
-	(sheet
-		(at 152.4 50.8)
-		(size 50.8 50.8)
-		(exclude_from_sim no)
-		(in_bom yes)
-		(on_board yes)
-		(dnp no)
-		(fields_autoplaced yes)
-		(stroke
-			(width 0.1524)
-			(type solid)
-		)
-		(fill
-			(color 0 0 0 0.0000)
-		)
-		(property "Sheetname" "Power"
-			(at 152.4 50.0884 0)
-			(effects
-				(font
-					(size 1.27 1.27)
-				)
-				(justify left bottom)
-			)
-		)
-		(property "Sheetfile" "Power.kicad_sch"
-			(at 152.4 102.1846 0)
+	(text "Print the 2nd DAC, but don't buy the\nnumber of spare QFNs needed for this\n\nThis is a de-risking step to avoid the\ndesign cost of revising the PCB (and\npossibly save money by using spare boards)"
+		(exclude_from_sim no)
+		(at 72.39 69.85 0)
+		(effects
+			(font
+				(size 1.27 1.27)
+			)
+			(justify left top)
+		)
+	)
+	(sheet
+		(at 228.6 63.5)
+		(size 25.4 50.8)
+		(exclude_from_sim no)
+		(in_bom yes)
+		(on_board yes)
+		(dnp no)
+		(fields_autoplaced yes)
+		(stroke
+			(width 0.1524)
+			(type solid)
+		)
+		(fill
+			(color 0 0 0 0.0000)
+		)
+		(property "Sheetname" "Teensy"
+			(at 228.6 62.7884 0)
+			(effects
+				(font
+					(size 1.27 1.27)
+				)
+				(justify left bottom)
+			)
+		)
+		(property "Sheetfile" "Teensy.kicad_sch"
+			(at 228.6 114.8846 0)
+			(effects
+				(font
+					(size 1.27 1.27)
+				)
+				(justify left top)
+			)
+		)
+		(instances
+			(project "MainBoard"
+				(path "/600cc1cc-74ca-4bfc-97a0-b230eb3afbcd"
+					(page "14")
+				)
+			)
+		)
+	)
+	(sheet
+		(at 127 139.7)
+		(size 25.4 25.4)
+		(exclude_from_sim no)
+		(in_bom yes)
+		(on_board yes)
+		(dnp no)
+		(fields_autoplaced yes)
+		(stroke
+			(width 0.1524)
+			(type solid)
+		)
+		(fill
+			(color 0 0 0 0.0000)
+		)
+		(property "Sheetname" "CDC"
+			(at 127 138.9884 0)
+			(effects
+				(font
+					(size 1.27 1.27)
+				)
+				(justify left bottom)
+			)
+		)
+		(property "Sheetfile" "CDC.kicad_sch"
+			(at 127 165.6846 0)
+			(effects
+				(font
+					(size 1.27 1.27)
+				)
+				(justify left top)
+			)
+		)
+		(instances
+			(project "MainBoard"
+				(path "/600cc1cc-74ca-4bfc-97a0-b230eb3afbcd"
+					(page "3")
+				)
+			)
+		)
+	)
+	(sheet
+		(at 177.8 50.8)
+		(size 25.4 76.2)
+		(exclude_from_sim no)
+		(in_bom yes)
+		(on_board yes)
+		(dnp no)
+		(fields_autoplaced yes)
+		(stroke
+			(width 0.1524)
+			(type solid)
+		)
+		(fill
+			(color 0 0 0 0.0000)
+		)
+		(property "Sheetname" "Isolation"
+			(at 177.8 50.0884 0)
+			(effects
+				(font
+					(size 1.27 1.27)
+				)
+				(justify left bottom)
+			)
+		)
+		(property "Sheetfile" "Isolation.kicad_sch"
+			(at 177.8 127.5846 0)
+			(effects
+				(font
+					(size 1.27 1.27)
+				)
+				(justify left top)
+			)
+		)
+		(instances
+			(project "MainBoard"
+				(path "/600cc1cc-74ca-4bfc-97a0-b230eb3afbcd"
+					(page "13")
+				)
+			)
+		)
+	)
+	(sheet
+		(at 127 101.6)
+		(size 25.4 25.4)
+		(exclude_from_sim no)
+		(in_bom yes)
+		(on_board yes)
+		(dnp no)
+		(fields_autoplaced yes)
+		(stroke
+			(width 0.1524)
+			(type solid)
+		)
+		(fill
+			(color 0 0 0 0.0000)
+		)
+		(property "Sheetname" "ADC"
+			(at 127 100.8884 0)
+			(effects
+				(font
+					(size 1.27 1.27)
+				)
+				(justify left bottom)
+			)
+		)
+		(property "Sheetfile" "ADC.kicad_sch"
+			(at 127 127.5846 0)
 			(effects
 				(font
@@
 	)
 	(sheet
-		(at 76.2 50.8)
-		(size 50.8 50.8)
-		(exclude_from_sim no)
-		(in_bom yes)
-		(on_board yes)
-		(dnp no)
-		(fields_autoplaced yes)
-		(stroke
-			(width 0.1524)
-			(type solid)
-		)
-		(fill
-			(color 0 0 0 0.0000)
-		)
-		(property "Sheetname" "CPU"
-			(at 76.2 50.0884 0)
-			(effects
-				(font
-					(size 1.27 1.27)
-				)
-				(justify left bottom)
-			)
-		)
-		(property "Sheetfile" "CPU.kicad_sch"
-			(at 76.2 102.1846 0)
-			(effects
-				(font
-					(size 1.27 1.27)
-				)
-				(justify left top)
-			)
-		)
-		(instances
-			(project "MainBoard"
-				(path "/600cc1cc-74ca-4bfc-97a0-b230eb3afbcd"
-					(page "6")
-				)
-			)
+		(at 127 63.5)
+		(size 25.4 25.4)
+		(exclude_from_sim no)
+		(in_bom yes)
+		(on_board yes)
+		(dnp no)
+		(fields_autoplaced yes)
+		(stroke
+			(width 0.1524)
+			(type solid)
+		)
+		(fill
+			(color 0 0 0 0.0000)
+		)
+		(property "Sheetname" "DAC2"
+			(at 127 62.7884 0)
+			(effects
+				(font
+					(size 1.27 1.27)
+				)
+				(justify left bottom)
+			)
+		)
+		(property "Sheetfile" "DAC.kicad_sch"
+			(at 127 89.4846 0)
+			(effects
+				(font
+					(size 1.27 1.27)
+				)
+				(justify left top)
+			)
+		)
+		(instances
+			(project "MainBoard"
+				(path "/600cc1cc-74ca-4bfc-97a0-b230eb3afbcd"
+					(page "5")
+				)
+			)
+		)
+	)
+	(sheet
+		(at 127 25.4)
+		(size 25.4 25.4)
+		(exclude_from_sim no)
+		(in_bom yes)
+		(on_board yes)
+		(dnp no)
+		(fields_autoplaced yes)
+		(stroke
+			(width 0.1524)
+			(type solid)
+		)
+		(fill
+			(color 0 0 0 0.0000)
+		)
+		(property "Sheetname" "DAC1"
+			(at 127 24.6884 0)
+			(effects
+				(font
+					(size 1.27 1.27)
+				)
+				(justify left bottom)
+			)
+		)
+		(property "Sheetfile" "DAC.kicad_sch"
+			(at 127 51.3846 0)
+			(effects
+				(font
+					(size 1.27 1.27)
+				)
+				(justify left top)
+			)
+		)
+		(instances
+			(project "MainBoard"
+				(path "/600cc1cc-74ca-4bfc-97a0-b230eb3afbcd"
+					(page "4")
+				)
+			)

Commit message: Save progress
Other:
- note added: "DAC1: - FineX - FineY - FineZ - CoarseZ all channels ±12 V (mode 1110)"
- note added: "DAC2: - Vbias - Vcomp - general purpose channel 1 - general purpose channel 2 all channels ±12 V (mode 1110)"
- note added: "Input: - 100 MΩ or 330 MΩ - switched by PCB swapping - design for 330 MΩ - debug with 100 MΩ ±12.288 V (mode 0000)"
- note added: "Input: - 3 pF total capacitance - 300 μm separation, debug with 1 mm - 13 aF/nm conversion time 109.6 ms (mode 111) max excitation voltage (mode 11) 10x resolution boost in software: - 100 samples at 9 Hz - 0.09 Hz measurement rate"
- note removed: "Print the 2nd DAC, but don't buy the number of spare QFNs needed for this This is a de-risking step to avoid the design cost of revising the PCB (and possibly save money by using spare boards)"
Changed lines of the file:
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@@
 	(generator_version "9.0")
 	(paper "A4")
-	(text "Print the 2nd DAC, but don't buy the\nnumber of spare QFNs needed for this\n\nThis is a de-risking step to avoid the\ndesign cost of revising the PCB (and\npossibly save money by using spare boards)"
+	(text "DAC2:\n- Vbias\n- Vcomp\n- general purpose channel 1\n- general purpose channel 2\n\nall channels ±12 V (mode 1110)"
 		(exclude_from_sim no)
-		(at 72.39 69.85 0)
+		(at 86.106 64.77 0)
 		(effects
 			(font
+				(size 1.27 1.27)
+			)
+			(justify left top)
+		)
+	)
+	(text "DAC1:\n- FineX\n- FineY\n- FineZ\n- CoarseZ\n\nall channels ±12 V (mode 1110)\n"
+		(exclude_from_sim no)
+		(at 86.106 26.162 0)
+		(effects
+			(font
+				(size 1.27 1.27)
+			)
+			(justify left top)
+		)
+	)
+	(text "Input:\n- 100 MΩ or 330 MΩ\n- switched by PCB swapping\n- design for 330 MΩ\n- debug with 100 MΩ\n\n±12.288 V (mode 0000)"
+		(exclude_from_sim no)
+		(at 86.106 105.156 0)
+		(effects
+			(font
+				(size 1.27 1.27)
+			)
+			(justify left top)
+		)
+	)
+	(text "Input:\n- 3 pF total capacitance\n- 300 μm separation, debug with 1 mm\n- 13 aF/nm\n\nconversion time 109.6 ms (mode 111)\nmax excitation voltage (mode 11)\n\n10x resolution boost in software:\n - 100 samples at 9 Hz\n - 0.09 Hz measurement rate"
+		(exclude_from_sim no)
+		(at 84.582 142.494 0)
+		(effects
+			(font

Commit message: Save progress
Other:
- note added: "DAC2: - Vbias - unassigned channel - unassigned channel - unassigned channel all channels ±12 V (mode 1110)"
- note removed: "DAC2: - Vbias - Vcomp - general purpose channel 1 - general purpose channel 2 all channels ±12 V (mode 1110)"
Changed lines of the file:
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@@
 	(generator_version "9.0")
 	(paper "A4")
-	(text "DAC2:\n- Vbias\n- Vcomp\n- general purpose channel 1\n- general purpose channel 2\n\nall channels ±12 V (mode 1110)"
+	(text "DAC2:\n- Vbias\n- unassigned channel\n- unassigned channel\n- unassigned channel\n\nall channels ±12 V (mode 1110)"
 		(exclude_from_sim no)
 		(at 86.106 64.77 0)

Commit message: Save progress
Other:
- note added: "DAC1: - fine X - fine Y - fine Z - coarse Z all channels ±12 V (mode 1110)"
- note added: "DAC2: - piezo voltage (Phase 0.2) - bias voltage (Phase II) ±12 V (mode 1110)"
- note removed: "DAC1: - FineX - FineY - FineZ - CoarseZ all channels ±12 V (mode 1110)"
- note removed: "DAC2: - Vbias - unassigned channel - unassigned channel - unassigned channel all channels ±12 V (mode 1110)"
Changed lines of the file:
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@@
 	(generator_version "9.0")
 	(paper "A4")
-	(text "DAC2:\n- Vbias\n- unassigned channel\n- unassigned channel\n- unassigned channel\n\nall channels ±12 V (mode 1110)"
+	(text "DAC2:\n- piezo voltage (Phase 0.2)\n- bias voltage (Phase II)\n\n±12 V (mode 1110)"
 		(exclude_from_sim no)
-		(at 86.106 64.77 0)
+		(at 86.868 64.77 0)
 		(effects
 			(font
@@
 		)
 	)
-	(text "DAC1:\n- FineX\n- FineY\n- FineZ\n- CoarseZ\n\nall channels ±12 V (mode 1110)\n"
+	(text "DAC1:\n- fine X\n- fine Y\n- fine Z\n- coarse Z\n\nall channels ±12 V (mode 1110)\n"
 		(exclude_from_sim no)
 		(at 86.106 26.162 0)
