File: Models/MainBoard/DAC2.kicad_sch (KiCad schematic)
At the start: 2 parts, among them U4 DAC81404

Commit message: Save progress
Parts:
- removed C6: 220 nF, 0603, symbol Device:C
- removed U4: DAC81404, symbol Vendor:DAC81404
- added C5: 220 nF, 0603, symbol Device:C
- added U5: DAC81401, symbol Vendor:DAC81401
Connections:
- net GND: now also C5.2, U5.11 (VSENSEN), U5.2 (VREFGND)
- new net: C5.1, U5.1 (VREFIO)
- new net: U5.10 (VSENSEP), U5.9 (VOUT)
- no-connect marks 4 -> 1
Other:
- note added: "Bias voltage and Phase 0.2 piezo voltage can be less precise than Phase II piezo voltage. No need to correct for IR drops or different ground potentials."
- note removed: "For the piezo driver channels, the load (28k resistor) sits on a different board. Connect OUT, SENSEP, and SENSEN electrically closer to the target load resistor. Thus, SENSEN will use the ground potential at the target destination instead of the main board."
- note removed: "bypass caps (for both DACs): AVDD: 100 nF, 10 uF AVSS: 100 nF, 10 uF DVDD: 100 nF, 10 uF IOVDD: 100 nF"

Commit message: Finished the DACs
Parts:
- added C14, C16, C18, C20: 100 nF, 0603, symbol Device:C
- added C15, C17, C19: 10 uF, 0805, symbol Device:C
- added NT10, NT11, NT12, NT9: NetTie_2, symbol Device:NetTie_2
- added R5: 10k, 1%, symbol Device:R_US
Connections:
- net GND: now also U5.19 (DVSS), C14.1, C15.1, C16.1, C17.1, C18.1, C19.1, C20.1
- net Output: now reaches U5.10 (VSENSEP), U5.9 (VOUT)
- net at U5.12 (FAULT_N): now also R5.1
- net MISO: now reaches U5.13 (SDO)
- net SCK: now reaches U5.14 (SCLK)
- net MOSI: now reaches U5.15 (SDIN)
- net CS: now reaches U5.16 (SYNC_N)
- net IOVDD: now reaches U5.17 (IOVDD)
- net IOVDD: now also C20.2, NT12.1, R5.2
- net DVDD: now reaches U5.20 (DVDD)
- net DVDD: now also C18.2, C19.2, NT11.1
- net AVSS: now reaches U5.3 (AVSS)
- net AVSS: now also C16.2, C17.2, NT10.1
- net AVDD: now reaches U5.5 (AVDD)
- net AVDD: now also C14.2, C15.2, NT9.1
- new net -15V: NT10.2
- new net 15V: NT9.2
- new net 3.3V: NT12.2
- new net 5V: NT11.2
- no-connect marks 1 -> 5
Other:
- note added: "Bias voltage and Phase 0.2 piezo voltage can be less precise than Phase II piezo voltage. No need to correct for IR drops or different ground potentials. Still, minimize the loop area of the electric field between positive and negative conductors of the output voltage difference. And/or interpret this as being aware of current return paths."
- note removed: "Bias voltage and Phase 0.2 piezo voltage can be less precise than Phase II piezo voltage. No need to correct for IR drops or different ground potentials."

Commit message: Finished the sensors
Changed lines of the file:
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@@
 	(wire
 		(pts
-			(xy 175.26 68.58) (xy 181.61 68.58)
+			(xy 175.26 68.58) (xy 177.8 68.58)
 		)
 		(stroke
@@
 	)
 	(label "IOVDD"
-		(at 181.61 68.58 0)
-		(effects
-			(font
+		(at 177.8 68.58 0)
+		(effects
+			(font

Commit message: Save progress
Parts:
- added R10: 4.7k, 1%, symbol Device:R_US
Connections:
- net Output: now also R10.2; no longer U5.10 (VSENSEP), U5.9 (VOUT)
- new net: R10.1, U5.10 (VSENSEP), U5.9 (VOUT)
Other:
- moved on the sheet: C5, R5, U5

Commit message: Save progress
Parts:
- removed NT10, NT11, NT12, NT9: NetTie_2, symbol Device:NetTie_2
Connections:
- net AVDD is gone; now on net 15V: C14.2, C15.2, U5.5 (AVDD)
- net AVSS is gone; now on net -15V: C16.2, C17.2, U5.3 (AVSS)
- net DVDD is gone; now on net 5V: C18.2, C19.2, U5.20 (DVDD)
- net IOVDD is gone; now on net 3.3V: C20.2, R5.2, U5.17 (IOVDD)

Commit message: Save progress
Connections:
- net GND: no longer U5.11 (VSENSEN)
- net Output: now also U5.10 (VSENSEP)
- net at R10.1, U5.9 (VOUT): no longer U5.10 (VSENSEP)
- new net SENSEN: U5.11 (VSENSEN)
Other:
- note removed: "Bias voltage and Phase 0.2 piezo voltage can be less precise than Phase II piezo voltage. No need to correct for IR drops or different ground potentials. Still, minimize the loop area of the electric field between positive and negative conductors of the output voltage difference. And/or interpret this as being aware of current return paths."
- moved on the sheet: R5
Changed lines of the file:
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@@
 	(generator_version "9.0")
 	(paper "A4")
-	(text "Bias voltage and Phase 0.2 piezo\nvoltage can be less precise than\nPhase II piezo voltage. No need\nto correct for IR drops or\ndifferent ground potentials.\n\nStill, minimize the loop area of\nthe electric field between positive\nand negative conductors of the\noutput voltage difference. And/or\ninterpret this as being aware of\ncurrent return paths."
-		(exclude_from_sim no)
-		(at 152.908 16.764 0)
-		(effects
-			(font
-				(size 1.27 1.27)
-			)
-			(justify left top)
-		)
-	)
 	(junction
 		(at 226.06 127)
@@
 	)
 	(junction
-		(at 152.4 66.04)
+		(at 208.28 101.6)
 		(diameter 0)
 		(color 0 0 0 0)
 	)
 	(junction
-		(at 208.28 101.6)
+		(at 167.64 66.04)
 		(diameter 0)
 		(color 0 0 0 0)
@@
 	(wire
 		(pts
-			(xy 149.86 73.66) (xy 156.21 73.66)
-		)
-		(stroke
-			(width 0)
-			(type default)
-		)
-	)
-	(wire
-		(pts
-			(xy 149.86 78.74) (xy 167.64 78.74)
+			(xy 149.86 73.66) (xy 170.18 73.66)
+		)
+		(stroke
+			(width 0)
+			(type default)
+		)
+	)
+	(wire
+		(pts
+			(xy 167.64 66.04) (xy 170.18 66.04)
+		)
+		(stroke
+			(width 0)
+			(type default)
+		)
+	)
+	(wire
+		(pts
+			(xy 157.48 86.36) (xy 167.64 86.36)
 		)
 		(stroke
@@
 	(wire
 		(pts
-			(xy 175.26 78.74) (xy 177.8 78.74)
+			(xy 175.26 86.36) (xy 177.8 86.36)
 		)
 		(stroke
@@
 	(wire
 		(pts
-			(xy 152.4 66.04) (xy 152.4 71.12)
-		)
-		(stroke
-			(width 0)
-			(type default)
-		)
-	)
-	(wire
-		(pts
 			(xy 226.06 127) (xy 226.06 139.7)
 		)
@@
 	(wire
 		(pts
-			(xy 165.1 66.04) (xy 170.18 66.04)
+			(xy 165.1 66.04) (xy 167.64 66.04)
 		)
 		(stroke
@@
 	(wire
 		(pts
-			(xy 149.86 71.12) (xy 152.4 71.12)
+			(xy 149.86 71.12) (xy 167.64 71.12)
 		)
 		(stroke
@@
 	(wire
 		(pts
-			(xy 149.86 66.04) (xy 152.4 66.04)
+			(xy 149.86 66.04) (xy 157.48 66.04)
 		)
 		(stroke
@@
 	(wire
 		(pts
-			(xy 152.4 66.04) (xy 157.48 66.04)
-		)
-		(stroke
-			(width 0)
-			(type default)
-		)
-	)
-	(wire
-		(pts
 			(xy 220.98 88.9) (xy 226.06 88.9)
 		)
@@
 	(wire
 		(pts
+			(xy 157.48 78.74) (xy 149.86 78.74)
+		)
+		(stroke
+			(width 0)
+			(type default)
+		)
+	)
+	(wire
+		(pts
+			(xy 167.64 66.04) (xy 167.64 71.12)
+		)
+		(stroke
+			(width 0)
+			(type default)
+		)
+	)
+	(wire
+		(pts
 			(xy 203.2 101.6) (xy 208.28 101.6)
 		)
@@
 		(pts
 			(xy 208.28 101.6) (xy 208.28 114.3)
+		)
+		(stroke
+			(width 0)
+			(type default)
+		)
+	)
+	(wire
+		(pts
+			(xy 157.48 86.36) (xy 157.48 78.74)
 		)
 		(stroke
@@
 	)
 	(label "IOVDD"
-		(at 177.8 78.74 0)
+		(at 177.8 86.36 0)
 		(effects
 			(font
@@
 			)
 			(justify right bottom)
+		)
+	)
+	(hierarchical_label "SENSEN"
+		(shape output)
+		(at 170.18 73.66 0)
+		(effects
+			(font
+				(size 1.27 1.27)
+			)
+			(justify left)
 		)
 	)
@@
 	)
 	(symbol
-		(lib_id "power:GND")
-		(at 156.21 73.66 90)
-		(unit 1)
-		(exclude_from_sim no)
-		(in_bom yes)
-		(on_board yes)
-		(dnp no)
-		(fields_autoplaced yes)
-		(property "Reference" "#PWR05"
-			(at 162.56 73.66 0)
-			(effects
-				(font
-					(size 1.27 1.27)
-				)
-				(hide yes)
-			)
-		)
-		(property "Value" "GND"
-			(at 160.02 73.6599 90)
-			(effects
-				(font
-					(size 1.27 1.27)
-				)
-				(justify right)
-			)
-		)
-		(property "Footprint" ""
-			(at 156.21 73.66 0)
-			(effects
-				(font
-					(size 1.27 1.27)
-				)
-				(hide yes)
-			)
-		)
-		(property "Datasheet" ""
-			(at 156.21 73.66 0)
-			(effects
-				(font
-					(size 1.27 1.27)
-				)
-				(hide yes)
-			)
-		)
-		(property "Description" "Power symbol creates a global label with name \"GND\" , ground"
-			(at 156.21 73.66 0)
-			(effects
-				(font
-					(size 1.27 1.27)
-				)
-				(hide yes)
-			)
-		)
-		(pin "1"
-		)
-		(instances
-			(project ""
-				(path "/600cc1cc-74ca-4bfc-97a0-b230eb3afbcd/29478a2e-751a-4158-b6e6-121ba76a9d10"
-					(reference "#PWR05")
-					(unit 1)
-				)
-			)
-		)
-	)
-	(symbol
 		(lib_id "Device:C")
 		(at 217.17 114.3 90)
@@
 	(symbol
 		(lib_id "Device:R_US")
-		(at 171.45 78.74 90)
+		(at 171.45 86.36 90)
 		(unit 1)
 		(exclude_from_sim no)
@@
 		(fields_autoplaced yes)
 		(property "Reference" "R5"
-			(at 171.45 72.39 90)
+			(at 171.45 80.01 90)
 			(effects
 				(font
@@
 		)
 		(property "Value" "10k, 1%"
-			(at 171.45 74.93 90)
+			(at 171.45 82.55 90)
 			(effects
 				(font
@@
 		)
 		(property "Footprint" ""
-			(at 171.704 77.724 90)
+			(at 171.704 85.344 90)
 			(effects
 				(font
@@
 		)
 		(property "Datasheet" "~"
-			(at 171.45 78.74 0)
+			(at 171.45 86.36 0)
 			(effects
 				(font
@@
 		)
 		(property "Description" "Resistor, US symbol"
-			(at 171.45 78.74 0)
+			(at 171.45 86.36 0)
 			(effects
 				(font
@@
 		)
 		(property "Purchase Link" ""
-			(at 171.45 78.74 0)
-			(effects
-				(font
+			(at 171.45 86.36 0)
+			(effects
+				(font

Commit message: Save progress
Connections:
- net Output: no longer U5.10 (VSENSEP)
- net at R10.1, U5.9 (VOUT): now also U5.10 (VSENSEP)
Other:
- note added: "In the DC regime, current across the limiter resistor should be ~0 when the load capacitor is fully charged. Delay in response while capacitor charges: 4.7k, 1.6 nF ± 15% first order RC filter 21.2 kHz ± 15% 5 time constants (0.7% settling) in 38 us 10 time constants (0.004% settling) in 75 us Time to cross range at 3.59 mm/s: 15.4 us, 65k half cycles/second Time to cross range at 0.359 mm/s: 154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"
- note added: "±2.5 mA current drive with 4.7k If connecting SENSEP to VOUT after the current limit resistor, the actual current limit could be more like ±250 uA. Current demands of PMN-PT piezo: 1.6 nF, 2.3 nm/V, 24 V 250 uA, 0.156 V/us, 0.359 mm/s Compare to LiNbO3 kinematic mount: 0.7 nF, 0.48 nm/V, 850 V 21 mA, 30 V/us, 14.4 mm/s"
- moved on the sheet: C5, R10, R5, U5

Commit message: Save progress
Parts:
- added NT12, NT13, NT14, NT15: NetTie_2, symbol Device:NetTie_2
Connections:
- net -15V: now also NT13.2; no longer C16.2, C17.2, U5.3 (AVSS)
- net 15V: now also NT12.2; no longer C14.2, C15.2, U5.5 (AVDD)
- net 3.3V: now also NT15.2; no longer C20.2, R5.2, U5.17 (IOVDD)
- net 5V: now also NT14.2; no longer C18.2, C19.2, U5.20 (DVDD)
- new net AVDD: C14.2, C15.2, NT12.1, U5.5 (AVDD)
- new net AVSS: C16.2, C17.2, NT13.1, U5.3 (AVSS)
- new net DVDD: C18.2, C19.2, NT14.1, U5.20 (DVDD)
- new net IOVDD: C20.2, NT15.1, R5.2, U5.17 (IOVDD)
