File: Models/MainBoard/ADC.kicad_sch (KiCad schematic)
At the start: 11 parts, among them U1 ADS8699

Commit message: Should be finished with components BOM
Parts:
- C1, C3, C5, C7: Cost (none) -> $0.087; Purchase Link (none) -> https://www.digikey.com/en/products/detail/murata-electroni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
- C2, C4, C6: Cost (none) -> $0.078; Purchase Link (none) -> https://www.digikey.com/en/products/detail/murata-electroni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
- R3: Cost (none) -> $0.030; Purchase Link (none) -> https://www.digikey.com/en/products/detail/vishay-dale/CRCW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
Changed lines of the file:
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@@
 			)
 		)
-		(property "Purchase Link" ""
+		(property "Purchase Link" "https://www.digikey.com/en/products/detail/murata-electronics/GRT188R61H105KE13D/5416752"
 			(at 217.17 76.2 0)
+			(effects
+				(font
+					(size 1.27 1.27)
+				)
+				(hide yes)
+			)
+		)
+		(property "Cost" "$0.078"
+			(at 217.17 76.2 90)
 			(effects
 				(font
@@
 			)
 		)
-		(property "Purchase Link" ""
+		(property "Purchase Link" "https://www.digikey.com/en/products/detail/murata-electronics/GRM21BR61E106KA73K/4905532"
 			(at 217.17 114.3 0)
+			(effects
+				(font
+					(size 1.27 1.27)
+				)
+				(hide yes)
+			)
+		)
+		(property "Cost" "$0.087"
+			(at 217.17 114.3 90)
 			(effects
 				(font
@@
 			)
 		)
-		(property "Purchase Link" ""
+		(property "Purchase Link" "https://www.digikey.com/en/products/detail/murata-electronics/GRT188R61H105KE13D/5416752"
 			(at 217.17 50.8 0)
+			(effects
+				(font
+					(size 1.27 1.27)
+				)
+				(hide yes)
+			)
+		)
+		(property "Cost" "$0.078"
+			(at 217.17 50.8 90)
 			(effects
 				(font
@@
 			)
 		)
-		(property "Purchase Link" ""
+		(property "Purchase Link" "https://www.digikey.com/en/products/detail/murata-electronics/GRM21BR61E106KA73K/4905532"
 			(at 217.17 63.5 0)
+			(effects
+				(font
+					(size 1.27 1.27)
+				)
+				(hide yes)
+			)
+		)
+		(property "Cost" "$0.087"
+			(at 217.17 63.5 90)
 			(effects
 				(font
@@
 			)
 		)
+		(property "Cost" "$0.087"
+			(at 50.8 97.79 0)
+			(effects
+				(font
+					(size 1.27 1.27)
+				)
+				(hide yes)
+			)
+		)
+		(property "Purchase Link" "https://www.digikey.com/en/products/detail/murata-electronics/GRM21BR61E106KA73K/4905532"
+			(at 50.8 97.79 0)
+			(effects
+				(font
+					(size 1.27 1.27)
+				)
+				(hide yes)
+			)
+		)
 		(pin "1"
 		)
@@
 			)
 		)
-		(property "Purchase Link" ""
+		(property "Purchase Link" "https://www.digikey.com/en/products/detail/murata-electronics/GRM21BR61E106KA73K/4905532"
 			(at 217.17 88.9 0)
+			(effects
+				(font
+					(size 1.27 1.27)
+				)
+				(hide yes)
+			)
+		)
+		(property "Cost" "$0.087"
+			(at 217.17 88.9 90)
 			(effects
 				(font
@@
 			)
 		)
-		(property "Purchase Link" ""
+		(property "Purchase Link" "https://www.digikey.com/en/products/detail/murata-electronics/GRT188R61H105KE13D/5416752"
 			(at 217.17 101.6 0)
+			(effects
+				(font
+					(size 1.27 1.27)
+				)
+				(hide yes)
+			)
+		)
+		(property "Cost" "$0.078"
+			(at 217.17 101.6 90)
 			(effects
 				(font
@@
 			(effects
 				(font
+					(size 1.27 1.27)
+				)
+				(hide yes)
+			)
+		)
+		(property "Cost" "$0.030"
+			(at 171.45 99.06 90)
+			(effects
+				(font
+					(size 1.27 1.27)
+				)
+				(hide yes)
+			)
+		)
+		(property "Purchase Link" "https://www.digikey.com/en/products/detail/vishay-dale/CRCW060310K0FKEA/1174782"
+			(at 171.45 99.06 90)
+			(effects
+				(font

Commit message: Save progress
Parts:
- U1: Purchase Link https://www.digikey.com/en/products/detail/texas-instrument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 -> (none)
Changed lines of the file:
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@@
 			)
 		)
-		(property "Purchase Link" "https://www.digikey.com/en/products/detail/texas-instruments/ADS8699IPWR/6600065"
+		(property "Purchase Link" ""
 			(at 86.36 81.28 0)
 			(effects

Commit message: Assigned footprints
Parts:
- C1, C3, C5, C7: footprint (none) -> TwoTerminal:CAPC0805
- C2, C4, C6: footprint (none) -> TwoTerminal:CAPC0603
- NT1, NT2: footprint (none) -> Connector_Custom:NetTie_0.2mm
- R3: footprint (none) -> TwoTerminal:RESC0603
- U1: footprint (none) -> IC:TSSOP-16

Commit message: I am overcomplicating the TIA1 board
Parts:
- NT1, NT2: footprint Connector_Custom:NetTie_0.2mm -> Connector_Custom:NetTie_0.15mm
Changed lines of the file:
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@@
 			)
 		)
-		(property "Footprint" "Connector_Custom:NetTie_0.2mm"
+		(property "Footprint" "Connector_Custom:NetTie_0.15mm"
 			(at 233.68 50.8 0)
 			(effects
@@
 			)
 		)
-		(property "Footprint" "Connector_Custom:NetTie_0.2mm"
+		(property "Footprint" "Connector_Custom:NetTie_0.15mm"
 			(at 233.68 76.2 0)
 			(effects

Commit message: Save progress
Parts:
- C1, C2, C3, C4, C5, C6, C7, R3: now left out of the parts list
Changed lines of the file:
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@@
 		(unit 1)
 		(exclude_from_sim no)
-		(in_bom yes)
+		(in_bom no)
 		(on_board yes)
 		(dnp no)
@@
 		(unit 1)
 		(exclude_from_sim no)
-		(in_bom yes)
+		(in_bom no)
 		(on_board yes)
 		(dnp no)
@@
 		(unit 1)
 		(exclude_from_sim no)
-		(in_bom yes)
+		(in_bom no)
 		(on_board yes)
 		(dnp no)
@@
 		(unit 1)
 		(exclude_from_sim no)
-		(in_bom yes)
+		(in_bom no)
 		(on_board yes)
 		(dnp no)
@@
 		(unit 1)
 		(exclude_from_sim no)
-		(in_bom yes)
+		(in_bom no)
 		(on_board yes)
 		(dnp no)
@@
 		(unit 1)
 		(exclude_from_sim no)
-		(in_bom yes)
+		(in_bom no)
 		(on_board yes)
 		(dnp no)
@@
 		(unit 1)
 		(exclude_from_sim no)
-		(in_bom yes)
+		(in_bom no)
 		(on_board yes)
 		(dnp no)
@@
 		(unit 1)
 		(exclude_from_sim no)
-		(in_bom yes)
-		(on_board yes)
-		(dnp no)
+		(in_bom no)
+		(on_board yes)
+		(dnp no)
