File: Models/MainBoard/CDC.kicad_sch (KiCad schematic)
At the start: 0 parts

Commit message: Finished the sensors
Parts:
- added C28: 100 nF, 0603, symbol Device:C
- added C29: 10 uF, 0805, symbol Device:C
- added NT15: NetTie_2, symbol Device:NetTie_2
- added R8, R9: 10k, 1%, symbol Device:R_US
- added U7: AD7745, symbol Custom:AD7745
Connections:
- new net 5V: NT15.2
- new net CIN: U7.8 (CIN1+)
- new net EXC: U7.3 (EXCA)
- new net GND: C28.1, C29.1, U7.13 (GND)
- new net SCL: R9.2, U7.1 (SCL)
- new net SDA: R8.2, U7.16 (SDA)
- new net VDD: C28.2, C29.2, NT15.1, R8.1, R9.1, U7.14 (VDD)
- no-connect marks 0 -> 7

Commit message: Save progress
Parts:
- removed NT15: NetTie_2, symbol Device:NetTie_2
Connections:
- net VDD is gone; now on net 5V: C28.2, C29.2, R8.1, R9.1, U7.14 (VDD)
Changed lines of the file:
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@@
-	(wire
-		(pts
-			(xy 237.49 50.8) (xy 242.57 50.8)
-		)
-		(stroke
-			(width 0)
-			(type default)
-		)
-	)
 	(wire
 		(pts
@@
 	(wire
 		(pts
-			(xy 227.33 50.8) (xy 232.41 50.8)
+			(xy 227.33 50.8) (xy 242.57 50.8)
 		)
 		(stroke
@@
 					(unit 1)
 				)
-			)
-		)
-	)
-	(symbol
-		(lib_id "Device:NetTie_2")
-		(at 234.95 50.8 0)
-		(unit 1)
-		(exclude_from_sim no)
-		(in_bom no)
-		(on_board yes)
-		(dnp no)
-		(fields_autoplaced yes)
-		(property "Reference" "NT15"
-			(at 234.95 45.72 0)
-			(effects
-				(font
-					(size 1.27 1.27)
-				)
-			)
-		)
-		(property "Value" "NetTie_2"
-			(at 234.95 48.26 0)
-			(effects
-				(font
-					(size 1.27 1.27)
-				)
-			)
-		)
-		(property "Footprint" ""
-			(at 234.95 50.8 0)
-			(effects
-				(font
-					(size 1.27 1.27)
-				)
-				(hide yes)
-			)
-		)
-		(property "Datasheet" "~"
-			(at 234.95 50.8 0)
-			(effects
-				(font
-					(size 1.27 1.27)
-				)
-				(hide yes)
-			)
-		)
-		(property "Description" "Net tie, 2 pins"
-			(at 234.95 50.8 0)
-			(effects
-				(font
-					(size 1.27 1.27)
-				)
-				(hide yes)
-			)
-		)
-		(pin "1"
-		)
-		(pin "2"
-		)
-		(instances
-			(project "MainBoard"
-				(path "/600cc1cc-74ca-4bfc-97a0-b230eb3afbcd/812a2394-e6f7-4194-9eea-57be5665ec29"
-					(reference "NT15")
-					(unit 1)
-				)

Commit message: Save progress
Parts:
- added NT7: NetTie_2, symbol Device:NetTie_2
Connections:
- net 5V: now also NT7.2; no longer C28.2, C29.2, R8.1, R9.1, U7.14 (VDD)
- new net VDD: C28.2, C29.2, NT7.1, R8.1, R9.1, U7.14 (VDD)
Other:
- moved on the sheet: C28, C29
Changed lines of the file:
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@@
 	(paper "A4")
-	(junction
-		(at 227.33 50.8)
-		(diameter 0)
-		(color 0 0 0 0)
-	)
 	(junction
 		(at 132.08 78.74)
@@
 	)
 	(junction
+		(at 226.06 50.8)
+		(diameter 0)
+		(color 0 0 0 0)
+	)
+	(junction
 		(at 91.44 78.74)
 		(diameter 0)
@@
 	)
 	(junction
-		(at 227.33 63.5)
+		(at 226.06 63.5)
 		(diameter 0)
 		(color 0 0 0 0)
 	)
 	(junction
-		(at 209.55 50.8)
+		(at 208.28 50.8)
 		(diameter 0)
 		(color 0 0 0 0)
@@
 	(wire
 		(pts
-			(xy 204.47 50.8) (xy 209.55 50.8)
+			(xy 236.22 50.8) (xy 241.3 50.8)
+		)
+		(stroke
+			(width 0)
+			(type default)
+		)
+	)
+	(wire
+		(pts
+			(xy 203.2 50.8) (xy 208.28 50.8)
 		)
 		(stroke
@@
 	(wire
 		(pts
-			(xy 222.25 63.5) (xy 227.33 63.5)
+			(xy 220.98 63.5) (xy 226.06 63.5)
 		)
 		(stroke
@@
 	(wire
 		(pts
-			(xy 209.55 63.5) (xy 214.63 63.5)
+			(xy 208.28 63.5) (xy 213.36 63.5)
 		)
 		(stroke
@@
 	(wire
 		(pts
-			(xy 214.63 50.8) (xy 209.55 50.8)
+			(xy 213.36 50.8) (xy 208.28 50.8)
 		)
 		(stroke
@@
 	(wire
 		(pts
-			(xy 222.25 50.8) (xy 227.33 50.8)
+			(xy 220.98 50.8) (xy 226.06 50.8)
 		)
 		(stroke
@@
 	(wire
 		(pts
+			(xy 226.06 50.8) (xy 231.14 50.8)
+		)
+		(stroke
+			(width 0)
+			(type default)
+		)
+	)
+	(wire
+		(pts
 			(xy 96.52 83.82) (xy 99.06 83.82)
 		)
@@
 	(wire
 		(pts
-			(xy 227.33 63.5) (xy 242.57 63.5)
+			(xy 226.06 63.5) (xy 241.3 63.5)
 		)
 		(stroke
@@
 	(wire
 		(pts
-			(xy 227.33 50.8) (xy 242.57 50.8)
-		)
-		(stroke
-			(width 0)
-			(type default)
-		)
-	)
-	(wire
-		(pts
 			(xy 96.52 96.52) (xy 99.06 96.52)
 		)
@@
 	(wire
 		(pts
-			(xy 227.33 63.5) (xy 227.33 50.8)
-		)
-		(stroke
-			(width 0)
-			(type default)
-		)
-	)
-	(wire
-		(pts
-			(xy 209.55 50.8) (xy 209.55 63.5)
+			(xy 226.06 63.5) (xy 226.06 50.8)
+		)
+		(stroke
+			(width 0)
+			(type default)
+		)
+	)
+	(wire
+		(pts
+			(xy 208.28 50.8) (xy 208.28 63.5)
 		)
 		(stroke
@@
 	)
 	(label "VDD"
-		(at 242.57 63.5 0)
+		(at 241.3 63.5 0)
 		(effects
 			(font
@@
 		)
 	)
-	(hierarchical_label "5V"
+	(global_label "5V"
 		(shape input)
-		(at 242.57 50.8 0)
+		(at 241.3 50.8 0)
+		(fields_autoplaced yes)
 		(effects
 			(font
@@
 			)
 			(justify left)
+		)
+		(property "Intersheetrefs" "${INTERSHEET_REFS}"
+			(at 246.5833 50.8 0)
+			(effects
+				(font
+					(size 1.27 1.27)
+				)
+				(justify left)
+				(hide yes)
+			)
 		)
 	)
@@
 	(symbol
 		(lib_id "power:GND")
-		(at 204.47 50.8 270)
+		(at 203.2 50.8 270)
 		(unit 1)
 		(exclude_from_sim no)
@@
 		(fields_autoplaced yes)
 		(property "Reference" "#PWR026"
-			(at 198.12 50.8 0)
+			(at 196.85 50.8 0)
 			(effects
 				(font
@@
 		)
 		(property "Value" "GND"
-			(at 200.66 50.7999 90)
+			(at 199.39 50.7999 90)
 			(effects
 				(font
@@
 		)
 		(property "Footprint" ""
-			(at 204.47 50.8 0)
+			(at 203.2 50.8 0)
 			(effects
 				(font
@@
 		)
 		(property "Datasheet" ""
-			(at 204.47 50.8 0)
+			(at 203.2 50.8 0)
 			(effects
 				(font
@@
 		)
 		(property "Description" "Power symbol creates a global label with name \"GND\" , ground"
-			(at 204.47 50.8 0)
+			(at 203.2 50.8 0)
 			(effects
 				(font
@@
 	(symbol
 		(lib_id "Device:C")
-		(at 218.44 50.8 90)
+		(at 217.17 50.8 90)
 		(unit 1)
 		(exclude_from_sim no)
@@
 		(fields_autoplaced yes)
 		(property "Reference" "C28"
-			(at 218.44 43.18 90)
+			(at 217.17 43.18 90)
 			(effects
 				(font
@@
 		)
 		(property "Value" "100 nF, 0603"
-			(at 218.44 45.72 90)
+			(at 217.17 45.72 90)
 			(effects
 				(font
@@
 		)
 		(property "Footprint" ""
-			(at 222.25 49.8348 0)
+			(at 220.98 49.8348 0)
 			(effects
 				(font
@@
 		)
 		(property "Datasheet" "~"
-			(at 218.44 50.8 0)
+			(at 217.17 50.8 0)
 			(effects
 				(font
@@
 		)
 		(property "Description" "Unpolarized capacitor"
-			(at 218.44 50.8 0)
+			(at 217.17 50.8 0)
 			(effects
 				(font
@@
 		)
 		(property "Purchase Link" ""
-			(at 218.44 50.8 0)
+			(at 217.17 50.8 0)
 			(effects
 				(font
@@
 	)
 	(symbol
+		(lib_id "Device:NetTie_2")
+		(at 233.68 50.8 0)
+		(unit 1)
+		(exclude_from_sim no)
+		(in_bom no)
+		(on_board yes)
+		(dnp no)
+		(fields_autoplaced yes)
+		(property "Reference" "NT7"
+			(at 233.68 45.72 0)
+			(effects
+				(font
+					(size 1.27 1.27)
+				)
+			)
+		)
+		(property "Value" "NetTie_2"
+			(at 233.68 48.26 0)
+			(effects
+				(font
+					(size 1.27 1.27)
+				)
+			)
+		)
+		(property "Footprint" ""
+			(at 233.68 50.8 0)
+			(effects
+				(font
+					(size 1.27 1.27)
+				)
+				(hide yes)
+			)
+		)
+		(property "Datasheet" "~"
+			(at 233.68 50.8 0)
+			(effects
+				(font
+					(size 1.27 1.27)
+				)
+				(hide yes)
+			)
+		)
+		(property "Description" "Net tie, 2 pins"
+			(at 233.68 50.8 0)
+			(effects
+				(font
+					(size 1.27 1.27)
+				)
+				(hide yes)
+			)
+		)
+		(pin "1"
+		)
+		(pin "2"
+		)
+		(instances
+			(project ""
+				(path "/600cc1cc-74ca-4bfc-97a0-b230eb3afbcd/812a2394-e6f7-4194-9eea-57be5665ec29"
+					(reference "NT7")
+					(unit 1)
+				)
+			)
+		)
+	)
+	(symbol
 		(lib_id "Device:C")
-		(at 218.44 63.5 90)
+		(at 217.17 63.5 90)
 		(unit 1)
 		(exclude_from_sim no)
@@
 		(fields_autoplaced yes)
 		(property "Reference" "C29"
-			(at 218.44 55.88 90)
+			(at 217.17 55.88 90)
 			(effects
 				(font
@@
 		)
 		(property "Value" "10 uF, 0805"
-			(at 218.44 58.42 90)
+			(at 217.17 58.42 90)
 			(effects
 				(font
@@
 		)
 		(property "Footprint" ""
-			(at 222.25 62.5348 0)
+			(at 220.98 62.5348 0)
 			(effects
 				(font
@@
 		)
 		(property "Datasheet" "~"
-			(at 218.44 63.5 0)
+			(at 217.17 63.5 0)
 			(effects
 				(font
@@
 		)
 		(property "Description" "Unpolarized capacitor"
-			(at 218.44 63.5 0)
+			(at 217.17 63.5 0)
 			(effects
 				(font
@@
 		)
 		(property "Purchase Link" ""
-			(at 218.44 63.5 0)
-			(effects
-				(font
+			(at 217.17 63.5 0)
+			(effects
+				(font

Commit message: Passes ERC
Parts:
- renumbered C28 to C8, C29 to C9, NT7 to NT3, R9 to R4, R8 to R5, U7 to U2
Changed lines of the file:
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@@
 		(dnp no)
 		(fields_autoplaced yes)
-		(property "Reference" "R9"
+		(property "Reference" "R4"
 			(at 93.98 71.1199 0)
 			(effects
@@
 			(project "MainBoard"
 				(path "/600cc1cc-74ca-4bfc-97a0-b230eb3afbcd/812a2394-e6f7-4194-9eea-57be5665ec29"
-					(reference "R9")
+					(reference "R4")
 					(unit 1)
 				)
@@
 		(dnp no)
 		(fields_autoplaced yes)
-		(property "Reference" "#PWR025"
+		(property "Reference" "#PWR038"
 			(at 139.7 86.36 0)
 			(effects
@@
 			(project ""
 				(path "/600cc1cc-74ca-4bfc-97a0-b230eb3afbcd/812a2394-e6f7-4194-9eea-57be5665ec29"
-					(reference "#PWR025")
+					(reference "#PWR038")
 					(unit 1)
 				)
@@
 		(dnp no)
 		(fields_autoplaced yes)
-		(property "Reference" "R8"
+		(property "Reference" "R5"
 			(at 134.62 71.1199 0)
 			(effects
@@
 			(project ""
 				(path "/600cc1cc-74ca-4bfc-97a0-b230eb3afbcd/812a2394-e6f7-4194-9eea-57be5665ec29"
-					(reference "R8")
+					(reference "R5")
 					(unit 1)
 				)
@@
 		(dnp no)
 		(fields_autoplaced yes)
-		(property "Reference" "#PWR026"
+		(property "Reference" "#PWR039"
 			(at 196.85 50.8 0)
 			(effects
@@
 			(project "MainBoard"
 				(path "/600cc1cc-74ca-4bfc-97a0-b230eb3afbcd/812a2394-e6f7-4194-9eea-57be5665ec29"
-					(reference "#PWR026")
+					(reference "#PWR039")
 					(unit 1)
 				)
@@
 		(dnp no)
 		(fields_autoplaced yes)
-		(property "Reference" "U7"
+		(property "Reference" "U2"
 			(at 114.3 71.12 0)
 			(effects
@@
 			(project ""
 				(path "/600cc1cc-74ca-4bfc-97a0-b230eb3afbcd/812a2394-e6f7-4194-9eea-57be5665ec29"
-					(reference "U7")
+					(reference "U2")
 					(unit 1)
 				)
@@
 		(dnp no)
 		(fields_autoplaced yes)
-		(property "Reference" "C28"
+		(property "Reference" "C8"
 			(at 217.17 43.18 90)
 			(effects
@@
 			(project "MainBoard"
 				(path "/600cc1cc-74ca-4bfc-97a0-b230eb3afbcd/812a2394-e6f7-4194-9eea-57be5665ec29"
-					(reference "C28")
+					(reference "C8")
 					(unit 1)
 				)
@@
 		(dnp no)
 		(fields_autoplaced yes)
-		(property "Reference" "NT7"
+		(property "Reference" "NT3"
 			(at 233.68 45.72 0)
 			(effects
@@
 			(project ""
 				(path "/600cc1cc-74ca-4bfc-97a0-b230eb3afbcd/812a2394-e6f7-4194-9eea-57be5665ec29"
-					(reference "NT7")
+					(reference "NT3")
 					(unit 1)
 				)
@@
 		(dnp no)
 		(fields_autoplaced yes)
-		(property "Reference" "C29"
+		(property "Reference" "C9"
 			(at 217.17 55.88 90)
 			(effects
@@
 			(project "MainBoard"
 				(path "/600cc1cc-74ca-4bfc-97a0-b230eb3afbcd/812a2394-e6f7-4194-9eea-57be5665ec29"
-					(reference "C29")
-					(unit 1)
-				)
+					(reference "C9")
+					(unit 1)
+				)

Commit message: Save progress
Parts:
- U2: Cost (none) -> $14.230; Purchase Link (none) -> https://www.digikey.com/en/products/detail/analog-devices-i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
Changed lines of the file:
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@@
+			)
+		)
+		(property "Cost" "$14.230"
+			(at 114.3 87.63 0)
+			(effects
+				(font
+					(size 1.27 1.27)
+				)
+				(hide yes)
+			)
+		)
+		(property "Purchase Link" "https://www.digikey.com/en/products/detail/analog-devices-inc/AD7745ARUZ-REEL/994647"
+			(at 114.3 87.63 0)
+			(effects
+				(font
+					(size 1.27 1.27)
+				)
+				(hide yes)
 			)
 		)

Commit message: Should be finished with components BOM
Parts:
- C8: Cost (none) -> $0.079; Purchase Link (none) -> https://www.digikey.com/en/products/detail/murata-electroni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
- C9: Cost (none) -> $0.087; Purchase Link (none) -> https://www.digikey.com/en/products/detail/murata-electroni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
- R4, R5: Cost (none) -> $0.030; Purchase Link (none) -> https://www.digikey.com/en/products/detail/vishay-dale/CRCW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
Changed lines of the file:
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@@
+			)
+		)
+		(property "Cost" "$0.030"
+			(at 91.44 72.39 0)
+			(effects
+				(font
+					(size 1.27 1.27)
+				)
+				(hide yes)
+			)
+		)
+		(property "Purchase Link" "https://www.digikey.com/en/products/detail/vishay-dale/CRCW060310K0FKEA/1174782"
+			(at 91.44 72.39 0)
+			(effects
+				(font
+					(size 1.27 1.27)
+				)
+				(hide yes)
 			)
 		)
@@
 			)
 		)
+		(property "Cost" "$0.030"
+			(at 132.08 72.39 0)
+			(effects
+				(font
+					(size 1.27 1.27)
+				)
+				(hide yes)
+			)
+		)
+		(property "Purchase Link" "https://www.digikey.com/en/products/detail/vishay-dale/CRCW060310K0FKEA/1174782"
+			(at 132.08 72.39 0)
+			(effects
+				(font
+					(size 1.27 1.27)
+				)
+				(hide yes)
+			)
+		)
 		(pin "2"
 		)
@@
 			)
 		)
-		(property "Purchase Link" ""
+		(property "Purchase Link" "https://www.digikey.com/en/products/detail/murata-electronics/GRM188R72A104KA35D/702549"
 			(at 217.17 50.8 0)
+			(effects
+				(font
+					(size 1.27 1.27)
+				)
+				(hide yes)
+			)
+		)
+		(property "Cost" "$0.079"
+			(at 217.17 50.8 90)
 			(effects
 				(font
@@
 			)
 		)
-		(property "Purchase Link" ""
+		(property "Purchase Link" "https://www.digikey.com/en/products/detail/murata-electronics/GRM21BR61E106KA73K/4905532"
 			(at 217.17 63.5 0)
 			(effects
 				(font
+					(size 1.27 1.27)
+				)
+				(hide yes)
+			)
+		)
+		(property "Cost" "$0.087"
+			(at 217.17 63.5 90)
+			(effects
+				(font

Commit message: Assigned footprints
Parts:
- C8: footprint (none) -> TwoTerminal:CAPC0603
- C9: footprint (none) -> TwoTerminal:CAPC0805
- NT3: footprint (none) -> Connector_Custom:NetTie_0.2mm
- R4, R5: footprint (none) -> TwoTerminal:RESC0603
- U2: footprint (none) -> IC:TSSOP-16
Changed lines of the file:
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@@
 			)
 		)
-		(property "Footprint" ""
+		(property "Footprint" "TwoTerminal:RESC0603"
 			(at 92.456 72.644 90)
 			(effects
@@
 			)
 		)
-		(property "Footprint" ""
+		(property "Footprint" "TwoTerminal:RESC0603"
 			(at 133.096 72.644 90)
 			(effects
@@
 			)
 		)
-		(property "Footprint" ""
+		(property "Footprint" "IC:TSSOP-16"
 			(at 114.3 87.63 0)
 			(effects
@@
 			)
 		)
-		(property "Footprint" ""
+		(property "Footprint" "TwoTerminal:CAPC0603"
 			(at 220.98 49.8348 0)
 			(effects
@@
 			)
 		)
-		(property "Footprint" ""
+		(property "Footprint" "Connector_Custom:NetTie_0.2mm"
 			(at 233.68 50.8 0)
 			(effects
@@
 			)
 		)
-		(property "Footprint" ""
+		(property "Footprint" "TwoTerminal:CAPC0805"
 			(at 220.98 62.5348 0)
 			(effects
