File: Models/MainBoard/CDC.kicad_sch (KiCad schematic)
At the start: 6 parts, among them U2 AD7745

Commit message: I am overcomplicating the TIA1 board
Parts:
- NT3: footprint Connector_Custom:NetTie_0.2mm -> Connector_Custom:NetTie_0.15mm
Changed lines of the file:
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@@
 			)
 		)
-		(property "Footprint" "Connector_Custom:NetTie_0.2mm"
+		(property "Footprint" "Connector_Custom:NetTie_0.15mm"
 			(at 233.68 50.8 0)
 			(effects

Commit message: Save progress
Parts:
- C8, C9, R4, R5: now left out of the parts list
Changed lines of the file:
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@@
 		(unit 1)
 		(exclude_from_sim no)
-		(in_bom yes)
+		(in_bom no)
 		(on_board yes)
 		(dnp no)
@@
 		(unit 1)
 		(exclude_from_sim no)
-		(in_bom yes)
+		(in_bom no)
 		(on_board yes)
 		(dnp no)
@@
 		(unit 1)
 		(exclude_from_sim no)
-		(in_bom yes)
+		(in_bom no)
 		(on_board yes)
 		(dnp no)
@@
 		(unit 1)
 		(exclude_from_sim no)
-		(in_bom yes)
-		(on_board yes)
-		(dnp no)
+		(in_bom no)
+		(on_board yes)
+		(dnp no)
