File: Models/MainBoard/Teensy.kicad_sch (KiCad schematic)
At the start: 0 parts

Commit message: Save progress
Parts:
- added J1, J2: Conn_01x24_Pin, symbol Connector:Conn_01x24_Pin
- added J3, J4: Conn_01x24_Socket, symbol Connector:Conn_01x24_Socket
- added U1: Teensy4.1, symbol teensy:Teensy4.1
Connections:
- new net: J1.1 (Pin_1), U1.25 (33_MCLK2)
- new net: J1.10 (Pin_10), U1.34 (GND)
- new net: J1.11 (Pin_11), U1.35 (13_SCK_LED)
- new net: J1.12 (Pin_12), U1.36 (14_A0_TX3_SPDIF_OUT)
- new net: J1.13 (Pin_13), U1.37 (15_A1_RX3_SPDIF_IN)
- new net: J1.14 (Pin_14), U1.38 (16_A2_RX4_SCL1)
- new net: J1.15 (Pin_15), U1.39 (17_A3_TX4_SDA1)
- new net: J1.16 (Pin_16), U1.40 (18_A4_SDA)
- new net: J1.17 (Pin_17), U1.41 (19_A5_SCL)
- new net: J1.18 (Pin_18), U1.42 (20_A6_TX5_LRCLK1)
- new net: J1.19 (Pin_19), U1.43 (21_A7_RX5_BCLK1)
- new net: J1.2 (Pin_2), U1.26 (34_RX8)
- new net: J1.20 (Pin_20), U1.44 (22_A8_CTX1)
- new net: J1.21 (Pin_21), U1.45 (23_A9_CRX1_MCLK1)
- new net: J1.22 (Pin_22), U1.46 (3V3)
- new net: J1.23 (Pin_23), U1.47 (GND)
- new net: J1.24 (Pin_24), U1.48 (VIN)
- new net: J1.3 (Pin_3), U1.27 (35_TX8)
- new net: J1.4 (Pin_4), U1.28 (36_CS)
- new net: J1.5 (Pin_5), U1.29 (37_CS)
- new net: J1.6 (Pin_6), U1.30 (38_CS1_IN1)
- new net: J1.7 (Pin_7), U1.31 (39_MISO1_OUT1A)
- new net: J1.8 (Pin_8), U1.32 (40_A16)
- new net: J1.9 (Pin_9), U1.33 (41_A17)
- new net: J2.1 (Pin_1), U1.1 (GND)
- new net: J2.10 (Pin_10), U1.10 (8_TX2_IN1)
- new net: J2.11 (Pin_11), U1.11 (9_OUT1C)
- new net: J2.12 (Pin_12), U1.12 (10_CS_MQSR)
- new net: J2.13 (Pin_13), U1.13 (11_MOSI_CTX1)
- new net: J2.14 (Pin_14), U1.14 (12_MISO_MQSL)
- new net: J2.15 (Pin_15), U1.15 (3V3)
- new net: J2.16 (Pin_16), U1.16 (24_A10_TX6_SCL2)
- new net: J2.17 (Pin_17), U1.17 (25_A11_RX6_SDA2)
- new net: J2.18 (Pin_18), U1.18 (26_A12_MOSI1)
- new net: J2.19 (Pin_19), U1.19 (27_A13_SCK1)
- new net: J2.2 (Pin_2), U1.2 (0_RX1_CRX2_CS1)
- new net: J2.20 (Pin_20), U1.20 (28_RX7)
- new net: J2.21 (Pin_21), U1.21 (29_TX7)
- new net: J2.22 (Pin_22), U1.22 (30_CRX3)
- new net: J2.23 (Pin_23), U1.23 (31_CTX3)
- new net: J2.24 (Pin_24), U1.24 (32_OUT1B)
- new net: J2.3 (Pin_3), U1.3 (1_TX1_CTX2_MISO1)
- new net: J2.4 (Pin_4), U1.4 (2_OUT2)
- new net: J2.5 (Pin_5), U1.5 (3_LRCLK2)
- new net: J2.6 (Pin_6), U1.6 (4_BCLK2)
- new net: J2.7 (Pin_7), U1.7 (5_IN2)
- new net: J2.8 (Pin_8), U1.8 (6_OUT1D)
- new net: J2.9 (Pin_9), U1.9 (7_RX2_OUT1A)
- no-connect marks 0 -> 19

Commit message: Save progress
Parts:
- J1, J2, U1: now left out of the parts list
- J3, J4: Cost (none) -> $1.350; Purchase Link (none) -> https://www.digikey.com/en/products/detail/sullins-connecto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
Changed lines of the file:
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@@
+			)
+		)
+		(property "Purchase Link" "https://www.digikey.com/en/products/detail/sullins-connector-solutions/PPPC241LFBN-RC/810196"
+			(at 96.52 90.17 0)
+			(effects
+				(font
+					(size 1.27 1.27)
+				)
+				(hide yes)
+			)
+		)
+		(property "Cost" "$1.350"
+			(at 96.52 90.17 0)
+			(effects
+				(font
+					(size 1.27 1.27)
+				)
+				(hide yes)
 			)
 		)
@@
 			)
 		)
+		(property "Purchase Link" "https://www.digikey.com/en/products/detail/sullins-connector-solutions/PPPC241LFBN-RC/810196"
+			(at 208.28 92.71 0)
+			(effects
+				(font
+					(size 1.27 1.27)
+				)
+				(hide yes)
+			)
+		)
+		(property "Cost" "$1.350"
+			(at 208.28 92.71 0)
+			(effects
+				(font
+					(size 1.27 1.27)
+				)
+				(hide yes)
+			)
+		)
 		(pin "15"
 		)
@@
 		(unit 1)
 		(exclude_from_sim no)
-		(in_bom yes)
-		(on_board yes)
+		(in_bom no)
+		(on_board no)
 		(dnp no)
 		(property "Reference" "J1"
@@
 		)
 		(property "Description" "Generic connector, single row, 01x24, script generated"
+			(at 119.38 90.17 0)
+			(effects
+				(font
+					(size 1.27 1.27)
+				)
+				(hide yes)
+			)
+		)
+		(property "Purchase Link" ""
 			(at 119.38 90.17 0)
 			(effects
@@
 		(unit 1)
 		(exclude_from_sim no)
-		(in_bom yes)
-		(on_board yes)
+		(in_bom no)
+		(on_board no)
 		(dnp no)
 		(property "Reference" "J2"
@@
 		)
 		(property "Description" "Generic connector, single row, 01x24, script generated"
+			(at 185.42 92.71 0)
+			(effects
+				(font
+					(size 1.27 1.27)
+				)
+				(hide yes)
+			)
+		)
+		(property "Purchase Link" ""
 			(at 185.42 92.71 0)
 			(effects
@@
 		(unit 1)
 		(exclude_from_sim no)
-		(in_bom yes)
-		(on_board yes)
+		(in_bom no)
+		(on_board no)
 		(dnp no)
 		(fields_autoplaced yes)
@@
 			(at 152.4 66.04 0)
 			(effects
+				(font
+					(size 1.27 1.27)
+				)
+				(hide yes)
+			)
+		)
+		(property "Purchase Link" ""
+			(at 152.4 66.04 0)
+			(effects

Commit message: Should be at a major turning point in the project
Connections:
- net GND: now reaches J3.10 (Pin_10)
- net GND: now also J3.23 (Pin_23), J4.1 (Pin_1)
- net SCK: now reaches J3.11 (Pin_11)
- net SDA: now reaches J3.16 (Pin_16)
- net SCL: now reaches J3.17 (Pin_17)
- net 3.3V: now reaches J3.22 (Pin_22)
- net CS1: now reaches J3.4 (Pin_4)
- net CS2: now reaches J3.5 (Pin_5)
- net CS3: now reaches J4.12 (Pin_12)
- net MOSI: now reaches J4.13 (Pin_13)
- net MISO: now reaches J4.14 (Pin_14)
- no-connect marks 19 -> 55
Other:
- moved on the sheet: J1, J2, J3, J4, U1

Commit message: Passes ERC
Parts:
- renumbered J3 to J15, J1 to J16, J2 to J17, J4 to J18, U1 to U7
Changed lines of the file:
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@@
 		(on_board yes)
 		(dnp no)
-		(property "Reference" "J3"
+		(property "Reference" "J15"
 			(at 94.488 57.658 0)
 			(effects
@@
 			(project ""
 				(path "/600cc1cc-74ca-4bfc-97a0-b230eb3afbcd/06f343a1-8f8d-44f8-9a8d-c3164f0f170f"
-					(reference "J3")
+					(reference "J15")
 					(unit 1)
 				)
@@
 		(on_board yes)
 		(dnp no)
-		(property "Reference" "J4"
+		(property "Reference" "J18"
 			(at 209.296 56.896 0)
 			(effects
@@
 			(project ""
 				(path "/600cc1cc-74ca-4bfc-97a0-b230eb3afbcd/06f343a1-8f8d-44f8-9a8d-c3164f0f170f"
-					(reference "J4")
+					(reference "J18")
 					(unit 1)
 				)
@@
 		(on_board no)
 		(dnp no)
-		(property "Reference" "J1"
+		(property "Reference" "J16"
 			(at 121.412 56.896 0)
 			(effects
@@
 			(project ""
 				(path "/600cc1cc-74ca-4bfc-97a0-b230eb3afbcd/06f343a1-8f8d-44f8-9a8d-c3164f0f170f"
-					(reference "J1")
+					(reference "J16")
 					(unit 1)
 				)
@@
 		(on_board no)
 		(dnp no)
-		(property "Reference" "J2"
+		(property "Reference" "J17"
 			(at 183.896 57.404 0)
 			(effects
@@
 			(project ""
 				(path "/600cc1cc-74ca-4bfc-97a0-b230eb3afbcd/06f343a1-8f8d-44f8-9a8d-c3164f0f170f"
-					(reference "J2")
+					(reference "J17")
 					(unit 1)
 				)
@@
 		(dnp no)
 		(fields_autoplaced yes)
-		(property "Reference" "U1"
+		(property "Reference" "U7"
 			(at 152.4 130.81 0)
 			(effects
@@
 			(project ""
 				(path "/600cc1cc-74ca-4bfc-97a0-b230eb3afbcd/06f343a1-8f8d-44f8-9a8d-c3164f0f170f"
-					(reference "U1")
+					(reference "U7")
 					(unit 1)
 				)

Commit message: Assigned footprints
Parts:
- J15, J18: footprint (none) -> Connector_Custom:PinConnector_1x24
Changed lines of the file:
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@@
 			)
 		)
-		(property "Footprint" ""
+		(property "Footprint" "Connector_Custom:PinConnector_1x24"
 			(at 96.52 91.44 0)
 			(effects
@@
 			)
 		)
-		(property "Footprint" ""
+		(property "Footprint" "Connector_Custom:PinConnector_1x24"
 			(at 208.28 93.98 0)
 			(effects

Commit message: Save progress
Parts:
- renumbered J15 to J16, J16 to J17, J17 to J18, J18 to J19
Changed lines of the file:
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@@
 		(on_board yes)
 		(dnp no)
-		(property "Reference" "J15"
+		(property "Reference" "J16"
 			(at 94.488 57.658 0)
 			(effects
@@
 			(project ""
 				(path "/600cc1cc-74ca-4bfc-97a0-b230eb3afbcd/06f343a1-8f8d-44f8-9a8d-c3164f0f170f"
-					(reference "J15")
+					(reference "J16")
 					(unit 1)
 				)
@@
 		(on_board yes)
 		(dnp no)
-		(property "Reference" "J18"
+		(property "Reference" "J19"
 			(at 209.296 56.896 0)
 			(effects
@@
 			(project ""
 				(path "/600cc1cc-74ca-4bfc-97a0-b230eb3afbcd/06f343a1-8f8d-44f8-9a8d-c3164f0f170f"
-					(reference "J18")
+					(reference "J19")
 					(unit 1)
 				)
@@
 		(on_board no)
 		(dnp no)
-		(property "Reference" "J16"
+		(property "Reference" "J17"
 			(at 121.412 56.896 0)
 			(effects
@@
 			(project ""
 				(path "/600cc1cc-74ca-4bfc-97a0-b230eb3afbcd/06f343a1-8f8d-44f8-9a8d-c3164f0f170f"
-					(reference "J16")
+					(reference "J17")
 					(unit 1)
 				)
@@
 		(on_board no)
 		(dnp no)
-		(property "Reference" "J17"
+		(property "Reference" "J18"
 			(at 183.896 57.404 0)
 			(effects
@@
 			(project ""
 				(path "/600cc1cc-74ca-4bfc-97a0-b230eb3afbcd/06f343a1-8f8d-44f8-9a8d-c3164f0f170f"
-					(reference "J17")
+					(reference "J18")
 					(unit 1)
 				)

Commit message: Save progress
Parts:
- J16, J19: footprint Connector_Custom:PinConnector_1x24 -> Connector_Custom:PinSocket_1x24
Changed lines of the file:
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@@
 			)
 		)
-		(property "Footprint" "Connector_Custom:PinConnector_1x24"
+		(property "Footprint" "Connector_Custom:PinSocket_1x24"
 			(at 96.52 91.44 0)
 			(effects
@@
 			)
 		)
-		(property "Footprint" "Connector_Custom:PinConnector_1x24"
+		(property "Footprint" "Connector_Custom:PinSocket_1x24"
 			(at 208.28 93.98 0)
 			(effects

Commit message: Save progress
Parts:
- J16, J19: now left out of the parts list
Changed lines of the file:
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@@
 		(unit 1)
 		(exclude_from_sim no)
-		(in_bom yes)
+		(in_bom no)
 		(on_board yes)
 		(dnp no)
@@
 		(unit 1)
 		(exclude_from_sim no)
-		(in_bom yes)
+		(in_bom no)
 		(on_board yes)
 		(dnp no)
