File: Models/TransimpedanceAmplifier/TransimpedanceAmplifier.kicad_sch (KiCad schematic)
At the start: 0 parts

Commit message: Save progress
Other:
- added sheet Sensor (Sensor.kicad_sch)
- note added: "Input: 15V power (grounded interconnect) Input: -15V power (grounded interconnect) Input: current Output: voltage (grounded interconnect)"
Changed lines of the file:
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@@
 	(generator_version "9.0")
 	(paper "A4")
+	(text "Input: 15V power (grounded interconnect)\nInput: -15V power (grounded interconnect)\nInput: current\nOutput: voltage (grounded interconnect)"
+		(exclude_from_sim no)
+		(at 158.242 76.962 0)
+		(effects
+			(font
+				(size 1.27 1.27)
+			)
+			(justify left top)
+		)
+	)
+	(sheet
+		(at 101.6 76.2)
+		(size 50.8 50.8)
+		(exclude_from_sim no)
+		(in_bom yes)
+		(on_board yes)
+		(dnp no)
+		(fields_autoplaced yes)
+		(stroke
+			(width 0.1524)
+			(type solid)
+		)
+		(fill
+			(color 0 0 0 0.0000)
+		)
+		(property "Sheetname" "Sensor"
+			(at 101.6 75.4884 0)
+			(effects
+				(font
+					(size 1.27 1.27)
+				)
+				(justify left bottom)
+			)
+		)
+		(property "Sheetfile" "Sensor.kicad_sch"
+			(at 101.6 127.5846 0)
+			(effects
+				(font
+					(size 1.27 1.27)
+				)
+				(justify left top)
+			)
+		)
+		(instances
+			(project "TransimpedanceAmplifier"
+				(path "/f19129fc-f916-4692-924c-ee308c6b3e1d"
+					(page "2")
+				)
+			)
+		)
+	)
 	(sheet_instances
 		(path "/"

Commit message: Save progress
Other:
- removed sheet Sensor
- added sheet Amplifier (Amplifier.kicad_sch)
Changed lines of the file:
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@@
 			(color 0 0 0 0.0000)
 		)
-		(property "Sheetname" "Sensor"
+		(property "Sheetname" "Amplifier"
 			(at 101.6 75.4884 0)
 			(effects
@@
 			)
 		)
-		(property "Sheetfile" "Sensor.kicad_sch"
+		(property "Sheetfile" "Amplifier.kicad_sch"
 			(at 101.6 127.5846 0)
 			(effects
