File: Models/PowerBoard/TIA2_Post.kicad_sch (KiCad schematic)
At the start: 0 parts

Commit message: Save progress
Other:
- added sheet Amplifier (Amplifier.kicad_sch)
- note added: "Input: 15V power Input: -15V power Input: AD8615 output Output: post voltage"
Changed lines of the file:
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@@
 	(generator_version "9.0")
 	(paper "A4")
+	(text "Input: 15V power\nInput: -15V power\nInput: AD8615 output\nOutput: post voltage"
+		(exclude_from_sim no)
+		(at 172.212 103.124 0)
+		(effects
+			(font
+				(size 1.27 1.27)
+			)
+			(justify left top)
+		)
+	)
+	(sheet
+		(at 127 101.6)
+		(size 40.64 30.48)
+		(exclude_from_sim no)
+		(in_bom yes)
+		(on_board yes)
+		(dnp no)
+		(fields_autoplaced yes)
+		(stroke
+			(width 0.1524)
+			(type solid)
+		)
+		(fill
+			(color 0 0 0 0.0000)
+		)
+		(property "Sheetname" "Amplifier"
+			(at 127 100.8884 0)
+			(effects
+				(font
+					(size 1.27 1.27)
+				)
+				(justify left bottom)
+			)
+		)
+		(property "Sheetfile" "Amplifier.kicad_sch"
+			(at 127 132.6646 0)
+			(effects
+				(font
+					(size 1.27 1.27)
+				)
+				(justify left top)
+			)
+		)
+		(instances
+			(project "PowerBoard"
+				(path "/c19e9b7b-7f36-470c-862a-1a648d3f14f6/3c1c1dcd-dbca-4c3e-a9c0-5c49f174be9d"
+					(page "7")
+				)
+			)
+		)
+	)
 )
