File: Models/PowerBoard/PowerBoard.kicad_sch (KiCad schematic)
At the start: 0 parts

Commit message: Save progress
Changed lines of the file:
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@@
 	(paper "A4")
 	(sheet
-		(at 50.8 50.8)
+		(at 50.8 76.2)
 		(size 50.8 50.8)
 		(exclude_from_sim no)
@@
 		)
 		(property "Sheetname" "WallPower"
-			(at 50.8 50.0884 0)
+			(at 50.8 75.4884 0)
 			(effects
 				(font
@@
 		)
 		(property "Sheetfile" "WallPower.kicad_sch"
-			(at 50.8 102.1846 0)
+			(at 50.8 127.5846 0)
 			(effects
 				(font
@@
 		)
 		(instances
-			(project "MainBoard"
-				(path "/600cc1cc-74ca-4bfc-97a0-b230eb3afbcd/d30698e6-a0ca-49f4-86ac-6bca70afd28d"
+			(project "PowerBoard"
+				(path "/c19e9b7b-7f36-470c-862a-1a648d3f14f6"
+					(page "2")
+				)
+			)
+		)
+	)
+	(sheet
+		(at 127 76.2)
+		(size 50.8 50.8)
+		(exclude_from_sim no)
+		(in_bom yes)
+		(on_board yes)
+		(dnp no)
+		(fields_autoplaced yes)
+		(stroke
+			(width 0.1524)
+			(type solid)
+		)
+		(fill
+			(color 0 0 0 0.0000)
+		)
+		(property "Sheetname" "HighVoltage"
+			(at 127 75.4884 0)
+			(effects
+				(font
+					(size 1.27 1.27)
+				)
+				(justify left bottom)
+			)
+		)
+		(property "Sheetfile" "HighVoltage.kicad_sch"
+			(at 127 127.5846 0)
+			(effects
+				(font
+					(size 1.27 1.27)
+				)
+				(justify left top)
+			)
+		)
+		(instances
+			(project "PowerBoard"
+				(path "/c19e9b7b-7f36-470c-862a-1a648d3f14f6"
 					(page "3")
 				)
@@
 	)
 	(sheet
-		(at 203.2 50.8)
+		(at 203.2 76.2)
 		(size 50.8 50.8)
 		(exclude_from_sim no)
@@
 		)
 		(property "Sheetname" "LowVoltage"
-			(at 203.2 50.0884 0)
+			(at 203.2 75.4884 0)
 			(effects
 				(font
@@
 		)
 		(property "Sheetfile" "LowVoltage.kicad_sch"
-			(at 203.2 102.1846 0)
+			(at 203.2 127.5846 0)
 			(effects
 				(font
@@
 		)
 		(instances
-			(project "MainBoard"
-				(path "/600cc1cc-74ca-4bfc-97a0-b230eb3afbcd/d30698e6-a0ca-49f4-86ac-6bca70afd28d"
-					(page "5")
-				)
-			)
-		)
-	)
-	(sheet
-		(at 127 50.8)
-		(size 50.8 50.8)
-		(exclude_from_sim no)
-		(in_bom yes)
-		(on_board yes)
-		(dnp no)
-		(fields_autoplaced yes)
-		(stroke
-			(width 0.1524)
-			(type solid)
-		)
-		(fill
-			(color 0 0 0 0.0000)
-		)
-		(property "Sheetname" "HighVoltage"
-			(at 127 50.0884 0)
-			(effects
-				(font
-					(size 1.27 1.27)
-				)
-				(justify left bottom)
-			)
-		)
-		(property "Sheetfile" "HighVoltage.kicad_sch"
-			(at 127 102.1846 0)
-			(effects
-				(font
-					(size 1.27 1.27)
-				)
-				(justify left top)
-			)
-		)
-		(instances
-			(project "MainBoard"
-				(path "/600cc1cc-74ca-4bfc-97a0-b230eb3afbcd/d30698e6-a0ca-49f4-86ac-6bca70afd28d"
+			(project "PowerBoard"
+				(path "/c19e9b7b-7f36-470c-862a-1a648d3f14f6"
 					(page "4")
 				)
@@
 		)
 	)
+	(sheet_instances
+		(path "/"
+			(page "1")
+		)
+	)
+	(embedded_fonts no)
 )

Commit message: Save progress
Other:
- removed sheet HighVoltage
- added sheet HighVoltage1 (HighVoltagePair.kicad_sch)
- added sheet HighVoltage2 (HighVoltagePair.kicad_sch)
- sheet LowVoltage ports: added 18V; removed none
- sheet WallPower ports: added -18V, 18V; removed none
Changed lines of the file:
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@@
 	(paper "A4")
 	(sheet
-		(at 50.8 76.2)
-		(size 50.8 50.8)
+		(at 152.4 76.2)
+		(size 50.8 25.4)
+		(exclude_from_sim no)
+		(in_bom yes)
+		(on_board yes)
+		(dnp no)
+		(fields_autoplaced yes)
+		(stroke
+			(width 0.1524)
+			(type solid)
+		)
+		(fill
+			(color 0 0 0 0.0000)
+		)
+		(property "Sheetname" "HighVoltage1"
+			(at 152.4 75.4884 0)
+			(effects
+				(font
+					(size 1.27 1.27)
+				)
+				(justify left bottom)
+			)
+		)
+		(property "Sheetfile" "HighVoltagePair.kicad_sch"
+			(at 152.4 102.1846 0)
+			(effects
+				(font
+					(size 1.27 1.27)
+				)
+				(justify left top)
+			)
+		)
+		(instances
+			(project "PowerBoard"
+				(path "/c19e9b7b-7f36-470c-862a-1a648d3f14f6"
+					(page "4")
+				)
+			)
+		)
+	)
+	(sheet
+		(at 50.8 101.6)
+		(size 50.8 25.4)
 		(exclude_from_sim no)
 		(in_bom yes)
@@
 		)
 		(property "Sheetname" "WallPower"
-			(at 50.8 75.4884 0)
+			(at 50.8 100.8884 0)
 			(effects
 				(font
@@
 			)
 		)
+		(pin "-18V" output
+			(at 101.6 121.92 0)
+			(effects
+				(font
+					(size 1.27 1.27)
+				)
+				(justify right)
+			)
+		)
+		(pin "18V" output
+			(at 101.6 106.68 0)
+			(effects
+				(font
+					(size 1.27 1.27)
+				)
+				(justify right)
+			)
+		)
 		(instances
 			(project "PowerBoard"
@@
 	)
 	(sheet
-		(at 127 76.2)
-		(size 50.8 50.8)
+		(at 152.4 127)
+		(size 50.8 25.4)
 		(exclude_from_sim no)
 		(in_bom yes)
@@
 			(color 0 0 0 0.0000)
 		)
-		(property "Sheetname" "HighVoltage"
-			(at 127 75.4884 0)
+		(property "Sheetname" "HighVoltage2"
+			(at 152.4 126.2884 0)
 			(effects
 				(font
@@
 			)
 		)
-		(property "Sheetfile" "HighVoltage.kicad_sch"
-			(at 127 127.5846 0)
+		(property "Sheetfile" "HighVoltagePair.kicad_sch"
+			(at 152.4 152.9846 0)
 			(effects
 				(font
@@
 			(project "PowerBoard"
 				(path "/c19e9b7b-7f36-470c-862a-1a648d3f14f6"
-					(page "3")
+					(page "5")
 				)
 			)
@@
 	)
 	(sheet
-		(at 203.2 76.2)
-		(size 50.8 50.8)
+		(at 152.4 25.4)
+		(size 50.8 25.4)
 		(exclude_from_sim no)
 		(in_bom yes)
@@
 		)
 		(property "Sheetname" "LowVoltage"
-			(at 203.2 75.4884 0)
+			(at 152.4 24.6884 0)
 			(effects
 				(font
@@
 		)
 		(property "Sheetfile" "LowVoltage.kicad_sch"
-			(at 203.2 127.5846 0)
+			(at 152.4 51.3846 0)
 			(effects
 				(font
@@
 			)
 		)
+		(pin "18V" input
+			(at 152.4 30.48 180)
+			(effects
+				(font
+					(size 1.27 1.27)
+				)
+				(justify left)
+			)
+		)

Commit message: Save progress
Other:
- sheet HighVoltage1 renamed 15V
- sheet HighVoltage2 renamed PreAmp
- sheet LowVoltage renamed Converter
- added sheet TIA2_Post (TIA2_Post.kicad_sch)
- sheet 15V: file HighVoltagePair.kicad_sch -> 15V.kicad_sch
- sheet Converter: file LowVoltage.kicad_sch -> Converter.kicad_sch
- sheet Converter ports: added none; removed 18V
- sheet PreAmp: file HighVoltagePair.kicad_sch -> PreAmp.kicad_sch
- note added: "Input: 15V power Input: -15V power Input: pre voltage Input: AD8615 output Output: post voltage Ground receptacles(s) for preamp not yet elaborated"
- note added: "Input: 18V power Input: -18V power Output: 15V power Output: -15V power"
- note added: "Input: 18V power Input: -18V power Output: 2.5V power Output: -1.5V power"
- note added: "Input: 18V power Output: 5V power Output: 3.3V power"
Changed lines of the file:
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@@
 	(generator_version "9.0")
 	(paper "A4")
-	(sheet
-		(at 152.4 76.2)
-		(size 50.8 25.4)
-		(exclude_from_sim no)
-		(in_bom yes)
-		(on_board yes)
-		(dnp no)
-		(fields_autoplaced yes)
-		(stroke
-			(width 0.1524)
-			(type solid)
-		)
-		(fill
-			(color 0 0 0 0.0000)
-		)
-		(property "Sheetname" "HighVoltage1"
-			(at 152.4 75.4884 0)
-			(effects
-				(font
-					(size 1.27 1.27)
-				)
-				(justify left bottom)
-			)
-		)
-		(property "Sheetfile" "HighVoltagePair.kicad_sch"
-			(at 152.4 102.1846 0)
+	(text "Input: 18V power\nOutput: 5V power\nOutput: 3.3V power"
+		(exclude_from_sim no)
+		(at 206.756 27.178 0)
+		(effects
+			(font
+				(size 1.27 1.27)
+			)
+			(justify left top)
+		)
+	)
+	(text "Input: 15V power\nInput: -15V power\nInput: pre voltage\nInput: AD8615 output\nOutput: post voltage\n\nGround receptacles(s) for\npreamp not yet elaborated"
+		(exclude_from_sim no)
+		(at 104.394 128.016 0)
+		(effects
+			(font
+				(size 1.27 1.27)
+			)
+			(justify left top)
+		)
+	)
+	(text "Input: 18V power\nInput: -18V power\nOutput: 2.5V power\nOutput: -1.5V power"
+		(exclude_from_sim no)
+		(at 206.248 102.87 0)
+		(effects
+			(font
+				(size 1.27 1.27)
+			)
+			(justify left top)
+		)
+	)
+	(text "Input: 18V power\nInput: -18V power\nOutput: 15V power\nOutput: -15V power"
+		(exclude_from_sim no)
+		(at 206.248 64.516 0)
+		(effects
+			(font
+				(size 1.27 1.27)
+			)
+			(justify left top)
+		)
+	)
+	(sheet
+		(at 152.4 63.5)
+		(size 50.8 25.4)
+		(exclude_from_sim no)
+		(in_bom yes)
+		(on_board yes)
+		(dnp no)
+		(fields_autoplaced yes)
+		(stroke
+			(width 0.1524)
+			(type solid)
+		)
+		(fill
+			(color 0 0 0 0.0000)
+		)
+		(property "Sheetname" "15V"
+			(at 152.4 62.7884 0)
+			(effects
+				(font
+					(size 1.27 1.27)
+				)
+				(justify left bottom)
+			)
+		)
+		(property "Sheetfile" "15V.kicad_sch"
+			(at 152.4 89.4846 0)
 			(effects
 				(font
@@
 	)
 	(sheet
-		(at 50.8 101.6)
+		(at 52.07 63.5)
 		(size 50.8 25.4)
 		(exclude_from_sim no)
@@
 		)
 		(property "Sheetname" "WallPower"
-			(at 50.8 100.8884 0)
+			(at 52.07 62.7884 0)
 			(effects
 				(font
@@
 		)
 		(property "Sheetfile" "WallPower.kicad_sch"
-			(at 50.8 127.5846 0)
+			(at 52.07 89.4846 0)
 			(effects
 				(font
@@
 		)
 		(pin "-18V" output
-			(at 101.6 121.92 0)
+			(at 102.87 83.82 0)
 			(effects
 				(font
@@
 		)
 		(pin "18V" output
-			(at 101.6 106.68 0)
+			(at 102.87 68.58 0)
 			(effects
 				(font
@@
 	)
 	(sheet
-		(at 152.4 127)
-		(size 50.8 25.4)
-		(exclude_from_sim no)
-		(in_bom yes)
-		(on_board yes)
-		(dnp no)
-		(fields_autoplaced yes)
-		(stroke
-			(width 0.1524)
-			(type solid)
-		)
-		(fill
-			(color 0 0 0 0.0000)
-		)
-		(property "Sheetname" "HighVoltage2"
-			(at 152.4 126.2884 0)
-			(effects
-				(font
-					(size 1.27 1.27)
-				)
-				(justify left bottom)
-			)
-		)
-		(property "Sheetfile" "HighVoltagePair.kicad_sch"
-			(at 152.4 152.9846 0)
+		(at 53.34 127)
+		(size 48.26 25.4)
+		(exclude_from_sim no)
+		(in_bom yes)
+		(on_board yes)
+		(dnp no)
+		(fields_autoplaced yes)
+		(stroke
+			(width 0.1524)
+			(type solid)
+		)
+		(fill
+			(color 0 0 0 0.0000)
+		)
+		(property "Sheetname" "TIA2_Post"
+			(at 53.34 126.2884 0)
+			(effects
+				(font
+					(size 1.27 1.27)
+				)
+				(justify left bottom)
+			)
+		)
+		(property "Sheetfile" "TIA2_Post.kicad_sch"
+			(at 53.34 152.9846 0)
+			(effects
+				(font
+					(size 1.27 1.27)
+				)
+				(justify left top)
+			)
+		)
+		(instances
+			(project "PowerBoard"
+				(path "/c19e9b7b-7f36-470c-862a-1a648d3f14f6"
+					(page "6")
+				)
+			)
+		)
+	)
+	(sheet
+		(at 152.4 101.6)
+		(size 50.8 25.4)
+		(exclude_from_sim no)
+		(in_bom yes)
+		(on_board yes)
+		(dnp no)
+		(fields_autoplaced yes)
+		(stroke
+			(width 0.1524)
+			(type solid)
+		)
+		(fill
+			(color 0 0 0 0.0000)
+		)
+		(property "Sheetname" "PreAmp"
+			(at 152.4 100.8884 0)
+			(effects
+				(font
+					(size 1.27 1.27)
+				)
+				(justify left bottom)
+			)
+		)
+		(property "Sheetfile" "PreAmp.kicad_sch"
+			(at 152.4 127.5846 0)
 			(effects
 				(font
@@
 			(color 0 0 0 0.0000)
 		)
-		(property "Sheetname" "LowVoltage"
+		(property "Sheetname" "Converter"
 			(at 152.4 24.6884 0)
 			(effects
@@
 			)
 		)
-		(property "Sheetfile" "LowVoltage.kicad_sch"
+		(property "Sheetfile" "Converter.kicad_sch"
 			(at 152.4 51.3846 0)
 			(effects
@@
 			)
 		)
-		(pin "18V" input
-			(at 152.4 30.48 180)
-			(effects
-				(font
-					(size 1.27 1.27)
-				)
-				(justify left)
-			)
-		)

Commit message: Finished the sensors
Other:
- note added: "Input: 15V power Input: -15V power Input: pre voltage Input: AD8615 output Output: post voltage Ground receptacles(s) for preamp not yet elaborated All GND nodes for this board should connect to a hierarchical sheet pin instead of the regular GND symbol, in case we need to create separate GND planes for TIA2_Post and Power."
- note removed: "Input: 15V power Input: -15V power Input: pre voltage Input: AD8615 output Output: post voltage Ground receptacles(s) for preamp not yet elaborated"
Changed lines of the file:
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@@
 		)
 	)
-	(text "Input: 15V power\nInput: -15V power\nInput: pre voltage\nInput: AD8615 output\nOutput: post voltage\n\nGround receptacles(s) for\npreamp not yet elaborated"
+	(text "Input: 15V power\nInput: -15V power\nInput: pre voltage\nInput: AD8615 output\nOutput: post voltage\n\nGround receptacles(s) for\npreamp not yet elaborated\n\nAll GND nodes for this board\nshould connect to a hierarchical\nsheet pin instead of the regular GND\nsymbol, in case we need to\ncreate separate GND planes for\nTIA2_Post and Power."
 		(exclude_from_sim no)
 		(at 104.394 128.016 0)

Commit message: Save progress
Other:
- note added: "Input: 15V power Input: -15V power Input: pre voltage Input: AD8615 output Output: post voltage Ground receptacles(s) for preamp not yet elaborated All GND nodes for this section should connect to a hierarchical sheet pin instead of the regular GND symbol, in case we need to create separate GND planes for TIA2_Post and Power."
- note removed: "Input: 15V power Input: -15V power Input: pre voltage Input: AD8615 output Output: post voltage Ground receptacles(s) for preamp not yet elaborated All GND nodes for this board should connect to a hierarchical sheet pin instead of the regular GND symbol, in case we need to create separate GND planes for TIA2_Post and Power."
Changed lines of the file:
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@@
 		)
 	)
-	(text "Input: 15V power\nInput: -15V power\nInput: pre voltage\nInput: AD8615 output\nOutput: post voltage\n\nGround receptacles(s) for\npreamp not yet elaborated\n\nAll GND nodes for this board\nshould connect to a hierarchical\nsheet pin instead of the regular GND\nsymbol, in case we need to\ncreate separate GND planes for\nTIA2_Post and Power."
+	(text "Input: 15V power\nInput: -15V power\nInput: pre voltage\nInput: AD8615 output\nOutput: post voltage\n\nGround receptacles(s) for\npreamp not yet elaborated\n\nAll GND nodes for this section\nshould connect to a hierarchical\nsheet pin instead of the regular GND\nsymbol, in case we need to\ncreate separate GND planes for\nTIA2_Post and Power."
 		(exclude_from_sim no)
 		(at 104.394 128.016 0)

Commit message: Save progress
Other:
- removed sheet TIA2_Post
- note removed: "Input: 15V power Input: -15V power Input: pre voltage Input: AD8615 output Output: post voltage Ground receptacles(s) for preamp not yet elaborated All GND nodes for this section should connect to a hierarchical sheet pin instead of the regular GND symbol, in case we need to create separate GND planes for TIA2_Post and Power."
Changed lines of the file:
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@@
-		)
-	)
-	(text "Input: 15V power\nInput: -15V power\nInput: pre voltage\nInput: AD8615 output\nOutput: post voltage\n\nGround receptacles(s) for\npreamp not yet elaborated\n\nAll GND nodes for this section\nshould connect to a hierarchical\nsheet pin instead of the regular GND\nsymbol, in case we need to\ncreate separate GND planes for\nTIA2_Post and Power."
-		(exclude_from_sim no)
-		(at 104.394 128.016 0)
-		(effects
-			(font
-				(size 1.27 1.27)
-			)
-			(justify left top)
 		)
 	)
@@
 				)
 			)
-		)
-	)
-	(sheet
-		(at 53.34 127)
-		(size 48.26 25.4)
-		(exclude_from_sim no)
-		(in_bom yes)
-		(on_board yes)
-		(dnp no)
-		(fields_autoplaced yes)
-		(stroke
-			(width 0.1524)
-			(type solid)
-		)
-		(fill
-			(color 0 0 0 0.0000)
-		)
-		(property "Sheetname" "TIA2_Post"
-			(at 53.34 126.2884 0)
-			(effects
-				(font
-					(size 1.27 1.27)
-				)
-				(justify left bottom)
-			)
-		)
-		(property "Sheetfile" "TIA2_Post.kicad_sch"
-			(at 53.34 152.9846 0)
-			(effects
-				(font
-					(size 1.27 1.27)
-				)
-				(justify left top)
-			)
-		)
-		(instances
-			(project "PowerBoard"
-				(path "/c19e9b7b-7f36-470c-862a-1a648d3f14f6"
-					(page "6")
-				)
-			)

Commit message: Save progress
Other:
- sheet 15V ports: added -15V, -18V, 15V, 18V; removed none
- sheet Converter ports: added 18V, 3.3V, 5V; removed none
- sheet PreAmp ports: added -1.5V, -18V, 18V, 2.5V; removed none
- note removed: "Input: 18V power Input: -18V power Output: 15V power Output: -15V power"
- note removed: "Input: 18V power Input: -18V power Output: 2.5V power Output: -1.5V power"
- note removed: "Input: 18V power Output: 5V power Output: 3.3V power"

Commit message: Save progress
Other:
- note added: "Allocate 2 pins on a large pin socket for each of the following nodes, in case design revisions require more boards: - 18V - -18V - GND - 5V (converter) - 3.3V - GND - 5V (preamp) - -5V (preamp)"
Changed lines of the file:
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@@
 	(generator_version "9.0")
 	(paper "A4")
+	(text "Allocate 2 pins on a large pin socket for\neach of the following nodes, in case design\nrevisions require more boards:\n- 18V\n- -18V\n- GND\n- 5V (converter)\n- 3.3V\n- GND\n- 5V (preamp)\n- -5V (preamp)"
+		(exclude_from_sim no)
+		(at 51.054 26.67 0)
+		(effects
+			(font
+				(size 1.27 1.27)
+			)
+			(justify left top)
+		)
+	)
 	(junction
 		(at 142.24 83.82)
