File: Models/PowerBoard/15V.kicad_sch (KiCad schematic)
At the start: 2 parts, among them U1 LM7815, 15V, 5%, U3 LM7915, -15V, 5%

Commit message: Save progress
Parts:
- added C1: 220 nF, 0603, symbol Device:C
- added C2: 100 nF, 0603, symbol Device:C
- added C3, C4: 1 uF, 0603, symbol Device:C
- added D1, D2: D_Schottky, symbol Device:D_Schottky
Connections:
- net at U1.1 (IN): now also C1.1
- net GND: now reaches U1.2 (GND)
- net GND: now also U3.1 (GND), C1.2, C2.2, C3.2, C4.1, D1.2 (A), D2.1 (K)
- net at U1.3 (OUT): now also C2.1, D1.1 (K)
- net at U3.2 (IN): now also C3.1
- net at U3.3 (OUT): now also C4.2, D2.2 (A)

Commit message: Save progres
Parts:
- added D10, D8: 1N4007W, symbol Device:D
Connections:
- net 18V: now reaches C1.1, U1.1 (IN)
- net -15V: now reaches C4.2, D2.2 (A), U3.3 (OUT)
- net 15V: now reaches C2.1, D1.1 (K), U1.3 (OUT)
- net -18V: now reaches C3.1, U3.2 (IN)

Commit message: Save progress
Parts:
- removed D10: 1N4007W, symbol Device:D
- added D7: 1N4007W, symbol Device:D
- added NT1, NT10, NT2, NT9: NetTie_2, symbol Device:NetTie_2
Connections:
- net -15V: now also NT9.2; no longer C4.2, D2.2 (A), U3.3 (OUT)
- net -18V: now also NT10.2; no longer C3.1, U3.2 (IN)
- net 15V: now also NT1.2; no longer C2.1, D1.1 (K), U1.3 (OUT)
- net 18V: now also NT2.1; no longer C1.1, U1.1 (IN)
- net at D8.1 (K): now also C1.1, U1.1 (IN), NT2.2
- net at D8.2 (A): now also C2.1, D1.1 (K), U1.3 (OUT), NT1.1
- new net: C4.2, D2.2 (A), D7.1 (K), NT9.1, U3.3 (OUT)
- new net: C3.1, D7.2 (A), NT10.1, U3.2 (IN)
Other:
- moved on the sheet: C3, C4, D2

Commit message: Save progress
Parts:
- removed NT1, NT10, NT2, NT9: NetTie_2, symbol Device:NetTie_2
Connections:
- net -15V: now also C4.2, D2.2 (A), D7.1 (K), U3.3 (OUT)
- net -18V: now also C3.1, D7.2 (A), U3.2 (IN)
- net 15V: now also C2.1, D1.1 (K), D8.2 (A), U1.3 (OUT)
- net 18V: now also C1.1, D8.1 (K), U1.1 (IN)

Commit message: Passes ERC
Parts:
- renumbered C3 to C5, C2 to C7, D8 to D1, D7 to D4, D2 to D5, D1 to D7
Changed lines of the file:
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@@
 		(dnp no)
 		(fields_autoplaced yes)
-		(property "Reference" "#PWR02"
+		(property "Reference" "#PWR032"
 			(at 110.49 58.42 0)
 			(effects
@@
 			(project ""
 				(path "/c19e9b7b-7f36-470c-862a-1a648d3f14f6/018e7d12-6b24-44c3-9b74-64995b8fa179"
-					(reference "#PWR02")
+					(reference "#PWR032")
 					(unit 1)
 				)
@@
 		(dnp no)
 		(fields_autoplaced yes)
-		(property "Reference" "D1"
+		(property "Reference" "D7"
 			(at 139.7 65.7224 90)
 			(effects
@@
 			(project ""
 				(path "/c19e9b7b-7f36-470c-862a-1a648d3f14f6/018e7d12-6b24-44c3-9b74-64995b8fa179"
-					(reference "D1")
+					(reference "D7")
 					(unit 1)
 				)
@@
 		(dnp no)
 		(fields_autoplaced yes)
-		(property "Reference" "#PWR03"
+		(property "Reference" "#PWR029"
 			(at 62.23 132.08 0)
 			(effects
@@
 			(project "PowerBoard"
 				(path "/c19e9b7b-7f36-470c-862a-1a648d3f14f6/018e7d12-6b24-44c3-9b74-64995b8fa179"
-					(reference "#PWR03")
+					(reference "#PWR029")
 					(unit 1)
 				)
@@
 		(dnp no)
 		(fields_autoplaced yes)
-		(property "Reference" "D7"
+		(property "Reference" "D4"
 			(at 114.3 134.6199 90)
 			(effects
@@
 			(project "PowerBoard"
 				(path "/c19e9b7b-7f36-470c-862a-1a648d3f14f6/018e7d12-6b24-44c3-9b74-64995b8fa179"
-					(reference "D7")
+					(reference "D4")
 					(unit 1)
 				)
@@
 		(dnp no)
 		(fields_autoplaced yes)
-		(property "Reference" "#PWR016"
+		(property "Reference" "#PWR042"
 			(at 137.16 80.01 0)
 			(effects
@@
 			(project "PowerBoard"
 				(path "/c19e9b7b-7f36-470c-862a-1a648d3f14f6/018e7d12-6b24-44c3-9b74-64995b8fa179"
-					(reference "#PWR016")
+					(reference "#PWR042")
 					(unit 1)
 				)
@@
 		(dnp no)
 		(fields_autoplaced yes)
-		(property "Reference" "D2"
+		(property "Reference" "D5"
 			(at 132.08 116.5224 90)
 			(effects
@@
 			(project "PowerBoard"
 				(path "/c19e9b7b-7f36-470c-862a-1a648d3f14f6/018e7d12-6b24-44c3-9b74-64995b8fa179"
-					(reference "D2")
+					(reference "D5")
 					(unit 1)
 				)
@@
 		(dnp no)
 		(fields_autoplaced yes)
-		(property "Reference" "#PWR019"
+		(property "Reference" "#PWR035"
 			(at 106.68 161.29 0)
 			(effects
@@
 			(project "PowerBoard"
 				(path "/c19e9b7b-7f36-470c-862a-1a648d3f14f6/018e7d12-6b24-44c3-9b74-64995b8fa179"
-					(reference "#PWR019")
+					(reference "#PWR035")
 					(unit 1)
 				)
@@
 		(dnp no)
 		(fields_autoplaced yes)
-		(property "Reference" "#PWR018"
+		(property "Reference" "#PWR039"
 			(at 129.54 105.41 0)
 			(effects
@@
 			(project "PowerBoard"
 				(path "/c19e9b7b-7f36-470c-862a-1a648d3f14f6/018e7d12-6b24-44c3-9b74-64995b8fa179"
-					(reference "#PWR018")
+					(reference "#PWR039")
 					(unit 1)
 				)
@@
 		(dnp no)
 		(fields_autoplaced yes)
-		(property "Reference" "D8"
+		(property "Reference" "D1"
 			(at 86.36 31.75 0)
 			(effects
@@
 			(project ""
 				(path "/c19e9b7b-7f36-470c-862a-1a648d3f14f6/018e7d12-6b24-44c3-9b74-64995b8fa179"
-					(reference "D8")
+					(reference "D1")
 					(unit 1)
 				)
@@
 		(dnp no)
 		(fields_autoplaced yes)
-		(property "Reference" "#PWR014"
+		(property "Reference" "#PWR028"
 			(at 66.04 80.01 0)
 			(effects
@@
 			(project "PowerBoard"
 				(path "/c19e9b7b-7f36-470c-862a-1a648d3f14f6/018e7d12-6b24-44c3-9b74-64995b8fa179"
-					(reference "#PWR014")
+					(reference "#PWR028")
 					(unit 1)
 				)
@@
 		(dnp no)
 		(fields_autoplaced yes)
-		(property "Reference" "C3"
+		(property "Reference" "C5"
 			(at 110.49 147.3199 0)
 			(effects
@@
 			(project "PowerBoard"
 				(path "/c19e9b7b-7f36-470c-862a-1a648d3f14f6/018e7d12-6b24-44c3-9b74-64995b8fa179"
-					(reference "C3")
+					(reference "C5")
 					(unit 1)
 				)
@@
 		(dnp no)
 		(fields_autoplaced yes)
-		(property "Reference" "#PWR015"
+		(property "Reference" "#PWR038"
 			(at 114.3 80.01 0)
 			(effects
@@
 			(project "PowerBoard"
 				(path "/c19e9b7b-7f36-470c-862a-1a648d3f14f6/018e7d12-6b24-44c3-9b74-64995b8fa179"
-					(reference "#PWR015")
+					(reference "#PWR038")
 					(unit 1)
 				)
@@
 		(dnp no)
 		(fields_autoplaced yes)
-		(property "Reference" "C2"
+		(property "Reference" "C7"
 			(at 118.11 66.0399 0)
 			(effects
@@
 			(project "PowerBoard"
 				(path "/c19e9b7b-7f36-470c-862a-1a648d3f14f6/018e7d12-6b24-44c3-9b74-64995b8fa179"
-					(reference "C2")
+					(reference "C7")
 					(unit 1)
 				)
@@
 		(dnp no)
 		(fields_autoplaced yes)
-		(property "Reference" "#PWR017"
+		(property "Reference" "#PWR034"
 			(at 106.68 105.41 0)
 			(effects
@@
 			(project "PowerBoard"
 				(path "/c19e9b7b-7f36-470c-862a-1a648d3f14f6/018e7d12-6b24-44c3-9b74-64995b8fa179"
-					(reference "#PWR017")
-					(unit 1)
-				)
+					(reference "#PWR034")
+					(unit 1)
+				)

Commit message: Save progress
Parts:
- D1, D4: Cost (none) -> $0.059
Changed lines of the file:
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@@
+			)
+		)
+		(property "Cost" "$0.059"
+			(at 111.76 135.89 90)
+			(effects
+				(font
+					(size 1.27 1.27)
+				)
+				(hide yes)
 			)
 		)
@@
 			(at 86.36 38.1 0)
 			(effects
+				(font
+					(size 1.27 1.27)
+				)
+				(hide yes)
+			)
+		)
+		(property "Cost" "$0.059"
+			(at 86.36 38.1 0)
+			(effects

Commit message: Should be finished with components BOM
Parts:
- C1: Cost (none) -> $0.074; Purchase Link (none) -> https://www.digikey.com/en/products/detail/murata-electroni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
- C4, C5: Cost (none) -> $0.078; Purchase Link (none) -> https://www.digikey.com/en/products/detail/murata-electroni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
- C7: Cost (none) -> $0.079; Purchase Link (none) -> https://www.digikey.com/en/products/detail/murata-electroni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
- D5, D7: Cost (none) -> $0.166; Purchase Link (none) -> https://www.digikey.com/en/products/detail/diodes-incorpora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
- U1: Cost (none) -> $1.800; Purchase Link (none) -> https://www.digikey.com/en/products/detail/texas-instrument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
- U3: Cost (none) -> $1.480; Purchase Link (none) -> https://www.mouser.com/ProductDetail/Texas-Instruments/LM79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
Changed lines of the file:
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@@
+			)
+		)
+		(property "Cost" "$0.074"
+			(at 66.04 67.31 0)
+			(effects
+				(font
+					(size 1.27 1.27)
+				)
+				(hide yes)
+			)
+		)
+		(property "Purchase Link" "https://www.digikey.com/en/products/detail/murata-electronics/GRM188R71H224KAC4D/5797498"
+			(at 66.04 67.31 0)
+			(effects
+				(font
+					(size 1.27 1.27)
+				)
+				(hide yes)
 			)
 		)
@@
 			)
 		)
+		(property "Cost" "$0.078"
+			(at 106.68 118.11 0)
+			(effects
+				(font
+					(size 1.27 1.27)
+				)
+				(hide yes)
+			)
+		)
+		(property "Purchase Link" "https://www.digikey.com/en/products/detail/murata-electronics/GRT188R61H105KE13D/5416752"
+			(at 106.68 118.11 0)
+			(effects
+				(font
+					(size 1.27 1.27)
+				)
+				(hide yes)
+			)
+		)
 		(pin "1"
 		)
@@
 			)
 		)
-		(property "Purchase Link" ""
+		(property "Purchase Link" "https://www.digikey.com/en/products/detail/texas-instruments/LM7815CT-NOPB/3901976"
+			(at 68.58 55.88 0)
+			(effects
+				(font
+					(size 1.27 1.27)
+				)
+				(hide yes)
+			)
+		)
+		(property "Cost" "$1.800"
 			(at 68.58 55.88 0)
 			(effects
@@
 		)
 		(property "Description" ""
+			(at 68.58 132.08 0)
+			(effects
+				(font
+					(size 1.27 1.27)
+				)
+				(hide yes)
+			)
+		)
+		(property "Cost" "$1.480"
+			(at 68.58 132.08 0)
+			(effects
+				(font
+					(size 1.27 1.27)
+				)
+				(hide yes)
+			)
+		)
+		(property "Purchase Link" "https://www.mouser.com/ProductDetail/Texas-Instruments/LM7915CT-NOPB?qs=QbsRYf82W3F%252BRPQrGl%252ByOA%3D%3D"
 			(at 68.58 132.08 0)
 			(effects
@@
 			)
 		)
-		(property "Purchase Link" ""
+		(property "Purchase Link" "https://www.digikey.com/en/products/detail/diodes-incorporated/1N5819HW-7-F/814970"
 			(at 137.16 67.31 0)
+			(effects
+				(font
+					(size 1.27 1.27)
+				)
+				(hide yes)
+			)
+		)
+		(property "Cost" "$0.166"
+			(at 137.16 67.31 90)
 			(effects
 				(font
@@
 			)
 		)
-		(property "Purchase Link" ""
+		(property "Purchase Link" "https://www.digikey.com/en/products/detail/diodes-incorporated/1N5819HW-7-F/814970"
 			(at 129.54 118.11 0)
+			(effects
+				(font
+					(size 1.27 1.27)
+				)
+				(hide yes)
+			)
+		)
+		(property "Cost" "$0.166"
+			(at 129.54 118.11 90)
 			(effects
 				(font
@@
 			)
 		)
-		(property "Purchase Link" ""
+		(property "Purchase Link" "https://www.digikey.com/en/products/detail/murata-electronics/GRT188R61H105KE13D/5416752"
+			(at 106.68 148.59 0)
+			(effects
+				(font
+					(size 1.27 1.27)
+				)
+				(hide yes)
+			)
+		)
+		(property "Cost" "$0.078"
 			(at 106.68 148.59 0)
 			(effects
@@
 			(at 114.3 67.31 0)
 			(effects
+				(font
+					(size 1.27 1.27)
+				)
+				(hide yes)
+			)
+		)
+		(property "Cost" "$0.079"
+			(at 114.3 67.31 0)
+			(effects
+				(font
+					(size 1.27 1.27)
+				)
+				(hide yes)
+			)
+		)
+		(property "Purchase Link" "https://www.digikey.com/en/products/detail/murata-electronics/GRM188R72A104KA35D/702549"
+			(at 114.3 67.31 0)
+			(effects
