File: Models/PowerBoard/Converter.kicad_sch (KiCad schematic)
At the start: 2 parts, among them U5 LM7805, 5V, 5%, U6 TLV76133, 3.3V, 1%

Commit message: Save progress
Parts:
- added C11, C12: 1 uF, 0603, symbol Device:C
- added C7: 220 nF, 0603, symbol Device:C
- added C8: 100 nF, 0603, symbol Device:C
- added D4, D6: D_Schottky, symbol Device:D_Schottky
Connections:
- net GND: now reaches U6.1 (GND)
- net GND: now also U5.2 (GND), C11.2, C12.2, C7.2, C8.2, D4.2 (A), D6.2 (A)
- net at U6.3 (IN): now also C11.1
- net at U6.4 (OUT): now also C12.1, D6.1 (K)
- net at U5.1 (IN): now also C7.1
- net at U5.3 (OUT): now also C8.1, D4.1 (K)
- no-connect marks 0 -> 1

Commit message: Save progres
Parts:
- added D11: 1N4007W, symbol Device:D
- added D9: D_Schottky, symbol Device:D_Schottky
Connections:
- net 5V: now reaches C8.1, D4.1 (K), U5.3 (OUT)
- net 5V: now also C11.1, U6.3 (IN)
- net 3.3V: now reaches C12.1, D6.1 (K), U6.4 (OUT)
- net 18V: now reaches C7.1, U5.1 (IN)

Commit message: Save progress
Parts:
- added NT5, NT6, NT7, NT8: NetTie_2, symbol Device:NetTie_2
Connections:
- net 18V: now also NT6.1; no longer C7.1, U5.1 (IN)
- net 3.3V: now also NT8.2; no longer C12.1, D6.1 (K), U6.4 (OUT)
- net 5V: now also NT5.2, NT7.1; no longer C11.1, C8.1, D4.1 (K), U5.3 (OUT), U6.3 (IN)
- net at D9.1 (K): now also C11.1, U6.3 (IN), NT7.2
- net at D9.2 (A): now also C12.1, D6.1 (K), U6.4 (OUT), NT8.1
- net at D11.1 (K): now also C7.1, U5.1 (IN), NT6.2
- net at D11.2 (A): now also C8.1, D4.1 (K), U5.3 (OUT), NT5.1

Commit message: Save progress
Parts:
- removed NT5, NT6, NT7, NT8: NetTie_2, symbol Device:NetTie_2
Connections:
- net 18V: now also C7.1, D11.1 (K), U5.1 (IN)
- net 3.3V: now also C12.1, D6.1 (K), D9.2 (A), U6.4 (OUT)
- net 5V: now also C11.1, C8.1, D11.2 (A), D4.1 (K), D9.1 (K), U5.3 (OUT), U6.3 (IN)

Commit message: Passes ERC
Parts:
- renumbered C7 to C2, C11 to C3, C12 to C6, D11 to D2, D9 to D3, D4 to D8, U5 to U2, U6 to U4
Changed lines of the file:
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@@
 		(dnp no)
 		(fields_autoplaced yes)
-		(property "Reference" "#PWR07"
+		(property "Reference" "#PWR031"
 			(at 107.95 137.16 0)
 			(effects
@@
 			(project "PowerBoard"
 				(path "/c19e9b7b-7f36-470c-862a-1a648d3f14f6/df1ba0e1-55fc-41f2-80f9-aaa8393d43d6"
-					(reference "#PWR07")
+					(reference "#PWR031")
 					(unit 1)
 				)
@@
 		(dnp no)
 		(fields_autoplaced yes)
-		(property "Reference" "#PWR06"
+		(property "Reference" "#PWR033"
 			(at 110.49 58.42 0)
 			(effects
@@
 			(project "PowerBoard"
 				(path "/c19e9b7b-7f36-470c-862a-1a648d3f14f6/df1ba0e1-55fc-41f2-80f9-aaa8393d43d6"
-					(reference "#PWR06")
+					(reference "#PWR033")
 					(unit 1)
 				)
@@
 		(dnp no)
 		(fields_autoplaced yes)
-		(property "Reference" "#PWR025"
+		(property "Reference" "#PWR030"
 			(at 68.58 156.21 0)
 			(effects
@@
 			(project "PowerBoard"
 				(path "/c19e9b7b-7f36-470c-862a-1a648d3f14f6/df1ba0e1-55fc-41f2-80f9-aaa8393d43d6"
-					(reference "#PWR025")
+					(reference "#PWR030")
 					(unit 1)
 				)
@@
 		(dnp no)
 		(fields_autoplaced yes)
-		(property "Reference" "#PWR020"
+		(property "Reference" "#PWR027"
 			(at 66.04 80.01 0)
 			(effects
@@
 			(project "PowerBoard"
 				(path "/c19e9b7b-7f36-470c-862a-1a648d3f14f6/df1ba0e1-55fc-41f2-80f9-aaa8393d43d6"
-					(reference "#PWR020")
+					(reference "#PWR027")
 					(unit 1)
 				)
@@
 		(dnp no)
 		(fields_autoplaced yes)
-		(property "Reference" "#PWR024"
+		(property "Reference" "#PWR036"
 			(at 111.76 156.21 0)
 			(effects
@@
 			(project "PowerBoard"
 				(path "/c19e9b7b-7f36-470c-862a-1a648d3f14f6/df1ba0e1-55fc-41f2-80f9-aaa8393d43d6"
-					(reference "#PWR024")
+					(reference "#PWR036")
 					(unit 1)
 				)
@@
 		(dnp no)
 		(fields_autoplaced yes)
-		(property "Reference" "#PWR022"
+		(property "Reference" "#PWR041"
 			(at 137.16 80.01 0)
 			(effects
@@
 			(project "PowerBoard"
 				(path "/c19e9b7b-7f36-470c-862a-1a648d3f14f6/df1ba0e1-55fc-41f2-80f9-aaa8393d43d6"
-					(reference "#PWR022")
+					(reference "#PWR041")
 					(unit 1)
 				)
@@
 		(dnp no)
 		(fields_autoplaced yes)
-		(property "Reference" "#PWR021"
+		(property "Reference" "#PWR037"
 			(at 114.3 80.01 0)
 			(effects
@@
 			(project "PowerBoard"
 				(path "/c19e9b7b-7f36-470c-862a-1a648d3f14f6/df1ba0e1-55fc-41f2-80f9-aaa8393d43d6"
-					(reference "#PWR021")
+					(reference "#PWR037")
 					(unit 1)
 				)
@@
 		(dnp no)
 		(fields_autoplaced yes)
-		(property "Reference" "D4"
+		(property "Reference" "D8"
 			(at 139.7 65.7224 90)
 			(effects
@@
 			(project "PowerBoard"
 				(path "/c19e9b7b-7f36-470c-862a-1a648d3f14f6/df1ba0e1-55fc-41f2-80f9-aaa8393d43d6"
-					(reference "D4")
+					(reference "D8")
 					(unit 1)
 				)
@@
 		(dnp no)
 		(fields_autoplaced yes)
-		(property "Reference" "C12"
+		(property "Reference" "C6"
 			(at 115.57 142.2399 0)
 			(effects
@@
 			(project "PowerBoard"
 				(path "/c19e9b7b-7f36-470c-862a-1a648d3f14f6/df1ba0e1-55fc-41f2-80f9-aaa8393d43d6"
-					(reference "C12")
+					(reference "C6")
 					(unit 1)
 				)
@@
 		(dnp no)
 		(fields_autoplaced yes)
-		(property "Reference" "D9"
+		(property "Reference" "D3"
 			(at 86.0425 107.95 0)
 			(effects
@@
 			(project "PowerBoard"
 				(path "/c19e9b7b-7f36-470c-862a-1a648d3f14f6/df1ba0e1-55fc-41f2-80f9-aaa8393d43d6"
-					(reference "D9")
+					(reference "D3")
 					(unit 1)
 				)
@@
 		(dnp no)
 		(fields_autoplaced yes)
-		(property "Reference" "U6"
+		(property "Reference" "U4"
 			(at 86.36 121.92 0)
 			(effects
@@
 			(project "PowerBoard"
 				(path "/c19e9b7b-7f36-470c-862a-1a648d3f14f6/df1ba0e1-55fc-41f2-80f9-aaa8393d43d6"
-					(reference "U6")
+					(reference "U4")
 					(unit 1)
 				)
@@
 		(dnp no)
 		(fields_autoplaced yes)
-		(property "Reference" "U5"
+		(property "Reference" "U2"
 			(at 86.36 45.72 0)
 			(effects
@@
 			(project "PowerBoard"
 				(path "/c19e9b7b-7f36-470c-862a-1a648d3f14f6/df1ba0e1-55fc-41f2-80f9-aaa8393d43d6"
-					(reference "U5")
+					(reference "U2")
 					(unit 1)
 				)
@@
 		(dnp no)
 		(fields_autoplaced yes)
-		(property "Reference" "#PWR023"
+		(property "Reference" "#PWR040"
 			(at 132.08 156.21 0)
 			(effects
@@
 			(project "PowerBoard"
 				(path "/c19e9b7b-7f36-470c-862a-1a648d3f14f6/df1ba0e1-55fc-41f2-80f9-aaa8393d43d6"
-					(reference "#PWR023")
+					(reference "#PWR040")
 					(unit 1)
 				)
@@
 		(dnp no)
 		(fields_autoplaced yes)
-		(property "Reference" "C11"
+		(property "Reference" "C3"
 			(at 72.39 142.2399 0)
 			(effects
@@
 			(project "PowerBoard"
 				(path "/c19e9b7b-7f36-470c-862a-1a648d3f14f6/df1ba0e1-55fc-41f2-80f9-aaa8393d43d6"
-					(reference "C11")
+					(reference "C3")
 					(unit 1)
 				)
@@
 		(dnp no)
 		(fields_autoplaced yes)
-		(property "Reference" "C7"
+		(property "Reference" "C2"
 			(at 69.85 66.0399 0)
 			(effects
@@
 			(project "PowerBoard"
 				(path "/c19e9b7b-7f36-470c-862a-1a648d3f14f6/df1ba0e1-55fc-41f2-80f9-aaa8393d43d6"
-					(reference "C7")
+					(reference "C2")
 					(unit 1)
 				)
@@
 		(dnp no)
 		(fields_autoplaced yes)
-		(property "Reference" "D11"
+		(property "Reference" "D2"
 			(at 86.36 31.75 0)
 			(effects
@@
 			(project "PowerBoard"
 				(path "/c19e9b7b-7f36-470c-862a-1a648d3f14f6/df1ba0e1-55fc-41f2-80f9-aaa8393d43d6"
-					(reference "D11")
-					(unit 1)
-				)
+					(reference "D2")
+					(unit 1)
+				)

Commit message: Save progress
Parts:
- D2: Cost (none) -> $0.059
Changed lines of the file:
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@@
+			)
+		)
+		(property "Cost" "$0.059"
+			(at 86.36 38.1 0)
+			(effects
+				(font
+					(size 1.27 1.27)
+				)
+				(hide yes)
 			)
 		)

Commit message: Should be finished with components BOM
Parts:
- C2: Cost (none) -> $0.074; Purchase Link (none) -> https://www.digikey.com/en/products/detail/murata-electroni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
- C3, C6: Cost (none) -> $0.078; Purchase Link (none) -> https://www.digikey.com/en/products/detail/murata-electroni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
- C8: Cost (none) -> $0.079; Purchase Link (none) -> https://www.digikey.com/en/products/detail/murata-electroni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
- D3, D6, D8: Cost (none) -> $0.166; Purchase Link (none) -> https://www.digikey.com/en/products/detail/diodes-incorpora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
- U2: Cost (none) -> $1.800; Purchase Link (none) -> https://www.digikey.com/en/products/detail/texas-instrument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
- U4: Cost (none) -> $0.480; Purchase Link (none) -> https://www.digikey.com/en/products/detail/texas-instrument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
Changed lines of the file:
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@@
 			)
 		)
-		(property "Purchase Link" ""
+		(property "Purchase Link" "https://www.digikey.com/en/products/detail/diodes-incorporated/1N5819HW-7-F/814970"
 			(at 137.16 67.31 0)
+			(effects
+				(font
+					(size 1.27 1.27)
+				)
+				(hide yes)
+			)
+		)
+		(property "Cost" "$0.166"
+			(at 137.16 67.31 90)
 			(effects
 				(font
@@
 			)
 		)
+		(property "Cost" "$0.078"
+			(at 111.76 143.51 0)
+			(effects
+				(font
+					(size 1.27 1.27)
+				)
+				(hide yes)
+			)
+		)
+		(property "Purchase Link" "https://www.digikey.com/en/products/detail/murata-electronics/GRT188R61H105KE13D/5416752"
+			(at 111.76 143.51 0)
+			(effects
+				(font
+					(size 1.27 1.27)
+				)
+				(hide yes)
+			)
+		)
 		(pin "1"
 		)
@@
 			)
 		)
-		(property "Purchase Link" ""
+		(property "Purchase Link" "https://www.digikey.com/en/products/detail/diodes-incorporated/1N5819HW-7-F/814970"
+			(at 86.36 114.3 0)
+			(effects
+				(font
+					(size 1.27 1.27)
+				)
+				(hide yes)
+			)
+		)
+		(property "Cost" "$0.166"
 			(at 86.36 114.3 0)
 			(effects
@@
 			)
 		)
+		(property "Cost" "$0.480"
+			(at 71.12 129.54 0)
+			(effects
+				(font
+					(size 1.27 1.27)
+				)
+				(hide yes)
+			)
+		)
+		(property "Purchase Link" "https://www.digikey.com/en/products/detail/texas-instruments/TLV76133DCYR/18716472"
+			(at 71.12 129.54 0)
+			(effects
+				(font
+					(size 1.27 1.27)
+				)
+				(hide yes)
+			)
+		)
 		(pin "3"
 		)
@@
 			)
 		)
+		(property "Cost" "$1.800"
+			(at 68.58 55.88 0)
+			(effects
+				(font
+					(size 1.27 1.27)
+				)
+				(hide yes)
+			)
+		)
+		(property "Purchase Link" "https://www.digikey.com/en/products/detail/texas-instruments/LM7805CT-NOPB/3901929"
+			(at 68.58 55.88 0)
+			(effects
+				(font
+					(size 1.27 1.27)
+				)
+				(hide yes)
+			)
+		)
 		(pin "1"
 		)
@@
 			)
 		)
+		(property "Cost" "$0.078"
+			(at 68.58 143.51 0)
+			(effects
+				(font
+					(size 1.27 1.27)
+				)
+				(hide yes)
+			)
+		)
+		(property "Purchase Link" "https://www.digikey.com/en/products/detail/murata-electronics/GRT188R61H105KE13D/5416752"
+			(at 68.58 143.51 0)
+			(effects
+				(font
+					(size 1.27 1.27)
+				)
+				(hide yes)
+			)
+		)
 		(pin "1"
 		)
@@
 			)
 		)
-		(property "Purchase Link" ""
+		(property "Purchase Link" "https://www.digikey.com/en/products/detail/diodes-incorporated/1N5819HW-7-F/814970"
 			(at 132.08 143.51 0)
+			(effects
+				(font
+					(size 1.27 1.27)
+				)
+				(hide yes)
+			)
+		)
+		(property "Cost" "$0.166"
+			(at 132.08 143.51 90)
 			(effects
 				(font
@@
 			)
 		)
+		(property "Cost" "$0.074"
+			(at 66.04 67.31 0)
+			(effects
+				(font
+					(size 1.27 1.27)
+				)
+				(hide yes)
+			)
+		)
+		(property "Purchase Link" "https://www.digikey.com/en/products/detail/murata-electronics/GRM188R71H224KAC4D/5797498"
+			(at 66.04 67.31 0)
+			(effects
+				(font
+					(size 1.27 1.27)
+				)
+				(hide yes)
+			)
+		)
 		(pin "1"
 		)
@@
 			(at 114.3 67.31 0)
 			(effects
+				(font
+					(size 1.27 1.27)
+				)
+				(hide yes)
+			)
+		)
+		(property "Cost" "$0.079"
+			(at 114.3 67.31 0)
+			(effects
+				(font
+					(size 1.27 1.27)
+				)
+				(hide yes)
+			)
+		)
+		(property "Purchase Link" "https://www.digikey.com/en/products/detail/murata-electronics/GRM188R72A104KA35D/702549"
+			(at 114.3 67.31 0)
+			(effects
