File: Models/PowerBoard/PowerBoard.kicad_pcb (KiCad board)
At the start: 2 copper layers, 0 parts

Commit message: Push uncommitted changes
Parts:
- added C1: 220 nF, 0603, TwoTerminal:CAPC0603, F.Cu at (162.6, 74.2)
- added C10: 1 uF, 0603, TwoTerminal:CAPC0603, F.Cu at (145.2, 124.0)
- added C11: 1 uF, 0603, TwoTerminal:CAPC0603, F.Cu at (145.2, 126.6)
- added C12: 100 nF, 0603, TwoTerminal:CAPC0603, F.Cu at (145.2, 129.2)
- added C13: 10 uF, 0805, TwoTerminal:CAPC0805, F.Cu at (149.8, 121.6)
- added C14: 10 uF, 0805, TwoTerminal:CAPC0805, F.Cu at (149.8, 124.7)
- added C2: 220 nF, 0603, TwoTerminal:CAPC0603, F.Cu at (102.2, 124.5)
- added C3: 1 uF, 0603, TwoTerminal:CAPC0603, F.Cu at (102.2, 127.2)
- added C4: 1 uF, 0603, TwoTerminal:CAPC0603, F.Cu at (162.6, 76.8)
- added C5: 1 uF, 0603, TwoTerminal:CAPC0603, F.Cu at (162.6, 79.5)
- added C6: 1 uF, 0603, TwoTerminal:CAPC0603, F.Cu at (102.2, 129.8)
- added C7: 100 nF, 0603, TwoTerminal:CAPC0603, F.Cu at (162.6, 82.1)
- added C8: 100 nF, 0603, TwoTerminal:CAPC0603, F.Cu at (102.2, 132.4)
- added C9: 220 nF, 0603, TwoTerminal:CAPC0603, F.Cu at (145.2, 121.4)
- added D1: 1N4007W, TwoTerminal:SOD-123FL, F.Cu at (163.7, 85.2)
- added D10: 1N4007W, TwoTerminal:SOD-123FL, F.Cu at (145.7, 111.2)
- added D11: D_Schottky, TwoTerminal:SOD-123, F.Cu at (145.7, 114.5)
- added D12: D_Schottky, TwoTerminal:SOD-123, F.Cu at (145.7, 117.8)
- added D2: 1N4007W, TwoTerminal:SOD-123FL, F.Cu at (115.8, 117.9)
- added D3: D_Schottky, TwoTerminal:SOD-123, F.Cu at (117.7, 124.8)
- added D4: 1N4007W, TwoTerminal:SOD-123FL, F.Cu at (163.7, 88.7)
- added D5: D_Schottky, TwoTerminal:SOD-123, F.Cu at (151.2, 88.7)
- added D6: D_Schottky, TwoTerminal:SOD-123, F.Cu at (117.7, 128.1)
- added D7: D_Schottky, TwoTerminal:SOD-123, F.Cu at (151.2, 91.9)
- added D8: D_Schottky, TwoTerminal:SOD-123, F.Cu at (117.7, 131.3)
- added D9: 1N4007W, TwoTerminal:SOD-123FL, F.Cu at (145.7, 107.7)
- added H1: Mounting Hole, M2.5, Connector_Custom:Keystone_24929, F.Cu at (133.8, 76.8)
- added H2: Mounting Hole, M2.5, Connector_Custom:Keystone_24929, F.Cu at (133.8, 84.5)
- added H3: Dowel Pin, M2.5, Connector_Custom:DowelPin_2.5mm, F.Cu at (144.1, 74.7)
- added H4: Mounting Hole, M2.5, Connector_Custom:Keystone_24929, F.Cu at (133.8, 92.3)
- added H5: Mounting Hole, M2.5, Connector_Custom:Keystone_24929, F.Cu at (133.8, 100.0)
- added H6: Dowel Pin, M2.5, Connector_Custom:DowelPin_2.5mm, F.Cu at (144.1, 78.3)
- added J11: Conn_01x09_Socket, Connector_Custom:PinConnector_1x9, F.Cu at (140.0, 85.5)
- added J12: Banana Socket, Green, Connector_Custom:Multicomp_24.243, F.Cu at (113.9, 79.8)
- added J13: Banana Socket, Black, Connector_Custom:Multicomp_24.243, F.Cu at (113.9, 93.5)
- added J14: Banana Socket, Blue, Connector_Custom:Multicomp_24.243, F.Cu at (113.9, 107.3)
- added RV1: 1k, 10%, ThreeTerminal:Bourns_3296Y, F.Cu at (133.2, 125.7)
- added RV2: 1k, 10%, ThreeTerminal:Bourns_3296Y, F.Cu at (139.7, 125.7)
- added U1: LM7815, 15V, 5%, ThreeTerminal:TO-220, F.Cu at (154.1, 77.0)
- added U2: LM7805, 5V, 5%, ThreeTerminal:TO-220, F.Cu at (106.2, 120.2)
- added U3: LM7915, -15V, 5%, ThreeTerminal:TO-220, F.Cu at (154.1, 84.0)
- added U4: TLV76133, 3.3V, 1%, ThreeTerminal:SOT-223, F.Cu at (109.4, 127.3)
- added U5: LM7805, 5V, 5%, ThreeTerminal:TO-220, F.Cu at (136.2, 110.0)
- added U6: LM7905, -5V, 5%, ThreeTerminal:TO-220, F.Cu at (136.2, 117.0)
