File: Models/PowerBoard/WallPower.kicad_sch (KiCad schematic)
At the start: 4 parts, among them J12 Banana Socket, Green, J13 Banana Socket, Black, J14 Banana Socket, Blue

Commit message: Finished layout of power board
Parts:
- J12: value Banana Socket, Green -> Banana Socket, Red; Purchase Link https://www.newark.com/multicomp/24-243-4/banana-jack-4mm-2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 -> https://www.newark.com/multicomp/24-243-1/pcb-socket-4mm-re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
- J14: value Banana Socket, Blue -> Banana Socket, Yellow; Purchase Link https://www.newark.com/multicomp/24-243-5/test-socket-32a-p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 -> https://www.newark.com/multicomp/24-243-3/test-socket-pcb-4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
Changed lines of the file:
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@@
 			)
 		)
-		(property "Value" "Banana Socket, Blue"
+		(property "Value" "Banana Socket, Yellow"
 			(at 168.91 98.4249 90)
 			(effects
@@
 			)
 		)
-		(property "Purchase Link" "https://www.newark.com/multicomp/24-243-5/test-socket-32a-panel-blue/dp/80P3614"
+		(property "Purchase Link" "https://www.newark.com/multicomp/24-243-3/test-socket-pcb-4mm-yellow/dp/80P3617"
 			(at 165.1 96.52 0)
 			(effects
@@
 			)
 		)
-		(property "Value" "Banana Socket, Green"
+		(property "Value" "Banana Socket, Red"
 			(at 168.91 73.0249 90)
 			(effects
@@
 			)
 		)
-		(property "Purchase Link" "https://www.newark.com/multicomp/24-243-4/banana-jack-4mm-24a-th-green/dp/80P3615"
+		(property "Purchase Link" "https://www.newark.com/multicomp/24-243-1/pcb-socket-4mm-red/dp/80P3616"
 			(at 165.1 71.12 0)
 			(effects
