File: Models/TIA2_Post/TIA2_Post.kicad_sch (KiCad schematic)
At the start: 0 parts

Commit message: Save progress
Other:
- note added: "Input: 15V power Input: -15V power Input: pre voltage Output: 2.5V power Output: -1.5V power Output: post voltage Ground connection(s) not yet elaborated"
- note removed: "Input: 15V power Input: -15V power Input: pre voltage (grounded interconnect) Output: 2.5V power (grounded interconnect) Output: -1.5V power (grounded interconnect) Output: post voltage"
Changed lines of the file:
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@@
 	(generator_version "9.0")
 	(paper "A4")
-	(text "Input: 15V power\nInput: -15V power\nInput: pre voltage (grounded interconnect)\nOutput: 2.5V power (grounded interconnect)\nOutput: -1.5V power (grounded interconnect)\nOutput: post voltage"
+	(text "Input: 15V power\nInput: -15V power\nInput: pre voltage\n\nOutput: 2.5V power\nOutput: -1.5V power\nOutput: post voltage\n\nGround connection(s) not yet elaborated"
 		(exclude_from_sim no)
 		(at 158.242 76.962 0)
