File: Models/TIA2_Post/TIA2_Post.kicad_pcb (KiCad board)
At the start: 2 copper layers, 0 parts

Commit message: First time that all PCBs are fully wired
Parts:
- added C1: 100 nF, 0603, TwoTerminal:CAPC0603, F.Cu at (103.7, 96.9)
- added C2: 100 nF, 0603, TwoTerminal:CAPC0603, F.Cu at (99.9, 104.7)
- added C3: 2 nF, 1%, TwoTerminal:CAPC0603, F.Cu at (98.5, 85.1)
- added D1: 1N4448W, TwoTerminal:SOD-123, F.Cu at (114.3, 101.6)
- added D2: 1N4448W, TwoTerminal:SOD-123, F.Cu at (114.3, 104.2)
- added D3: 1N4448W, TwoTerminal:SOD-123, F.Cu at (122.4, 83.2)
- added D4: 1N4448W, TwoTerminal:SOD-123, F.Cu at (122.4, 94.6)
- added D5: 10V, 1%, ThreeTerminal:SOT-23, F.Cu at (128.0, 86.8)
- added D6: 10V, 1%, ThreeTerminal:SOT-23, F.Cu at (128.0, 91.0)
- added H1: MountingHole, Connector_Custom:DowelPin_2.5mm, F.Cu at (130.8, 101.6)
- added H2: MountingHole, Connector_Custom:DowelPin_2.5mm, F.Cu at (125.7, 104.9)
- added J1: Conn_01x03_Pin, Connector_Custom:PinHeader_1x3, F.Cu at (134.6, 85.1)
- added J2: Conn_01x03_Socket, Connector_Custom:PinSocket_1x3, F.Cu at (99.1, 92.7)
- added J3: Conn_01x06_Socket, Connector_Custom:PinSocket_1x6, F.Cu at (134.6, 99.1)
- added J4: Conn_01x02_Pin, Connector_Custom:PinHeader_1x2, F.Cu at (109.2, 99.1)
- added J5: Conn_01x02_Pin, Connector_Custom:PinHeader_1x2, F.Cu at (116.8, 88.9)
- added Q1: Q_PNP_BEC, ThreeTerminal:SOT-23, F.Cu at (122.4, 86.8)
- added Q2: Q_NPN_BEC, ThreeTerminal:SOT-23, F.Cu at (122.4, 91.0)
- added R1: 10, 1%, TwoTerminal:RESC0603, F.Cu at (131.5, 83.1)
- added R10: 10k, 1%, TwoTerminal:RESC0603, F.Cu at (128.0, 94.6)
- added R2: 1k, 1%, TwoTerminal:RESC0603, F.Cu at (103.9, 104.7)
- added R3: 24k, 1%, TwoTerminal:RESC0603, F.Cu at (107.9, 104.7)
- added R4: 1.3k, 1%, TwoTerminal:RESC0603, F.Cu at (100.6, 85.1)
- added R5: 240k, 1%, TwoTerminal:RESC0603, F.Cu at (114.3, 99.2)
- added R6: 10k, 1%, TwoTerminal:RESC0603, F.Cu at (118.1, 99.2)
- added R7: 1k, 1%, TwoTerminal:RESC0603, F.Cu at (116.8, 84.0)
- added R8: 1k, 1%, TwoTerminal:RESC0603, F.Cu at (116.8, 93.6)
- added R9: 10k, 1%, TwoTerminal:RESC0603, F.Cu at (128.0, 83.2)
- added RV1: 10k, 10%, ThreeTerminal:Bourns_3296Y, F.Cu at (104.9, 86.4)
- added RV2: 200k, 10%, ThreeTerminal:Bourns_3296Y, F.Cu at (111.2, 86.4)
- added U1: OP37G, IC:SOIC-8, F.Cu at (102.2, 100.7)
Routing:
- net GND: track 0.00 -> 79.1 mm, vias 0 -> 1
- net 15V: track 0.00 -> 75.1 mm, vias 0 -> 1
- net /PostVoltage: track 0.00 -> 50.9 mm, vias 0 -> 6
- net -15V: track 0.00 -> 50.6 mm
- net Net-(D1-K): track 0.00 -> 17.2 mm
- net /PreVoltage: track 0.00 -> 15.8 mm
- net /Amplifier/InvertingInput: track 0.00 -> 15.2 mm, vias 0 -> 2
- net Net-(D6-*): track 0.00 -> 11.9 mm
- net /Limiter/Clamped_Output: track 0.00 -> 11.4 mm
- net /AD8615_Output: track 0.00 -> 10.1 mm
- net Net-(D5-K): track 0.00 -> 8.34 mm
- net Net-(D1-A): track 0.00 -> 7.74 mm
- net Net-(D3-K): track 0.00 -> 7.60 mm
- net Net-(R4-Pad2): track 0.00 -> 4.24 mm
- net Net-(D4-A): track 0.00 -> 3.96 mm
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- added copper zone on B.Cu, net /PostVoltage
- added copper zone on B.Cu, net ISO_GND
Other:
- board outline added: 39.3 x 26.9 mm
- board text added: "25x"
