File: Models/HighVoltageBoard/WallPower.kicad_sch (KiCad schematic)
At the start: 0 parts

Commit message: Save progress
Parts:
- added BT1, BT2: R4G650-0.1, symbol Custom:R4G650-0.1
Connections:
- new net -450V: BT2.3 (V-)
- new net 450V: BT1.1 (V+)
- new net GND: BT1.2 (GND), BT1.3 (V-), BT2.1 (V+), BT2.2 (GND)

Commit message: Save progress
Parts:
- added D1, D2: Vr = 1.3 kV, symbol Device:D
Connections:
- net -450V: now also D2.2 (A); no longer BT2.3 (V-)
- net 450V: now also D1.1 (K); no longer BT1.1 (V+)
- no-connect marks 0 -> 4
Other:
- note added: "power cord receptacle type not known yet"

Commit message: Save progress
Parts:
- D1, D2: value Vr = 1.3 kV -> Vr = 2 kV
Connections:
- net GND: no longer BT1.2 (GND), BT1.3 (V-), BT2.1 (V+), BT2.2 (GND)
- new net: BT1.2 (GND), BT1.3 (V-), BT2.1 (V+), BT2.2 (GND)
- no-connect marks 4 -> 6

Commit message: Save progress
Parts:
- D1, D2: Purchase Link (none) -> https://www.digikey.com/en/products/detail/taiwan-semicondu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
Changed lines of the file:
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@@
 			)
 		)
-		(property "Purchase Link" ""
+		(property "Purchase Link" "https://www.digikey.com/en/products/detail/taiwan-semiconductor-corporation/GS1Z/28023582"
 			(at 158.75 109.22 0)
 			(effects
@@
 			)
 		)
-		(property "Purchase Link" ""
+		(property "Purchase Link" "https://www.digikey.com/en/products/detail/taiwan-semiconductor-corporation/GS1Z/28023582"
 			(at 158.75 78.74 0)
 			(effects

Commit message: Save progress
Parts:
- added D7, D8: Vr = 451V, symbol Device:D_Zener
Connections:
- net -450V: now also D8.2 (A)
- net 450V: now also D7.1 (K)
- net GND: now also D7.2 (A), D8.1 (K)

Commit message: Save progress
Connections:
- net -450V_PreDiode: now reaches D2.1 (K)
- net 450V_PreDiode: now reaches D1.2 (A)
Other:
- moved on the sheet: D1, D2, D7, D8

Commit message: Save progress
Connections:
- net -450V renamed V-
- net 450V renamed V+
Changed lines of the file:
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@@
 		)
 	)
-	(hierarchical_label "450V"
+	(hierarchical_label "V+"
 		(shape output)
 		(at 182.88 78.74 0)
@@
 		)
 	)
-	(hierarchical_label "-450V"
+	(hierarchical_label "V-"
 		(shape output)
 		(at 182.88 109.22 0)

Commit message: Save progress
Parts:
- added R13, R14: 1M, 5%, 0.33W, 800V, symbol Device:R_US
Connections:
- net GND: now also R13.2, R14.1
- net V+: now also R13.1
- net V-: now also R14.2
