File: Models/HighVoltageBoard/WallPower.kicad_sch (KiCad schematic)
At the start: 8 parts

Commit message: Save progress
Parts:
- added J1: Conn_01x02_Socket, symbol Connector:Conn_01x02_Socket
Connections:
- net -450V_PreDiode: no longer D2.1 (K)
- net 450V_PreDiode: no longer D1.2 (A)
- now unconnected: BT1.2 (GND), BT1.3 (V-), BT2.1 (V+), BT2.2 (GND)
- no-connect marks 6 -> 0
Other:
- note added: "power cord receptacle type: banana socket WARNING: connection is high voltage, but not CAT III rated"
- note removed: "power cord receptacle type not known yet"
- moved on the sheet: BT1, BT2

Commit message: Save progress
Parts:
- added J2: Banana Socket, Yellow, symbol Connector:Conn_01x02_Socket
- added J3: Banana Socket, Black, symbol Connector:Conn_01x02_Socket
- BT1, BT2: now left out of the parts list
- J1: value Conn_01x02_Socket -> Banana Socket, Red; Cost (none) -> $1.490; Purchase Link (none) -> https://www.newark.com/multicomp/24-243-1/pcb-socket-4mm-re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
Connections:
- net -450V_PreDiode: now also D2.1 (K), J2.1 (Pin_1), J2.2 (Pin_2)
- net 450V_PreDiode: now also D1.2 (A), J1.1 (Pin_1), J1.2 (Pin_2)
- net GND: now also J3.1 (Pin_1), J3.2 (Pin_2)
- no-connect marks 0 -> 6
Other:
- note added: "WARNING: connection is high voltage, but not CAT III rated"
- note removed: "power cord receptacle type: banana socket WARNING: connection is high voltage, but not CAT III rated"
- moved on the sheet: BT1, BT2, J1

Commit message: Passes ERC
Parts:
- renumbered D7 to D3, D8 to D4, J1 to J2, J2 to J4, R13 to R1, R14 to R2
Changed lines of the file:
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@@
 		(dnp no)
 		(fields_autoplaced yes)
-		(property "Reference" "D8"
+		(property "Reference" "D4"
 			(at 180.34 100.3299 90)
 			(effects
@@
 			(project "HighVoltageBoard"
 				(path "/c83b09c9-14ae-4b68-b7fa-4c89bba29dc5/1d0db973-f635-4db8-8646-beeec420ec2b"
-					(reference "D8")
+					(reference "D4")
 					(unit 1)
 				)
@@
 		(on_board yes)
 		(dnp no)
-		(property "Reference" "R13"
+		(property "Reference" "R1"
 			(at 198.12 85.0899 0)
 			(effects
@@
 			(project ""
 				(path "/c83b09c9-14ae-4b68-b7fa-4c89bba29dc5/1d0db973-f635-4db8-8646-beeec420ec2b"
-					(reference "R13")
+					(reference "R1")
 					(unit 1)
 				)
@@
 		(on_board yes)
 		(dnp no)
-		(property "Reference" "J1"
+		(property "Reference" "J2"
 			(at 135.89 73.0249 90)
 			(effects
@@
 			(project ""
 				(path "/c83b09c9-14ae-4b68-b7fa-4c89bba29dc5/1d0db973-f635-4db8-8646-beeec420ec2b"
-					(reference "J1")
+					(reference "J2")
 					(unit 1)
 				)
@@
 		(dnp no)
 		(fields_autoplaced yes)
-		(property "Reference" "J2"
+		(property "Reference" "J4"
 			(at 135.89 103.5049 90)
 			(effects
@@
 			(project "HighVoltageBoard"
 				(path "/c83b09c9-14ae-4b68-b7fa-4c89bba29dc5/1d0db973-f635-4db8-8646-beeec420ec2b"
-					(reference "J2")
+					(reference "J4")
 					(unit 1)
 				)
@@
 		(dnp no)
 		(fields_autoplaced yes)
-		(property "Reference" "D7"
+		(property "Reference" "D3"
 			(at 180.34 85.0899 90)
 			(effects
@@
 			(project "HighVoltageBoard"
 				(path "/c83b09c9-14ae-4b68-b7fa-4c89bba29dc5/1d0db973-f635-4db8-8646-beeec420ec2b"
-					(reference "D7")
+					(reference "D3")
 					(unit 1)
 				)
@@
 		(on_board yes)
 		(dnp no)
-		(property "Reference" "#PWR01"
+		(property "Reference" "#PWR010"
 			(at 219.71 93.98 0)
 			(effects
@@
 			(project ""
 				(path "/c83b09c9-14ae-4b68-b7fa-4c89bba29dc5/1d0db973-f635-4db8-8646-beeec420ec2b"
-					(reference "#PWR01")
+					(reference "#PWR010")
 					(unit 1)
 				)
@@
 		(on_board yes)
 		(dnp no)
-		(property "Reference" "R14"
+		(property "Reference" "R2"
 			(at 198.12 100.3299 0)
 			(effects
@@
 			(project "HighVoltageBoard"
 				(path "/c83b09c9-14ae-4b68-b7fa-4c89bba29dc5/1d0db973-f635-4db8-8646-beeec420ec2b"
-					(reference "R14")
-					(unit 1)
-				)
+					(reference "R2")
+					(unit 1)
+				)

Commit message: Save progress
Parts:
- D1, D2: Cost (none) -> $0.093
- D3, D4: Cost (none) -> $0.370
- R1, R2: Cost (none) -> $0.109
Changed lines of the file:
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@@
+			)
+		)
+		(property "Cost" "$0.370"
+			(at 177.8 101.6 90)
+			(effects
+				(font
+					(size 1.27 1.27)
+				)
+				(hide yes)
 			)
 		)
@@
 			)
 		)
+		(property "Cost" "$0.093"
+			(at 168.91 109.22 0)
+			(effects
+				(font
+					(size 1.27 1.27)
+				)
+				(hide yes)
+			)
+		)
 		(pin "1"
 		)
@@
 			)
 		)
+		(property "Cost" "$0.093"
+			(at 168.91 78.74 0)
+			(effects
+				(font
+					(size 1.27 1.27)
+				)
+				(hide yes)
+			)
+		)
 		(pin "1"
 		)
@@
 		)
 		(property "Purchase Link" "https://www.digikey.com/en/products/detail/vishay-dale/RCV12061M00JNEA/4303607"
+			(at 195.58 86.36 0)
+			(effects
+				(font
+					(size 1.27 1.27)
+				)
+				(hide yes)
+			)
+		)
+		(property "Cost" "$0.109"
 			(at 195.58 86.36 0)
 			(effects
@@
 			)
 		)
+		(property "Cost" "$0.370"
+			(at 177.8 86.36 90)
+			(effects
+				(font
+					(size 1.27 1.27)
+				)
+				(hide yes)
+			)
+		)
 		(pin "2"
 		)
@@
 			(at 195.58 101.6 0)
 			(effects
+				(font
+					(size 1.27 1.27)
+				)
+				(hide yes)
+			)
+		)
+		(property "Cost" "$0.109"
+			(at 195.58 101.6 0)
+			(effects

Commit message: Assigned footprints
Parts:
- D1, D2: footprint (none) -> TwoTerminal:DO-214AC
- D3, D4: footprint (none) -> TwoTerminal:DO-214AA
- J2, J3, J4: footprint (none) -> Connector_Custom:Multicomp_24.243
- R1, R2: footprint (none) -> TwoTerminal:RESC1206_RCV
Changed lines of the file:
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@@
 			)
 		)
-		(property "Footprint" ""
+		(property "Footprint" "TwoTerminal:DO-214AA"
 			(at 177.8 101.6 0)
 			(effects
@@
 			)
 		)
-		(property "Footprint" ""
+		(property "Footprint" "TwoTerminal:DO-214AC"
 			(at 168.91 109.22 0)
 			(effects
@@
 			)
 		)
-		(property "Footprint" ""
+		(property "Footprint" "TwoTerminal:DO-214AC"
 			(at 168.91 78.74 0)
 			(effects
@@
 			)
 		)
-		(property "Footprint" ""
+		(property "Footprint" "TwoTerminal:RESC1206_RCV"
 			(at 196.596 86.614 90)
 			(effects
@@
 			)
 		)
-		(property "Footprint" ""
+		(property "Footprint" "Connector_Custom:Multicomp_24.243"
 			(at 132.08 73.66 0)
 			(effects
@@
 			)
 		)
-		(property "Footprint" ""
+		(property "Footprint" "Connector_Custom:Multicomp_24.243"
 			(at 132.08 104.14 0)
 			(effects
@@
 			)
 		)
-		(property "Footprint" ""
+		(property "Footprint" "TwoTerminal:DO-214AA"
 			(at 177.8 86.36 0)
 			(effects
@@
 			)
 		)
-		(property "Footprint" ""
+		(property "Footprint" "Connector_Custom:Multicomp_24.243"
 			(at 132.08 88.9 0)
 			(effects
@@
 			)
 		)
-		(property "Footprint" ""
+		(property "Footprint" "TwoTerminal:RESC1206_RCV"
 			(at 196.596 101.854 90)
 			(effects

Commit message: Save progress
Parts:
- renumbered J2 to J3, J3 to J4, J4 to J5
Changed lines of the file:
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@@
 		(on_board yes)
 		(dnp no)
-		(property "Reference" "J2"
+		(property "Reference" "J3"
 			(at 135.89 73.0249 90)
 			(effects
@@
 			(project ""
 				(path "/c83b09c9-14ae-4b68-b7fa-4c89bba29dc5/1d0db973-f635-4db8-8646-beeec420ec2b"
-					(reference "J2")
+					(reference "J3")
 					(unit 1)
 				)
@@
 		(dnp no)
 		(fields_autoplaced yes)
-		(property "Reference" "J4"
+		(property "Reference" "J5"
 			(at 135.89 103.5049 90)
 			(effects
@@
 			(project "HighVoltageBoard"
 				(path "/c83b09c9-14ae-4b68-b7fa-4c89bba29dc5/1d0db973-f635-4db8-8646-beeec420ec2b"
-					(reference "J4")
+					(reference "J5")
 					(unit 1)
 				)
@@
 		(on_board yes)
 		(dnp no)
-		(property "Reference" "#PWR010"
+		(property "Reference" "#PWR011"
 			(at 219.71 93.98 0)
 			(effects
@@
 			(project ""
 				(path "/c83b09c9-14ae-4b68-b7fa-4c89bba29dc5/1d0db973-f635-4db8-8646-beeec420ec2b"
-					(reference "#PWR010")
+					(reference "#PWR011")
 					(unit 1)
 				)
@@
 		(dnp no)
 		(fields_autoplaced yes)
-		(property "Reference" "J3"
+		(property "Reference" "J4"
 			(at 135.89 88.2649 90)
 			(effects
@@
 			(project "HighVoltageBoard"
 				(path "/c83b09c9-14ae-4b68-b7fa-4c89bba29dc5/1d0db973-f635-4db8-8646-beeec420ec2b"
-					(reference "J3")
-					(unit 1)
-				)
+					(reference "J4")
+					(unit 1)
+				)

Commit message: Finished layout of power board
Parts:
- J3: value Banana Socket, Red -> Banana Socket, Green; Purchase Link https://www.newark.com/multicomp/24-243-1/pcb-socket-4mm-re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 -> https://www.newark.com/multicomp/24-243-4/banana-jack-4mm-2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
- J5: value Banana Socket, Yellow -> Banana Socket, Blue; Purchase Link https://www.newark.com/multicomp/24-243-3/test-socket-pcb-4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 -> https://www.newark.com/multicomp/24-243-5/test-socket-32a-p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
Changed lines of the file:
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@@
 			)
 		)
-		(property "Value" "Banana Socket, Red"
+		(property "Value" "Banana Socket, Green"
 			(at 135.89 75.5649 90)
 			(effects
@@
 			)
 		)
-		(property "Purchase Link" "https://www.newark.com/multicomp/24-243-1/pcb-socket-4mm-red/dp/80P3616"
+		(property "Purchase Link" "https://www.newark.com/multicomp/24-243-4/banana-jack-4mm-24a-th-green/dp/80P3615"
 			(at 132.08 73.66 0)
 			(effects
@@
 			)
 		)
-		(property "Value" "Banana Socket, Yellow"
+		(property "Value" "Banana Socket, Blue"
 			(at 135.89 106.0449 90)
 			(effects
@@
 			)
 		)
-		(property "Purchase Link" "https://www.newark.com/multicomp/24-243-3/test-socket-pcb-4mm-yellow/dp/80P3617"
+		(property "Purchase Link" "https://www.newark.com/multicomp/24-243-5/test-socket-32a-panel-blue/dp/80P3614"
 			(at 132.08 104.14 0)
 			(effects
