File: Models/HighVoltageBoard/HighVoltageBoard.kicad_pcb (KiCad board)
At the start: 2 copper layers, 0 parts

Commit message: Save progress
Other:
- board text added: "Layer 4: signals and power Layer 3: GND (temp.) Layer 2: signals and power (temp.) Layer 1: GND violates IPC-2221 clearance of 0.25 mm only permit 0.2 mm distance to GND never allow between two high voltage conductors, which could be 900V instead of 450V minimize length of regions with 0.2 mm distance to GND conductor high voltage vias should respect 0.8 mm clearance to GND conductor DESIGN REVIS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"
Changed lines of the file:
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@@
 	)
 	(net 0 "")
+	(gr_text "Layer 4: signals and power\nLayer 3: GND (temp.)\nLayer 2: signals and power (temp.)\nLayer 1: GND\n\nviolates IPC-2221 clearance of 0.25 mm\nonly permit 0.2 mm distance to GND\nnever allow between two high voltage conductors,\nwhich could be 900V instead of 450V\n\nminimize length of regions with\n0.2 mm distance to GND conductor\n\nhigh voltage vias should respect 0.8 mm\nclearance to GND conductor\n\nDESIGN REVISION: 4-layer PCB\nno longer needed or helpful\nfor the routing problem"
+		(at 134.9 166.9 0)
+		(layer "Cmts.User")
+		(effects
+			(font
+				(size 0.8 0.8)
+				(thickness 0.12)
+			)
+			(justify left top)
+		)
+	)
 	(embedded_fonts no)
 )
