File: Models/PracticeBoard/PracticeBoard.kicad_sch (KiCad schematic)
At the start: 0 parts

Commit message: Save progress
Other:
- note added: "Contents: 1x 32-VQFN 5x5 1x TSSOP-16 1x SOIC-16-Wide 2x 2220 Capacitor (exclude from steel template) VQFN purchase link: https://www.digikey.com/en/products/detail/texas-instruments/MSPM0C1105SRHBR/27802389 SOIC-16-Wide: ISO6761 because so cheap"
Changed lines of the file:
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@@
 	(generator_version "9.0")
 	(paper "A4")
+	(text "Contents:\n1x 32-VQFN 5x5\n1x TSSOP-16\n1x SOIC-16-Wide\n2x 2220 Capacitor (exclude from steel template)\n\nVQFN purchase link: https://www.digikey.com/en/products/detail/texas-instruments/MSPM0C1105SRHBR/27802389\nSOIC-16-Wide: ISO6761 because so cheap"
+		(exclude_from_sim no)
+		(at 102.108 52.07 0)
+		(effects
+			(font
+				(size 1.27 1.27)
+			)
+			(justify left top)
+		)
+	)
 	(sheet_instances
 		(path "/"

Commit message: Save progress
Other:
- note added: "Contents: 1x 32-VQFN 5x5 1x TSSOP-16 1x SOIC-16-Wide 1x 2220 Capacitor (exclude from steel template) 1x Vishay resistor (exclude from steel template) VQFN purchase link: https://www.digikey.com/en/products/detail/texas-instruments/MSPM0C1105SRHBR/27802389 SOIC-16-Wide: ISO6761 because so cheap Changed my mind about practice board for now Just omit the SOIC-16-Wide from steel template for main boa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"
- note removed: "Contents: 1x 32-VQFN 5x5 1x TSSOP-16 1x SOIC-16-Wide 2x 2220 Capacitor (exclude from steel template) VQFN purchase link: https://www.digikey.com/en/products/detail/texas-instruments/MSPM0C1105SRHBR/27802389 SOIC-16-Wide: ISO6761 because so cheap"
Changed lines of the file:
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@@
 	(generator_version "9.0")
 	(paper "A4")
-	(text "Contents:\n1x 32-VQFN 5x5\n1x TSSOP-16\n1x SOIC-16-Wide\n2x 2220 Capacitor (exclude from steel template)\n\nVQFN purchase link: https://www.digikey.com/en/products/detail/texas-instruments/MSPM0C1105SRHBR/27802389\nSOIC-16-Wide: ISO6761 because so cheap"
+	(text "Contents:\n1x 32-VQFN 5x5\n1x TSSOP-16\n1x SOIC-16-Wide\n1x 2220 Capacitor (exclude from steel template)\n1x Vishay resistor (exclude from steel template)\n\nVQFN purchase link: https://www.digikey.com/en/products/detail/texas-instruments/MSPM0C1105SRHBR/27802389\nSOIC-16-Wide: ISO6761 because so cheap\n\nChanged my mind about practice board for now\nJust omit the SOIC-16-Wide from steel template for main board\nSolder paste application is now less error-prone\nNo need to spend time designing practice board"
 		(exclude_from_sim no)
 		(at 102.108 52.07 0)
