File: Models/TIA1/TIA1.kicad_pcb (KiCad board)
At the start: 2 copper layers, 0 parts

Commit message: Push uncommitted changes
Parts:
- added C1: 100 nF, 0603, TwoTerminal:CAPC0603, F.Cu at (149.0, 90.2)
- added C2: 100 nF, 0603, TwoTerminal:CAPC0603, F.Cu at (149.0, 92.8)
- added J1: Conn_01x03_Pin, Connector_Custom:PinConnector_1x3, F.Cu at (144.7, 77.2)
- added J2: Conn_01x08_Socket, Connector_Custom:PinConnector_1x8, F.Cu at (135.5, 83.6)
- added J3: Conn_01x08_Socket, Connector_Custom:PinConnector_1x8, F.Cu at (140.1, 83.6)
- added R1: 100M, 5%, 0603, TwoTerminal:RESC0603, F.Cu at (144.6, 90.2)
- added R2: 10, 1%, TwoTerminal:RESC0603, F.Cu at (144.6, 92.9)
- added U1: OPA828, IC:SOIC-8, F.Cu at (146.9, 85.6)

Commit message: Save progress
Parts:
- removed C1, C2: 100 nF, 0603, TwoTerminal:CAPC0603
- removed J1: Conn_01x03_Pin, Connector_Custom:PinConnector_1x3
- removed J2, J3: Conn_01x08_Socket, Connector_Custom:PinConnector_1x8
- removed R1: 100M, 5%, 0603, TwoTerminal:RESC0603
- removed R2: 10, 1%, TwoTerminal:RESC0603
- removed U1: OPA828, IC:SOIC-8
