File: Models/TIA1/TIA1.kicad_pcb (KiCad board)
At the start: 2 copper layers, 21.8 x 16.5 mm, 8 parts, among them J1 Conn_01x03_Pin, J2 Conn_01x06_Socket, J3 Conn_01x08_Socket, U1 OPA828

Commit message: I am overcomplicating the TIA1 board
Parts:
- removed R2: 10, 1%, TwoTerminal:RESC0603
- added R3: 10, 1%, TwoTerminal:RESC0603, F.Cu at (152.9, 91.1)
- J2: value Conn_01x06_Socket -> Conn_01x08_Socket; footprint Connector_Custom:PinSocket_1x6 -> Connector_Custom:PinSocket_1x8
- moved J3 15.2 mm to (158.7, 94.8)
- moved J2 13.0 mm to (158.7, 79.6)
- moved R1 2.59 mm to (154.6, 86.0)
- moved C1 2.58 mm to (165.8, 86.0)
- moved U1 2.58 mm to (160.6, 87.7)
- moved C2 2.58 mm to (158.2, 91.7)
Connections:
- J2 pad 1: /-15V -> /Current
- J2 pad 2: GND -> /Current
- J2 pad 3: /ISO_GND -> /Current
- J2 pad 4: /PostVoltage -> /Current
- J2 pad 5: GND -> /BiasVoltage
- J2 pad 6: /15V -> /BiasVoltage
- J3 pad 1: /Current -> /-15V
- J3 pad 2: /Current -> GND
- J3 pad 3: /Current -> /15V
- J3 pad 4: /Current -> GND
- J3 pad 5: /BiasVoltage -> /PostVoltage
- J3 pad 6: /BiasVoltage -> /ISO_GND
- J3 pad 8: /BiasVoltage -> /ISO_GND
Routing:
- net /PostVoltage: track 0.00 -> 31.0 mm
- net /BiasVoltage: track 0.00 -> 24.3 mm
- net /ISO_GND: track 0.00 -> 24.2 mm, vias 0 -> 2
- net /Current: track 0.00 -> 20.4 mm
- net /15V: track 0.00 -> 16.2 mm
- net /-15V: track 0.00 -> 11.1 mm
- net GND: track 0.00 -> 6.22 mm, vias 0 -> 5
- net Net-(J1-Pin_3): track 0.00 -> 3.96 mm
Other:
- board size 21.8 x 16.5 mm -> 21.8 x 19 mm

Commit message: Save progress
Parts:
- removed R3: 10, 1%, TwoTerminal:RESC0603
- added R2: 10, 1%, TwoTerminal:RESC0603, F.Cu at (152.7, 91.2)
Changed lines of the file:
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@@
 		)
+	)
+	(footprint "TwoTerminal:RESC0603"
+		(layer "F.Cu")
+		(at 152.73 91.17 90)
+		(property "Reference" "R2"
+			(at 0.0475 -1.385 90)
+			(unlocked yes)
+			(layer "F.SilkS")
+			(hide yes)
+			(effects
+				(font
+					(size 0.8 0.8)
+					(thickness 0.12)
+				)
+			)
+		)
+		(property "Value" "10, 1%"
+			(at 0.0475 -0.185 90)
+			(unlocked yes)
+			(layer "F.Fab")
+			(effects
+				(font
+					(size 0.8 0.8)
+					(thickness 0.12)
+				)
+			)
+		)
+		(property "Datasheet" "~"
+			(at 0 0 90)
+			(unlocked yes)
+			(layer "F.Fab")
+			(hide yes)
+			(effects
+				(font
+					(size 0.8 0.8)
+					(thickness 0.12)
+				)
+			)
+		)
+		(property "Description" "Resistor, US symbol"
+			(at 0 0 90)
+			(unlocked yes)
+			(layer "F.Fab")
+			(hide yes)
+			(effects
+				(font
+					(size 0.8 0.8)
+					(thickness 0.12)
+				)
+			)
+		)
+		(property "Purchase Link" "https://www.digikey.com/en/products/detail/vishay-dale/CRCW060310R0FKEA/1174440"
+			(at 0 0 90)
+			(unlocked yes)
+			(layer "F.Fab")
+			(hide yes)
+			(effects
+				(font
+					(size 0.8 0.8)
+					(thickness 0.12)
+				)
+			)
+		)
+		(property "Cost" "$0.030"
+			(at 0 0 90)
+			(unlocked yes)
+			(layer "F.Fab")
+			(hide yes)
+			(effects
+				(font
+					(size 0.8 0.8)
+					(thickness 0.12)
+				)
+			)
+		)
+		(property ki_fp_filters "R_*")
+		(sheetname "/")
+		(sheetfile "TIA1.kicad_sch")
+		(attr smd)
+		(fp_line
+			(start 0.225 -0.585)
+			(end -0.225 -0.585)
+			(stroke
+				(width 0.12)
+				(type default)
+			)
+			(layer "F.SilkS")
+		)
+		(fp_line
+			(start -0.225 0.585)
+			(end 0.225 0.585)
+			(stroke
+				(width 0.12)
+				(type default)
+			)
+			(layer "F.SilkS")
+		)
+		(fp_rect
+			(start -1.675 -0.815)
+			(end 1.675 0.815)
+			(stroke
+				(width 0.05)
+				(type default)
+			)
+			(fill no)
+			(layer "F.CrtYd")
+		)
+		(fp_rect
+			(start -0.825 -0.475)
+			(end 0.825 0.475)
+			(stroke
+				(width 0.1)
+				(type default)
+			)
+			(fill no)
+			(layer "F.Fab")
+		)
+		(fp_text user "${REFERENCE}"
+			(at 0.0475 1.015 90)
+			(unlocked yes)
+			(layer "F.Fab")
+			(effects
+				(font
+					(size 0.8 0.8)
+					(thickness 0.12)
+				)
+			)
+		)
+		(pad "1" smd roundrect
+			(at -0.855 0 90)
+			(size 1.14 1.13)
+			(layers "F.Cu" "F.Mask" "F.Paste")
+			(roundrect_rratio 0.25)
+			(net 4 "Net-(J1-Pin_3)")
+			(pintype "passive")
+			(thermal_bridge_angle 45)
+		)
+		(pad "2" smd roundrect
+			(at 0.855 0 90)
+			(size 1.14 1.13)
+			(layers "F.Cu" "F.Mask" "F.Paste")
+			(roundrect_rratio 0.25)
+			(net 1 "GND")
+			(pintype "passive")
+			(thermal_bridge_angle 45)
+		)
+		(embedded_fonts no)
 	)
 	(footprint "TwoTerminal:CAPC0603"
@@
 			(roundrect_rratio 0.25)
 			(net 8 "/PostVoltage")
-			(pintype "passive")
-			(thermal_bridge_angle 45)
-		)
-		(embedded_fonts no)
-	)
-	(footprint "TwoTerminal:RESC0603"
-		(layer "F.Cu")
-		(at 152.86 91.11 90)
-		(property "Reference" "R3"
-			(at 0.0475 -1.385 90)
-			(unlocked yes)
-			(layer "F.SilkS")
-			(hide yes)
-			(effects
-				(font
-					(size 0.8 0.8)
-					(thickness 0.12)
-				)
-			)
-		)
-		(property "Value" "10, 1%"
-			(at 0.0475 -0.185 90)
-			(unlocked yes)
-			(layer "F.Fab")
-			(effects
-				(font
-					(size 0.8 0.8)
-					(thickness 0.12)
-				)
-			)
-		)
-		(property "Datasheet" "~"
-			(at 0 0 90)
-			(unlocked yes)
-			(layer "F.Fab")
-			(hide yes)
-			(effects
-				(font
-					(size 0.8 0.8)
-					(thickness 0.12)
-				)
-			)
-		)
-		(property "Description" "Resistor, US symbol"
-			(at 0 0 90)
-			(unlocked yes)
-			(layer "F.Fab")
-			(hide yes)
-			(effects
-				(font
-					(size 0.8 0.8)
-					(thickness 0.12)
-				)
-			)
-		)
-		(property "Purchase Link" "https://www.digikey.com/en/products/detail/vishay-dale/CRCW060310R0FKEA/1174440"
-			(at 0 0 90)
-			(unlocked yes)
-			(layer "F.Fab")
-			(hide yes)
-			(effects
-				(font
-					(size 0.8 0.8)
-					(thickness 0.12)
-				)
-			)
-		)
-		(property "Cost" "$0.030"
-			(at 0 0 90)
-			(unlocked yes)
-			(layer "F.Fab")
-			(hide yes)
-			(effects
-				(font
-					(size 0.8 0.8)
-					(thickness 0.12)
-				)
-			)
-		)
-		(property ki_fp_filters "R_*")
-		(sheetname "/")
-		(sheetfile "TIA1.kicad_sch")
-		(attr smd)
-		(fp_line
-			(start 0.225 -0.585)
-			(end -0.225 -0.585)
-			(stroke
-				(width 0.12)
-				(type default)
-			)
-			(layer "F.SilkS")
-		)
-		(fp_line
-			(start -0.225 0.585)
-			(end 0.225 0.585)
-			(stroke
-				(width 0.12)
-				(type default)
-			)
-			(layer "F.SilkS")
-		)
-		(fp_rect
-			(start -1.675 -0.815)
-			(end 1.675 0.815)
-			(stroke
-				(width 0.05)
-				(type default)
-			)
-			(fill no)
-			(layer "F.CrtYd")
-		)
-		(fp_rect
-			(start -0.825 -0.475)
-			(end 0.825 0.475)
-			(stroke
-				(width 0.1)
-				(type default)
-			)
-			(fill no)
-			(layer "F.Fab")
-		)
-		(fp_text user "${REFERENCE}"
-			(at 0.0475 1.015 90)
-			(unlocked yes)
-			(layer "F.Fab")
-			(effects
-				(font
-					(size 0.8 0.8)
-					(thickness 0.12)
-				)
-			)
-		)
-		(pad "1" smd roundrect
-			(at -0.855 0 90)
-			(size 1.14 1.13)
-			(layers "F.Cu" "F.Mask" "F.Paste")
-			(roundrect_rratio 0.25)
-			(net 4 "Net-(J1-Pin_3)")
-			(pintype "passive")
-			(thermal_bridge_angle 45)
-		)
-		(pad "2" smd roundrect
-			(at 0.855 0 90)
-			(size 1.14 1.13)
-			(layers "F.Cu" "F.Mask" "F.Paste")
-			(roundrect_rratio 0.25)
-			(net 1 "GND")
 			(pintype "passive")
 			(thermal_bridge_angle 45)
@@
 	)
 	(segment
-		(start 153.895 90.255)
-		(end 153.9 90.26)
-		(width 0.2)
-		(layer "F.Cu")
-		(net 1)
-	)
-	(segment
 		(start 160.84 89.45)
 		(end 160.84 92.64)
@@
 	)
 	(segment
-		(start 152.86 90.255)
-		(end 153.895 90.255)
+		(start 152.73 90.315)
+		(end 153.775 90.315)
+		(width 0.2)
+		(layer "F.Cu")
+		(net 1)
+	)
+	(segment
+		(start 153.775 90.315)
+		(end 153.78 90.32)
 		(width 0.2)
 		(layer "F.Cu")
@@
 	)
 	(via
-		(at 153.9 90.26)
+		(at 153.78 90.32)
 		(size 0.6)
 		(drill 0.3)
@@
 	)
 	(segment
-		(start 152.86 91.965)
-		(end 152.005 91.965)
+		(start 149.81 89.77)
+		(end 152.065 92.025)
 		(width 0.2)
 		(layer "F.Cu")
@@
 	)
 	(segment
-		(start 152.005 91.965)
-		(end 149.81 89.77)
-		(width 0.2)
-		(layer "F.Cu")
+		(start 152.065 92.025)
+		(end 152.73 92.025)
+		(width 0.2)
+		(layer "F.Cu")
