File: Models/TIA1/TIA1.kicad_sch (KiCad schematic)
At the start: 8 parts, among them J1 Conn_01x03_Pin, J2 Conn_01x08_Socket, J3 Conn_01x08_Socket, U1 OPA828

Commit message: Save progress
Parts:
- J2, J3: Cost $0.53 -> $0.530
- R1: Cost (none) -> $0.280
- U1: Cost (none) -> $7.45; Purchase Link (none) -> https://www.digikey.com/en/products/detail/texas-instrument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
Changed lines of the file:
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@@
 			)
 		)
-		(property "Cost" "$0.53"
+		(property "Cost" "$0.530"
 			(at 218.44 38.1 90)
 			(effects
@@
 			)
 		)
-		(property "Purchase Link" ""
+		(property "Purchase Link" "https://www.digikey.com/en/products/detail/texas-instruments/OPA828IDR/10820196"
+			(at 137.16 73.66 0)
+			(effects
+				(font
+					(size 1.27 1.27)
+				)
+				(hide yes)
+			)
+		)
+		(property "Cost" "$7.45"
 			(at 137.16 73.66 0)
 			(effects
@@
 			)
 		)
+		(property "Cost" "$0.280"
+			(at 135.89 99.06 90)
+			(effects
+				(font
+					(size 1.27 1.27)
+				)
+				(hide yes)
+			)
+		)
 		(pin "1"
 		)
@@
 			)
 		)
-		(property "Cost" "$0.53"
+		(property "Cost" "$0.530"
 			(at 218.44 71.12 90)
 			(effects

Commit message: Should be finished with components BOM
Parts:
- C1, C2: Cost (none) -> $0.079; Purchase Link (none) -> https://www.digikey.com/en/products/detail/murata-electroni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
- R2: value 10 -> 10, 1%; Cost (none) -> $0.030; Purchase Link (none) -> https://www.digikey.com/en/products/detail/vishay-dale/CRCW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
Other:
- note added: "OPA828: already have one in stock, but order two spares to not worry about supply during Phase II"
Changed lines of the file:
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@@
 	(generator_version "9.0")
 	(paper "A4")
+	(text "OPA828: already have one in stock, but order two\nspares to not worry about supply during Phase II"
+		(exclude_from_sim no)
+		(at 142.494 60.198 0)
+		(effects
+			(font
+				(size 1.27 1.27)
+			)
+			(justify left top)
+		)
+	)
 	(junction
 		(at 228.6 45.72)
@@
 			)
 		)
-		(property "Value" "10"
+		(property "Value" "10, 1%"
 			(at 152.4 36.83 90)
 			(effects
@@
 			)
 		)
-		(property "Purchase Link" ""
+		(property "Purchase Link" "https://www.digikey.com/en/products/detail/vishay-dale/CRCW060310R0FKEA/1174440"
 			(at 152.4 40.64 0)
+			(effects
+				(font
+					(size 1.27 1.27)
+				)
+				(hide yes)
+			)
+		)
+		(property "Cost" "$0.030"
+			(at 152.4 40.64 90)
 			(effects
 				(font
@@
 			)
 		)
-		(property "Purchase Link" ""
+		(property "Purchase Link" "https://www.digikey.com/en/products/detail/murata-electronics/GRM188R72A104KA35D/702549"
+			(at 121.92 120.65 0)
+			(effects
+				(font
+					(size 1.27 1.27)
+				)
+				(hide yes)
+			)
+		)
+		(property "Cost" "$0.079"
 			(at 121.92 120.65 0)
 			(effects
@@
 			)
 		)
-		(property "Purchase Link" ""
+		(property "Purchase Link" "https://www.digikey.com/en/products/detail/murata-electronics/GRM188R72A104KA35D/702549"
 			(at 147.32 120.65 0)
 			(effects
+				(font
+					(size 1.27 1.27)
+				)
+				(hide yes)
+			)
+		)
+		(property "Cost" "$0.079"
+			(at 147.32 120.65 0)
+			(effects

Commit message: Save progress
Parts:
- U1: Cost $7.45 -> $7.450
Other:
- note added: "OPA828: Already have one in stock; order two spares (3 total) and stock will be 4. That way, do not have to worry about supply during Phase II."
- note removed: "OPA828: already have one in stock, but order two spares to not worry about supply during Phase II"
Changed lines of the file:
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@@
 	(generator_version "9.0")
 	(paper "A4")
-	(text "OPA828: already have one in stock, but order two\nspares to not worry about supply during Phase II"
+	(text "OPA828: Already have one in stock; order two spares\n(3 total) and stock will be 4. That way, do not\nhave to worry about supply during Phase II."
 		(exclude_from_sim no)
-		(at 142.494 60.198 0)
+		(at 141.224 57.912 0)
 		(effects
 			(font
@@
 			)
 		)
-		(property "Cost" "$7.45"
+		(property "Cost" "$7.450"
 			(at 137.16 73.66 0)
 			(effects

Commit message: Assigned footprints
Parts:
- C1, C2: footprint (none) -> TwoTerminal:CAPC0603
- J1: footprint (none) -> Connector_Custom:PinConnector_1x3
- J2, J3: footprint (none) -> Connector_Custom:PinConnector_1x8
- R1, R2: footprint (none) -> TwoTerminal:RESC0603
- U1: footprint (none) -> IC:SOIC-8
Changed lines of the file:
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@@
 			)
 		)
-		(property "Footprint" ""
+		(property "Footprint" "Connector_Custom:PinConnector_1x8"
 			(at 218.44 38.1 0)
 			(effects
@@
 			)
 		)
-		(property "Footprint" ""
+		(property "Footprint" "IC:SOIC-8"
 			(at 137.16 73.66 0)
 			(effects
@@
 			)
 		)
-		(property "Footprint" ""
+		(property "Footprint" "TwoTerminal:RESC0603"
 			(at 136.144 98.044 90)
 			(effects
@@
 			)
 		)
-		(property "Footprint" ""
+		(property "Footprint" "TwoTerminal:RESC0603"
 			(at 152.654 39.624 90)
 			(effects
@@
 			)
 		)
-		(property "Footprint" ""
+		(property "Footprint" "Connector_Custom:PinConnector_1x3"
 			(at 143.51 33.02 0)
 			(effects
@@
 			)
 		)
-		(property "Footprint" ""
+		(property "Footprint" "Connector_Custom:PinConnector_1x8"
 			(at 218.44 71.12 0)
 			(effects
@@
 			)
 		)
-		(property "Footprint" ""
+		(property "Footprint" "TwoTerminal:CAPC0603"
 			(at 122.8852 124.46 0)
 			(effects
@@
 			)
 		)
-		(property "Footprint" ""
+		(property "Footprint" "TwoTerminal:CAPC0603"
 			(at 148.2852 124.46 0)
 			(effects

Commit message: Save progress
Other:
- moved on the sheet: J1, R2
Changed lines of the file:
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@@
 	(wire
 		(pts
-			(xy 146.05 38.1) (xy 146.05 40.64)
+			(xy 157.48 43.18) (xy 157.48 45.72)
 		)
 		(stroke
@@
 	(wire
 		(pts
-			(xy 138.43 40.64) (xy 140.97 40.64)
+			(xy 149.86 45.72) (xy 152.4 45.72)
 		)
 		(stroke
@@
 	(wire
 		(pts
-			(xy 146.05 40.64) (xy 148.59 40.64)
+			(xy 157.48 45.72) (xy 160.02 45.72)
 		)
 		(stroke
@@
 	(wire
 		(pts
-			(xy 143.51 45.72) (xy 148.59 45.72)
+			(xy 154.94 50.8) (xy 160.02 50.8)
 		)
 		(stroke
@@
 	(wire
 		(pts
-			(xy 143.51 38.1) (xy 143.51 45.72)
-		)
-		(stroke
-			(width 0)
-			(type default)
-		)
-	)
-	(wire
-		(pts
-			(xy 140.97 38.1) (xy 140.97 40.64)
+			(xy 154.94 43.18) (xy 154.94 50.8)
+		)
+		(stroke
+			(width 0)
+			(type default)
+		)
+	)
+	(wire
+		(pts
+			(xy 152.4 43.18) (xy 152.4 45.72)
 		)
 		(stroke
@@
 	(wire
 		(pts
-			(xy 156.21 40.64) (xy 158.75 40.64)
+			(xy 167.64 45.72) (xy 170.18 45.72)
 		)
 		(stroke
@@
 	)
 	(label "ISO_GND"
-		(at 148.59 45.72 0)
+		(at 160.02 50.8 0)
 		(effects
 			(font
@@
 	(symbol
 		(lib_id "Device:R_US")
-		(at 152.4 40.64 90)
+		(at 163.83 45.72 90)
 		(unit 1)
 		(exclude_from_sim no)
@@
 		(fields_autoplaced yes)
 		(property "Reference" "R2"
-			(at 152.4 34.29 90)
+			(at 163.83 39.37 90)
 			(effects
 				(font
@@
 		)
 		(property "Value" "10, 1%"
-			(at 152.4 36.83 90)
+			(at 163.83 41.91 90)
 			(effects
 				(font
@@
 		)
 		(property "Footprint" "TwoTerminal:RESC0603"
-			(at 152.654 39.624 90)
+			(at 164.084 44.704 90)
 			(effects
 				(font
@@
 		)
 		(property "Datasheet" "~"
-			(at 152.4 40.64 0)
+			(at 163.83 45.72 0)
 			(effects
 				(font
@@
 		)
 		(property "Description" "Resistor, US symbol"
-			(at 152.4 40.64 0)
+			(at 163.83 45.72 0)
 			(effects
 				(font
@@
 		)
 		(property "Purchase Link" "https://www.digikey.com/en/products/detail/vishay-dale/CRCW060310R0FKEA/1174440"
-			(at 152.4 40.64 0)
+			(at 163.83 45.72 0)
 			(effects
 				(font
@@
 		)
 		(property "Cost" "$0.030"
-			(at 152.4 40.64 90)
+			(at 163.83 45.72 90)
 			(effects
 				(font
@@
 	(symbol
 		(lib_id "Connector:Conn_01x03_Pin")
-		(at 143.51 33.02 90)
+		(at 154.94 38.1 90)
 		(mirror x)
 		(unit 1)
@@
 		(dnp no)
 		(property "Reference" "J1"
-			(at 143.51 27.94 90)
+			(at 154.94 33.02 90)
 			(effects
 				(font
@@
 		)
 		(property "Value" "Conn_01x03_Pin"
-			(at 143.51 30.48 90)
+			(at 154.94 35.56 90)
 			(effects
 				(font
@@
 		)
 		(property "Footprint" "Connector_Custom:PinConnector_1x3"
-			(at 143.51 33.02 0)
+			(at 154.94 38.1 0)
 			(effects
 				(font
@@
 		)
 		(property "Datasheet" "~"
-			(at 143.51 33.02 0)
+			(at 154.94 38.1 0)
 			(effects
 				(font
@@
 		)
 		(property "Description" "Generic connector, single row, 01x03, script generated"
-			(at 143.51 33.02 0)
+			(at 154.94 38.1 0)
 			(effects
 				(font
@@
 		)
 		(property "Purchase Link" "https://www.digikey.com/en/products/detail/sullins-connector-solutions/PRPC024SAAN-RC/2775230"
-			(at 143.51 33.02 0)
+			(at 154.94 38.1 0)
 			(effects
 				(font
@@
 		)
 		(property "Cost" "$0.563"
-			(at 143.51 33.02 90)
+			(at 154.94 38.1 90)
 			(effects
 				(font
@@
 	(symbol
 		(lib_id "power:GND")
-		(at 138.43 40.64 270)
+		(at 149.86 45.72 270)
 		(unit 1)
 		(exclude_from_sim no)
@@
 		(fields_autoplaced yes)
 		(property "Reference" "#PWR02"
-			(at 132.08 40.64 0)
+			(at 143.51 45.72 0)
 			(effects
 				(font
@@
 		)
 		(property "Value" "GND"
-			(at 134.62 40.6399 90)
+			(at 146.05 45.7199 90)
 			(effects
 				(font
@@
 		)
 		(property "Footprint" ""
-			(at 138.43 40.64 0)
+			(at 149.86 45.72 0)
 			(effects
 				(font
@@
 		)
 		(property "Datasheet" ""
-			(at 138.43 40.64 0)
+			(at 149.86 45.72 0)
 			(effects
 				(font
@@
 		)
 		(property "Description" "Power symbol creates a global label with name \"GND\" , ground"
-			(at 138.43 40.64 0)
+			(at 149.86 45.72 0)
 			(effects
 				(font
@@
 	(symbol
 		(lib_id "power:GND")
-		(at 158.75 40.64 90)
+		(at 170.18 45.72 90)
 		(unit 1)
 		(exclude_from_sim no)
@@
 		(fields_autoplaced yes)
 		(property "Reference" "#PWR04"
-			(at 165.1 40.64 0)
+			(at 176.53 45.72 0)
 			(effects
 				(font
@@
 		)
 		(property "Value" "GND"
-			(at 162.56 40.6399 90)
+			(at 173.99 45.7199 90)
 			(effects
 				(font
@@
 		)
 		(property "Footprint" ""
-			(at 158.75 40.64 0)
+			(at 170.18 45.72 0)
 			(effects
 				(font
@@
 		)
 		(property "Datasheet" ""
-			(at 158.75 40.64 0)
+			(at 170.18 45.72 0)
 			(effects
 				(font
@@
 		)
 		(property "Description" "Power symbol creates a global label with name \"GND\" , ground"
-			(at 158.75 40.64 0)
-			(effects
-				(font
+			(at 170.18 45.72 0)
+			(effects
+				(font

Commit message: Save progress
Parts:
- J1: footprint Connector_Custom:PinConnector_1x3 -> Connector_Custom:PinHeader_1x3
- J2, J3: footprint Connector_Custom:PinConnector_1x8 -> Connector_Custom:PinSocket_1x8
Changed lines of the file:
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@@
 			)
 		)
-		(property "Footprint" "Connector_Custom:PinConnector_1x8"
+		(property "Footprint" "Connector_Custom:PinSocket_1x8"
 			(at 218.44 38.1 0)
 			(effects
@@
 			)
 		)
-		(property "Footprint" "Connector_Custom:PinConnector_1x3"
+		(property "Footprint" "Connector_Custom:PinHeader_1x3"
 			(at 154.94 38.1 0)
 			(effects
@@
 			)
 		)
-		(property "Footprint" "Connector_Custom:PinConnector_1x8"
+		(property "Footprint" "Connector_Custom:PinSocket_1x8"
 			(at 218.44 71.12 0)
 			(effects

Commit message: Save progress
Parts:
- removed J3: Conn_01x08_Socket, Connector_Custom:PinSocket_1x8, symbol Connector:Conn_01x08_Socket
- added J2: Conn_01x06_Socket, Connector_Custom:PinSocket_1x6, symbol Connector:Conn_01x06_Socket
- renumbered J2 to J3
Connections:
- net -15V: now also J2.1 (Pin_1)
- net 15V: now also J2.6 (Pin_6)
- net GND: now also J2.2 (Pin_2), J2.5 (Pin_5)
- net ISO_GND: now also J2.3 (Pin_3)
- net PostVoltage: now also J2.4 (Pin_4)
Changed lines of the file:
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@@
+	(wire
+		(pts
+			(xy 215.9 83.82) (xy 215.9 76.2)
+		)
+		(stroke
+			(width 0)
+			(type default)
+		)
+	)
 	(wire
 		(pts
@@
 	(wire
 		(pts
-			(xy 220.98 76.2) (xy 220.98 86.36)
-		)
-		(stroke
-			(width 0)
-			(type default)
-		)
-	)
-	(wire
-		(pts
 			(xy 147.32 124.46) (xy 147.32 127)
 		)
@@
 	(wire
 		(pts
-			(xy 215.9 76.2) (xy 215.9 86.36)
-		)
-		(stroke
-			(width 0)
-			(type default)
-		)
-	)
-	(wire
-		(pts
 			(xy 121.92 114.3) (xy 121.92 116.84)
 		)
@@
 	(wire
 		(pts
+			(xy 218.44 76.2) (xy 218.44 83.82)
+		)
+		(stroke
+			(width 0)
+			(type default)
+		)
+	)
+	(wire
+		(pts
 			(xy 127 76.2) (xy 129.54 76.2)
 		)
@@
 	(wire
 		(pts
+			(xy 210.82 76.2) (xy 210.82 83.82)
+		)
+		(stroke
+			(width 0)
+			(type default)
+		)
+	)
+	(wire
+		(pts
 			(xy 210.82 43.18) (xy 210.82 45.72)
 		)
@@
 	(wire
 		(pts
-			(xy 226.06 76.2) (xy 226.06 86.36)
-		)
-		(stroke
-			(width 0)
-			(type default)
-		)
-	)
-	(wire
-		(pts
 			(xy 124.46 76.2) (xy 127 76.2)
 		)
@@
 	(wire
 		(pts
-			(xy 210.82 76.2) (xy 210.82 86.36)
-		)
-		(stroke
-			(width 0)
-			(type default)
-		)
-	)
-	(wire
-		(pts
 			(xy 226.06 43.18) (xy 226.06 45.72)
 		)
@@
 		(pts
 			(xy 147.32 73.66) (xy 147.32 99.06)
+		)
+		(stroke
+			(width 0)
+			(type default)
+		)
+	)
+	(wire
+		(pts
+			(xy 223.52 76.2) (xy 223.52 83.82)
 		)
 		(stroke
@@
 		)
 	)
-	(label "BiasVoltage"
-		(at 220.98 86.36 270)
+	(label "PostVoltage"
+		(at 218.44 83.82 270)
 		(effects
 			(font
@@
 	)
 	(label "ISO_GND"
-		(at 223.52 76.2 270)
+		(at 215.9 83.82 270)
 		(effects
 			(font
@@
 		)
 	)
-	(label "-15V"
-		(at 215.9 86.36 270)
+	(label "15V"
+		(at 223.52 83.82 270)
 		(effects
 			(font
@@
 		)
 	)
-	(label "PostVoltage"
-		(at 226.06 86.36 270)
-		(effects
-			(font
-				(size 1.27 1.27)
-			)
-			(justify right bottom)
-		)
-	)
-	(label "15V"
-		(at 210.82 86.36 270)
+	(label "-15V"
+		(at 210.82 83.82 270)
 		(effects
 			(font
@@
 			)
 			(justify left bottom)
-		)
-	)
-	(label "ISO_GND"
-		(at 228.6 76.2 270)
-		(effects
-			(font
-				(size 1.27 1.27)
-			)
-			(justify right bottom)
 		)
 	)
@@
 		(dnp no)
 		(fields_autoplaced yes)
-		(property "Reference" "J2"
+		(property "Reference" "J3"
 			(at 219.71 33.02 90)
 			(effects
@@
 			(project ""
 				(path "/f19129fc-f916-4692-924c-ee308c6b3e1d"
-					(reference "J2")
+					(reference "J3")
 					(unit 1)
 				)
@@
 	)
 	(symbol
-		(lib_id "Connector:Conn_01x08_Socket")
-		(at 218.44 71.12 90)
-		(unit 1)
-		(exclude_from_sim no)
-		(in_bom yes)
-		(on_board yes)
-		(dnp no)
-		(fields_autoplaced yes)
-		(property "Reference" "J3"
-			(at 219.71 66.04 90)
-			(effects
-				(font
-					(size 1.27 1.27)
-				)
-			)
-		)
-		(property "Value" "Conn_01x08_Socket"
-			(at 219.71 68.58 90)
-			(effects
-				(font
-					(size 1.27 1.27)
-				)
-			)
-		)
-		(property "Footprint" "Connector_Custom:PinSocket_1x8"
-			(at 218.44 71.12 0)
-			(effects
-				(font
-					(size 1.27 1.27)
-				)
-				(hide yes)
-			)
-		)
-		(property "Datasheet" "~"
-			(at 218.44 71.12 0)
-			(effects
-				(font
-					(size 1.27 1.27)
-				)
-				(hide yes)
-			)
-		)
-		(property "Description" "Generic connector, single row, 01x08, script generated"
-			(at 218.44 71.12 0)
-			(effects
-				(font
-					(size 1.27 1.27)
-				)
-				(hide yes)
-			)
-		)
-		(property "Purchase Link" "https://www.digikey.com/en/products/detail/sullins-connector-solutions/PPPC081LFBN-RC/810180"
-			(at 218.44 71.12 0)
-			(effects
-				(font
-					(size 1.27 1.27)
-				)
-				(hide yes)
-			)
-		)
-		(property "Cost" "$0.530"
-			(at 218.44 71.12 90)
-			(effects
-				(font
-					(size 1.27 1.27)
-				)
-				(hide yes)
-			)
-		)
-		(pin "2"
-		)
-		(pin "1"
-		)
-		(pin "4"
-		)
-		(pin "3"
-		)
-		(pin "5"
-		)
-		(pin "8"
-		)
-		(pin "7"
-		)
-		(pin "6"
-		)
-		(instances
-			(project "TIA1"
-				(path "/f19129fc-f916-4692-924c-ee308c6b3e1d"
-					(reference "J3")
-					(unit 1)
-				)
-			)
-		)
-	)
-	(symbol
 		(lib_id "power:GND")
 		(at 149.86 45.72 270)
@@
 	(symbol
 		(lib_id "power:GND")
-		(at 218.44 76.2 0)
+		(at 220.98 76.2 0)
 		(unit 1)
 		(exclude_from_sim no)
@@
 		(fields_autoplaced yes)
 		(property "Reference" "#PWR06"
-			(at 218.44 82.55 0)
+			(at 220.98 82.55 0)
 			(effects
 				(font
@@
 		)
 		(property "Value" "GND"
-			(at 218.44 81.28 0)
+			(at 220.98 81.28 0)
 			(effects
 				(font
@@
 		)
 		(property "Footprint" ""
-			(at 218.44 76.2 0)
+			(at 220.98 76.2 0)
 			(effects
 				(font
@@
 		)
 		(property "Datasheet" ""
-			(at 218.44 76.2 0)
+			(at 220.98 76.2 0)
 			(effects
 				(font
@@
 		)
 		(property "Description" "Power symbol creates a global label with name \"GND\" , ground"
-			(at 218.44 76.2 0)
+			(at 220.98 76.2 0)
 			(effects
 				(font
@@
 		)
 		(instances
-			(project ""
+			(project "TIA1"
 				(path "/f19129fc-f916-4692-924c-ee308c6b3e1d"
 					(reference "#PWR05")
 					(unit 1)
 				)
+			)
+		)
+	)
+	(symbol
+		(lib_id "Connector:Conn_01x06_Socket")
+		(at 215.9 71.12 90)
+		(unit 1)
+		(exclude_from_sim no)
+		(in_bom yes)
+		(on_board yes)
+		(dnp no)
+		(fields_autoplaced yes)
+		(property "Reference" "J2"
+			(at 217.17 66.04 90)
+			(effects
+				(font
+					(size 1.27 1.27)
+				)
+			)
+		)
+		(property "Value" "Conn_01x06_Socket"
+			(at 217.17 68.58 90)
+			(effects
+				(font
+					(size 1.27 1.27)
+				)
+			)
+		)
+		(property "Footprint" "Connector_Custom:PinSocket_1x6"
+			(at 215.9 71.12 0)
+			(effects
+				(font
+					(size 1.27 1.27)
+				)
+				(hide yes)
+			)
+		)
+		(property "Datasheet" "~"
+			(at 215.9 71.12 0)
+			(effects
+				(font
+					(size 1.27 1.27)
+				)
+				(hide yes)
+			)
+		)
+		(property "Description" "Generic connector, single row, 01x06, script generated"
+			(at 215.9 71.12 0)
+			(effects
+				(font
+					(size 1.27 1.27)
+				)
+				(hide yes)
+			)
+		)
+		(property "Purchase Link" "https://www.digikey.com/en/products/detail/sullins-connector-solutions/PPPC061LFBN-RC/810178"
+			(at 215.9 71.12 0)
+			(effects
+				(font
+					(size 1.27 1.27)
+				)
+				(hide yes)
+			)
+		)
+		(property "Cost" "$0.470"
+			(at 215.9 71.12 90)
+			(effects
+				(font
+					(size 1.27 1.27)
+				)
+				(hide yes)
+			)
+		)
+		(pin "1"
+		)
+		(pin "2"
+		)
+		(pin "3"
+		)
+		(pin "4"
+		)
+		(pin "5"
+		)
+		(pin "6"
+		)
+		(instances
+			(project ""
+				(path "/f19129fc-f916-4692-924c-ee308c6b3e1d"
+					(reference "J2")
+					(unit 1)
+				)
