File: Models/TIA2_Pre/TIA2_Pre.kicad_pcb (KiCad board)
At the start: 2 copper layers, 0 parts

Commit message: First time that all PCBs are fully wired
Parts:
- added C1: 1 uF, 0603, TwoTerminal:CAPC0603, F.Cu at (126.2, 99.8)
- added C2: 1 uF, 0603, TwoTerminal:CAPC0603, F.Cu at (131.2, 95.6)
- added J1: Conn_01x03_Pin, Connector_Custom:PinHeader_1x3, F.Cu at (118.1, 96.5)
- added J2: Conn_01x04_Socket, Connector_Custom:PinSocket_1x4, F.Cu at (121.9, 104.1)
- added J3: Conn_01x08_Socket, Connector_Custom:PinSocket_1x8, F.Cu at (127.0, 88.9)
- added J4: Conn_01x05_Socket, Connector_Custom:PinSocket_1x5, F.Cu at (135.9, 99.1)
- added R1: 10, 1%, TwoTerminal:RESC0603, F.Cu at (121.1, 100.2)
- added R2: 1G, 5%, 0603, TwoTerminal:RESC0603, F.Cu at (123.0, 94.6)
- added U1: AD8615, IC:AD8615, F.Cu at (127.6, 96.7)
Routing:
- net /ISO_GND: track 0.00 -> 32.8 mm, vias 0 -> 2
- net /Current: track 0.00 -> 19.5 mm
- net /PreVoltage: track 0.00 -> 18.1 mm
- net /-1.5V: track 0.00 -> 17.0 mm
- net /BiasVoltage: track 0.00 -> 12.7 mm
- net /2.5V: track 0.00 -> 11.6 mm
- net /AD8615_Output: track 0.00 -> 8.70 mm, vias 0 -> 2
- net GND: track 0.00 -> 6.28 mm, vias 0 -> 5
- net Net-(J1-Pin_3): track 0.00 -> 3.83 mm
- added copper zone on B.Cu, net GND
Other:
- board outline added: 21.8 x 19 mm
- board text added: "1 GΩ"
