File: Models/Stencil/MainBoard1.kicad_pcb (KiCad board)
At the start: 4 copper layers, 77 x 62.5 mm, 82 parts, among them J1 Conn_Coaxial, J10 Conn_01x03_Pin, J11 Conn_01x03_Pin, J12 Conn_01x03_Pin, J13 Conn_01x02_Pin, J14 Conn_01x13_Pin, J15 Conn_01x13_Pin, J16 Conn_01x24_Socket, J19 Conn_01x24_Socket, J2 Conn_Coaxial, J3 Conn_Coaxial, J4 Conn_Coaxial, J5 Conn_Coaxial, J6 Conn_Coaxial, J7 Conn_01x03_Pin, J8 Conn_01x03_Pin, J9 Conn_01x03_Pin, U1 ADS8699, U2 AD7745, U3 DAC81404, U4 DAC81401, U5 ISO7761DW, U6 ISO1641DW

Commit message: Save progress
Parts:
- removed C1, C12, C14, C16, C20, C22, C24, C3, C5, C7, C9: 10 uF, 0805, TwoTerminal:CAPC0805
- removed C10, C18: 220 nF, 0603, TwoTerminal:CAPC0603
- removed C11, C13, C15, C17, C19, C21, C23, C25, C26, C27, C28, C29, C8: 100 nF, 0603, TwoTerminal:CAPC0603
- removed C2, C4, C6: 1 uF, 0603, TwoTerminal:CAPC0603
- removed R1, R2: 10, 1%, TwoTerminal:RESC0603
- removed R10, R11, R12, R6, R9: 10k, 1%, TwoTerminal:RESC0603
- removed U5: ISO7761DW, IC:SOIC-16-Wide
- removed U6: ISO1641DW, IC:SOIC-16-Wide
Other:
- board text added: "${REFERENCE}"
