File: Models/Stencil/MainBoard2.kicad_pcb (KiCad board)
At the start: 4 copper layers, 77 x 62.5 mm, 82 parts, among them J1 Conn_Coaxial, J10 Conn_01x03_Pin, J11 Conn_01x03_Pin, J12 Conn_01x03_Pin, J13 Conn_01x02_Pin, J14 Conn_01x13_Pin, J15 Conn_01x13_Pin, J16 Conn_01x24_Socket, J19 Conn_01x24_Socket, J2 Conn_Coaxial, J3 Conn_Coaxial, J4 Conn_Coaxial, J5 Conn_Coaxial, J6 Conn_Coaxial, J7 Conn_01x03_Pin, J8 Conn_01x03_Pin, J9 Conn_01x03_Pin, U1 ADS8699, U2 AD7745, U3 DAC81404, U4 DAC81401, U5 ISO7761DW, U6 ISO1641DW

Commit message: Save progress
Parts:
- removed C17: 100 nF, 0603, TwoTerminal:CAPC0603
- removed R1, R2: 10, 1%, TwoTerminal:RESC0603
- removed U1: ADS8699, IC:TSSOP-16
- removed U2: AD7745, IC:TSSOP-16
- removed U3: DAC81404, IC:VQFN-32
- removed U4: DAC81401, IC:TSSOP-20
