File: Models/STM_PCB/PreAmp/PreAmp.kicad_pcb (KiCad board)
At the start: 2 copper layers, 19.9 x 16.5 mm, 7 parts, among them J1 Conn_Coaxial, J2 Conn_01x03_Socket, J3 Conn_01x03_Socket, U1 AD8615

Commit message: Save progress
Parts:
- moved J1 1.00 mm to (154.7, 99.1)
Routing:
- net /Current: track 9.00 -> 8.00 mm
Other:
- board size 19.9 x 16.5 mm -> 18.9 x 16.5 mm
- board text added: "Rearrange this board to be thinner in the Y dimension"
Changed lines of the file:
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@@
 	(footprint "Connector_Custom:Samtec_MMCX_SMT"
 		(layer "F.Cu")
-		(at 153.67 99.06)
+		(at 154.67 99.06)
 		(property "Reference" "J1"
 			(at 0.34 -2.55 0)
@@
 	)
 	(gr_arc
-		(start 151.25 97.64)
-		(mid 151.542893 96.932893)
-		(end 152.25 96.64)
+		(start 152.25 97.64)
+		(mid 152.542893 96.932893)
+		(end 153.25 96.64)
 		(stroke
 			(width 0.05)
@@
 	)
 	(gr_line
-		(start 151.25 100.48)
-		(end 151.25 97.64)
+		(start 152.25 100.48)
+		(end 152.25 97.64)
 		(stroke
 			(width 0.05)
@@
 	)
 	(gr_line
+		(start 153.25 96.64)
+		(end 156.42 96.64)
+		(stroke
+			(width 0.05)
+			(type default)
+		)
+		(layer "Edge.Cuts")
+	)
+	(gr_line
 		(start 170.15 107.29)
 		(end 158.42 107.29)
-		(stroke
-			(width 0.05)
-			(type default)
-		)
-		(layer "Edge.Cuts")
-	)
-	(gr_line
-		(start 152.25 96.64)
-		(end 156.42 96.64)
 		(stroke
 			(width 0.05)
@@
 		(start 157.42 102.48)
 		(end 157.42 106.29)
+		(stroke
+			(width 0.05)
+			(type default)
+		)
+		(layer "Edge.Cuts")
+	)
+	(gr_line
+		(start 153.25 101.48)
+		(end 156.42 101.48)
 		(stroke
 			(width 0.05)
@@
 	)
 	(gr_arc
-		(start 152.25 101.48)
-		(mid 151.542893 101.187107)
-		(end 151.25 100.48)
-		(stroke
-			(width 0.05)
-			(type default)
-		)
-		(layer "Edge.Cuts")
-	)
-	(gr_line
-		(start 156.42 101.48)
-		(end 152.25 101.48)
+		(start 153.25 101.48)
+		(mid 152.542893 101.187107)
+		(end 152.25 100.48)
 		(stroke
 			(width 0.05)
@@
 		)
 	)
+	(gr_text "Rearrange this board to be thinner in\nthe Y dimension"
+		(at 174.06 99.67 0)
+		(layer "Cmts.User")
+		(effects
+			(font
+				(size 0.8 0.8)
+				(thickness 0.12)
+			)
+			(justify left bottom)
+		)
+	)
 	(segment
 		(start 162.69 103.63)
@@
 	)
 	(segment
-		(start 152.4 97.79)
-		(end 152.4 98.77)
-		(width 0.2)
-		(layer "F.Cu")
-		(net 2)
-	)
-	(segment
-		(start 154.94 100.33)
-		(end 154.94 99.35)
+		(start 153.4 97.79)
+		(end 153.4 98.77)
+		(width 0.2)
+		(layer "F.Cu")
+		(net 2)
+	)
+	(segment
+		(start 155.94 100.33)
+		(end 155.94 99.35)
 		(width 0.2)
 		(layer "F.Cu")
@@
 	)
 	(segment
-		(start 152.4 100.33)
-		(end 153.38 100.33)
+		(start 153.4 100.33)
+		(end 154.38 100.33)
 		(width 0.2)
 		(layer "F.Cu")
@@
 	)
 	(segment
-		(start 154.94 97.79)
-		(end 153.96 97.79)
+		(start 155.94 97.79)
+		(end 154.96 97.79)
 		(width 0.2)
 		(layer "F.Cu")
@@
 	)
 	(via
-		(at 153.96 97.79)
+		(at 154.96 97.79)
 		(size 0.6)
 		(drill 0.3)
@@
 	)
 	(via
-		(at 152.4 98.77)
+		(at 153.4 98.77)
 		(size 0.6)
 		(drill 0.3)
@@
 	)
 	(via
-		(at 154.94 99.35)
+		(at 155.94 99.35)
 		(size 0.6)
 		(drill 0.3)
@@
 	)
 	(via
-		(at 153.38 100.33)
+		(at 154.38 100.33)
 		(size 0.6)
 		(drill 0.3)
@@
 	)
 	(segment
-		(start 156.34 98.11)
-		(end 158.7675 98.11)
-		(width 0.2)
-		(layer "F.Cu")
-		(net 4)
-	)
-	(segment
-		(start 155.701 98.749)
-		(end 156.34 98.11)
+		(start 156.571 98.749)
+		(end 157.21 98.11)
 		(width 0.2)
 		(layer "F.Cu")
@@
 	)
 	(segment
-		(start 153.67 99.06)
-		(end 153.981 98.749)
+		(start 154.981 98.749)
+		(end 156.571 98.749)
+		(width 0.2)
+		(layer "F.Cu")
+		(net 4)
+	)
+	(segment
+		(start 157.21 98.11)
+		(end 158.7675 98.11)
+		(width 0.2)
+		(layer "F.Cu")
+		(net 4)
+	)
+	(segment
+		(start 154.67 99.06)
+		(end 154.981 98.749)
 		(width 0.2)
 		(layer "F.Cu")
@@
 		(start 158.7675 98.0075)
 		(end 159.985 96.79)
-		(width 0.2)
-		(layer "F.Cu")
-		(net 4)
-	)
-	(segment
-		(start 153.981 98.749)
-		(end 155.701 98.749)
 		(width 0.2)
 		(layer "F.Cu")
@@
 		(polygon
 			(pts
-				(xy 170.65 91.33) (xy 157.92 91.33) (xy 157.92 96.14) (xy 156.92 97.14) (xy 151.75 97.14) (xy 151.75 100.98)
+				(xy 170.65 91.33) (xy 157.92 91.33) (xy 157.92 96.14) (xy 156.92 97.14) (xy 152.75 97.14) (xy 152.75 100.98)
 				(xy 156.92 100.98) (xy 157.92 101.98) (xy 157.92 106.79) (xy 170.65 106.79)
 			)

Commit message: Fixed the PCB
Parts:
- added H1: MountingHole_Pad, Connector_Custom:KJ_D21SH, B.Cu at (159.8, 101.5)
- added H2: MountingHole_Pad, Connector_Custom:KJ_D21SH, B.Cu at (166.3, 94.8)
- added H3: MountingHole_Pad, Connector_Custom:KJ_D21SH, B.Cu at (172.9, 101.5)
- C1, C2: value 1 uF, 0603 -> 1 uF, 0603, 25V, X7R
- moved J2 5.37 mm to (170.5, 100.7)
- moved J3 4.42 mm to (170.5, 95.6)
- moved C1 1.00 mm to (159.4, 101.5)
- moved C2 1.00 mm to (164.0, 97.0)
- moved U1 1.00 mm to (160.0, 98.1)
- moved J1 0.91 mm to (154.7, 98.2)
- moved R1 0.45 mm to (160.3, 94.5), turned to 0 degrees
Routing:
- net /2.5V: track 8.89 -> 14.5 mm
- net /-1.5V: track 10.8 -> 15.2 mm
- net /PreVoltage: track 4.29 -> 6.97 mm
- net /AD8615_Output: track 9.18 -> 9.93 mm, vias 2 -> 0
- net /Current: track 8.00 -> 7.41 mm
Other:
- board size 18.9 x 16.5 mm -> 23 x 11.4 mm
- board text removed: "1 GΩ"
- board text removed: "Rearrange this board to be thinner in the Y dimension"
