File: Models/STM_PCB/PreAmp/PreAmp.kicad_sch (KiCad schematic)
At the start: 7 parts, among them J1 Conn_Coaxial, J2 Conn_01x03_Socket, J3 Conn_01x03_Socket, U1 AD8615

Commit message: Save progress
Other:
- note added: "May need to add bottom pads for connecting to shield through 3 magnets holding the board"
Changed lines of the file:
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@@
+		)
+	)
+	(text "May need to add bottom pads for connecting\nto shield through 3 magnets holding the board"
+		(exclude_from_sim no)
+		(at 170.434 36.322 0)
+		(effects
+			(font
+				(size 1.27 1.27)
+			)
+			(justify left top)
 		)
 	)

Commit message: Fixed the PCB
Parts:
- added H1, H2, H3: MountingHole_Pad, Connector_Custom:KJ_D21SH, symbol Mechanical:MountingHole_Pad
- C1, C2: value 1 uF, 0603 -> 1 uF, 0603, 25V, X7R; Cost $0.078 -> $0.13; Purchase Link https://www.digikey.com/en/products/detail/murata-electronics/GRT188R61H105KE13D/5416752 -> https://www.digikey.com/en/products/detail/murata-electronics/GRT188R71E105KE13D/10694256; now in the parts list
Connections:
- net GND: now also H1.1, H2.1, H3.1
Other:
- note added: "Magnets on back are attached with conductive epoxy through 125°C, 2-hour bake. All other components on the board are rated for 125°C."
- note removed: "May need to add bottom pads for connecting to shield through 3 magnets holding the board"
- moved on the sheet: C2

Commit message: Save progress
Other:
- note added: "Inserted into MMCX connector: 0.3 mm diameter, W wire"
- note added: "Tips must be W instead of Pt to maximize eigenfrequency and thus minimize severity of vibrational coupling. A simple analysis of fine X, coarse Y, coarse Z has minimum 25 kHz. 3.53 mm x 0.3 mm Pt wire is 10 kHz. 2.53 mm: protrudes 1 mm from MMCX ring 3.53 mm: protrudes 2 mm from MMCX ring W, 2.53 mm: 31 kHz W, 3.53 mm: 16 kHz Pt, 2.53 mm: 19 kHz Pt, 3.53 mm: 10 kHz"
- note removed: "Inserted into MMCX connector: 0.3 mm diameter, pure Pt wire"
Changed lines of the file:
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@@
 	(generator_version "9.0")
 	(paper "A4")
-	(text "Inserted into MMCX connector:\n0.3 mm diameter, pure Pt wire"
+	(text "Tips must be W instead of Pt to maximize\neigenfrequency and thus minimize severity\nof vibrational coupling. A simple analysis\nof fine X, coarse Y, coarse Z has minimum 25 kHz.\n3.53 mm x 0.3 mm Pt wire is 10 kHz.\n\n2.53 mm: protrudes 1 mm from MMCX ring\n3.53 mm: protrudes 2 mm from MMCX ring\n\nW, 2.53 mm: 31 kHz\nW, 3.53 mm: 16 kHz\nPt, 2.53 mm: 19 kHz\nPt, 3.53 mm: 10 kHz"
+		(exclude_from_sim no)
+		(at 27.178 108.712 0)
+		(effects
+			(font
+				(size 1.27 1.27)
+			)
+			(justify left top)
+		)
+	)
+	(text "Inserted into MMCX connector:\n0.3 mm diameter, W wire"
 		(exclude_from_sim no)
 		(at 50.8 63.5 0)
