File: Models/HighVoltageBoard2/Simulation/OPA828.kicad_sch (KiCad schematic)
At the start: 13 parts, among them U2 ${SIM.PARAMS}

Commit message: Pick this back up when I return to it
Parts:
- removed C18, C19, C20, C21, C22, C23: 114p, symbol Device:C
- removed C30: 3.978e-8, symbol Device:C
- removed C31: 1.591e-3, symbol Device:C
- removed R19, R20: 1, symbol Device:R_US
- removed U2: ${SIM.PARAMS}, symbol Simulation_SPICE:OPAMP
- removed V7, V8: ${SIM.PARAMS}, symbol Simulation_SPICE:VDC
- added C24, C25: 100n, symbol Device:C
- added C26: 10p, symbol Device:C
- added C27, C28: 0.2p, symbol Device:C
- added C29: 1.2p, symbol Device:C
- added R16, R18: 30k, symbol Device:R_US
- added R17: 11.0k, symbol Device:R_US
- added U1: ${SIM.PARAMS}, symbol Simulation_SPICE:OPAMP
- added V5, V6: 15, symbol Simulation_SPICE:VDC
Connections:
- net GND: now also C24.2, C25.1, C26.1, U1.1 (+), V5.2, V6.1
- new net: C26.2, C27.2, C28.2, C29.1, R16.2, R17.2, R18.1, U1.2 (-)
- new net -15V: C25.2, U1.4 (V-), V6.2
- new net 15V: C24.1, U1.3 (V+), V5.1
- new net IN_COARSE: C28.1, R17.1
- new net IN_FINE: C27.1, R16.1
- new net OUT: C29.2, R18.2, U1.5
- no-connect marks 2 -> 0
Other:
- note added: "1.0 pF compensation capacitor on R_f required to avoid instability"
- note removed: "resistors: 1 = 20 kHz 2 = 10 kHz 4 = 5 kHz Q-factor: 100"
- note removed: "the amount of PA79 overshoot doesn't matter; any short voltage step will make the piezo resonate with an amplitude of twice the DAC step size ... come back to this problem tomorrow resonant noise ≥ 2 * DAC resolution... maybe we can at least low-pass filter the fine Z output before summing with the coarse output in the OPA828 stage? make the compensation capacitor swappable, tuning it to match a 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"
- note removed: "wire the slave (with 20% larger current limit) to the electrode with 10% larger effective capacitance"
