File: Models/HighVoltageBoard2/Simulation/Piezo.kicad_sch (KiCad schematic)
At the start: 13 parts, among them U2 ${SIM.PARAMS}

Commit message: Save progress
Other:
- note added: "capacitors: Q = 100 1.591e-3 3.978e-8 Q = 20 3.183e-4 1.989e-7"
- note added: "resistors: 1 = 20 kHz 2 = 10 kHz 4 = 5 kHz"
- note removed: "resistors: 1 = 20 kHz 2 = 10 kHz 4 = 5 kHz Q-factor: 100"
Changed lines of the file:
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@@
 	(generator_version "10.0")
 	(paper "A4")
-	(text "resistors:\n1 = 20 kHz\n2 = 10 kHz\n4 = 5 kHz\n\nQ-factor: 100"
+	(text "capacitors:\n\nQ = 100\n1.591e-3\n3.978e-8\n\nQ = 20\n3.183e-4\n1.989e-7"
 		(exclude_from_sim no)
-		(at 120.65 74.422 0)
+		(at 146.558 64.008 0)
+		(effects
+			(font
+				(size 1.27 1.27)
+			)
+			(justify left top)
+		)
+	)
+	(text "resistors:\n\n1 = 20 kHz\n2 = 10 kHz\n4 = 5 kHz"
+		(exclude_from_sim no)
+		(at 120.65 72.136 0)
 		(effects
 			(font
@@
 		)
 		(property "Sim.Params" "dc=0 ampl=0 f=0 td=0 theta=0 phase=0 ac=1 ph=0"
-			(at 127.762 128.524 0)
-			(show_name no)
-			(do_not_autoplace no)
+			(at 127.508 127.508 0)
+			(show_name no)
+			(do_not_autoplace no)

Commit message: Save progress
Parts:
- C18, C19, C20, C21, C22, C23: value 114p -> {cappiezo}
- R19, R20: value 1 -> 4
Other:
- note added: "default piezo capacitance: 114p"
Changed lines of the file:
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@@
 	(text "wire the slave (with 20% larger current limit)\nto the electrode with 10% larger effective capacitance"
 		(exclude_from_sim no)
-		(at 27.178 22.098 0)
+		(at 27.686 14.986 0)
+		(effects
+			(font
+				(size 1.27 1.27)
+			)
+			(justify left top)
+		)
+	)
+	(text "default piezo capacitance: 114p"
+		(exclude_from_sim no)
+		(at 27.94 23.622 0)
 		(effects
 			(font
@@
 			)
 		)
-		(property "Value" "114p"
+		(property "Value" "{cappiezo}"
 			(at 54.61 109.2199 0)
 			(show_name no)
@@
 			)
 		)
-		(property "Value" "114p"
+		(property "Value" "{cappiezo}"
 			(at 54.61 58.4199 0)
 			(show_name no)
@@
 			)
 		)
-		(property "Value" "114p"
+		(property "Value" "{cappiezo}"
 			(at 54.61 83.8199 0)
 			(show_name no)
@@
 			)
 		)
-		(property "Value" "114p"
+		(property "Value" "{cappiezo}"
 			(at 54.61 71.1199 0)
 			(show_name no)
@@
 			)
 		)
-		(property "Value" "1"
+		(property "Value" "4"
 			(at 146.05 97.79 90)
 			(show_name no)
@@
 			)
 		)
-		(property "Value" "114p"
+		(property "Value" "{cappiezo}"
 			(at 54.61 45.7199 0)
 			(show_name no)
@@
 			)
 		)
-		(property "Value" "114p"
+		(property "Value" "{cappiezo}"
 			(at 54.61 96.5199 0)
 			(show_name no)
@@
 			)
 		)
-		(property "Value" "1"
+		(property "Value" "4"
 			(at 133.35 97.79 90)
 			(show_name no)
