File: Models/HighVoltageBoard2/Simulation/HighVoltageBoard2_Simulation.kicad_sch (KiCad schematic)
At the start: 17 parts, among them IC1 PA79DK

Commit message: Good progress on SPICE analysis
Parts:
- removed R3, R4: 8.75k, symbol Device:R_US
- added C10: 8p, symbol Device:C
- added C8, C9: 1.3p, symbol Device:C
- added R10: 1.5k, symbol Device:R_US
- added R11: 50k, symbol Device:R_US
- added R8: 15, symbol Device:R_US
- added R9: 35.7k, symbol Device:R_US
- added V3: ${SIM.PARAMS}, symbol Simulation_SPICE:VDC
Connections:
- net -175V: now also V2.2
- net 175V: now also V1.1
- net GND: now also C10.2, C9.1, R10.1, R11.2, V3.2
- net at IC1.1 (-IN_A): now also C8.1, C9.2, R10.2, R9.1
- net at IC1.17 (CL_A): now also R8.1
- net OUT: now reaches IC1.18 (OUT_A)
- net OUT: now also C10.1, C8.2, R11.1, R8.2, R9.2
- net IN: now reaches IC1.2 (+IN_A)
- net IN: now also V3.1
Other:
- note added: "current limit master: 15 Ω slave: 12 Ω"
- note added: "master: input resistors: YAGEO MFP-25 1.3 pF parasitic capacitance slave: input resistor: 390k SMT 0.5 pF parasitic capacitance"
- moved on the sheet: C1, C2, R1, R2, V1, V2

Commit message: Progress on designing HighVoltageBoard2
Parts:
- added C11: 10n, symbol Device:C
- added R3: 20k, symbol Device:R_US
- C10: value 8p -> 700p
- C8, C9: value 1.3p -> 0.3p
- R10: value 1.5k -> 390k
- R9: value 35.7k -> 390k
- V1, V2: value 150 -> 170
Connections:
- net GND: now also IC1.2 (+IN_A), R3.2; no longer C9.1, R10.1
- net IN: now also C9.1, R10.1; no longer IC1.2 (+IN_A)
- net -IN: now reaches C8.1, C9.2, IC1.1 (-IN_A), R10.2, R9.1
- net -IN: now also C11.1
- new net: C11.2, R3.1
Other:
- note added: "TNPW0805 (200k) 150 V rating <0.3 pF parasitic capacitance 0.1%, 25 ppm/°C Rf = 2x 200k in series [probably not needed, but let's be conservative regarding R_f C_f cutoff, in case the SPICE simulation is wrong]"
- note added: "current limit safe vs. design requirement master: 15 Ω / 6 Ω slave: 12 Ω / 5 Ω the safe limits are to help in a fault condition where the current shorts it will be easier to test with the safe ones first, and once we have experience, replace with more optimized resistors design the board to make broken amplifiers easily replaced only do this modification on the amplifier for the Z axis, or whiche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"
- note added: "master: input resistors: YAGEO MFP-25 0.5-1.5 pF parasitic capacitance [not required with board design that has replaceable amplifiers] slave: input resistor: same as Rf"
- note added: "what elements to add to stabilize the slave, with -1 gain? resistor: 39k (application note formula) 23k (simulation, C_f = 0.05 pF) 38k (simulation, C_f = 0.3 pF) 20k (decision) capacitor (20k, C_f = 0.05 pF) 1.6 nF (application note formula) 4.5 nF (simulation) capacitor (20k, C_f = 0.3 pF) 1.6 nF (application note formula) 3.0 nF (simulation) 10.0 nF (decision) effect on input-output Bode plot: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"
- note removed: "current limit master: 15 Ω slave: 12 Ω"
- note removed: "master: input resistors: YAGEO MFP-25 1.3 pF parasitic capacitance slave: input resistor: 390k SMT 0.5 pF parasitic capacitance"

Commit message: Save progress
Parts:
- removed C10: 700p, symbol Device:C
- removed C6: 2.2p, symbol Device:C
- removed C7: 33p, symbol Device:C
- removed IC1: PA79DK, PA162DK, symbol PA79DK:PA79DK
- removed R11: 50k, symbol Device:R_US
- removed R7: 3.3k, symbol Device:R_US
- removed R8: 15, symbol Device:R_US
- added R10: 5, symbol Device:R_US
- added R17: 50k, symbol Device:R_US
- added R3: 40k, symbol Device:R_US
- added R_A_probe1, R_B_probe1: 0.1, symbol Device:R_US
- added V3: ${SIM.PARAMS}, symbol Simulation_SPICE:VDC
- C3: value 2.2p -> 0.2p
- C4: value 100n -> 10n
- C5: value 100n -> 0.5p
- C6: renamed from C9; value 0.3p -> 0.5p
- C7: renamed from C11; value 10n -> 100n
- C8: value 0.3p -> 0.5p
- R5: value 3.3k -> 400k
- R6: value 340k -> 6
- R7: renamed from R10; value 390k -> 400k
- R8: renamed from R3; value 20k -> 50k
- R9: value 390k -> 400k
- renumbered V3 to V4
Connections:
- net -175V: no longer C5.1
- net 175V: no longer C4.2, R6.2
- net GND: now also R17.1, V3.2; no longer C4.1, C5.2
- net IN: now also C3.1, R3.1, V3.1; no longer C6.1, R7.1
- net PA79A/-IN: now reaches R5.1
- net PA79A/-IN: now also C3.2, C4.1, C5.1, R3.2
- net OUTA: now reaches R5.2
- net OUTA: now also C5.2, C6.1, R6.2, R7.1, R_A_probe1.1; no longer C3.2
- net -CC_A renamed PA79A/CL
- net PA79A/CL: no longer C3.1
- net -IN renamed PA79B/-IN
- net OUT renamed OUTB
- net OUTB: now also R10.2, R_B_probe1.1
- new net: C4.2, R17.2
- new net PA79B/CL: R10.1
- new net Piezo/OUTA: R_A_probe1.2
- new net Piezo/OUTB: R_B_probe1.2
- no-connect marks 10 -> 0
Other:
- added sheet PA79A (PA79_Single.kicad_sch)
- added sheet PA79B (PA79_Single.kicad_sch)
- added sheet Piezo (Piezo.kicad_sch)
- note added: "Rf: 1206 or 1210 resistor keepout zone on closest inner copper layer to make capacitance closer to expectation"
- note added: "effect of gain on stability [C_f = 0.2 pF, C_c = 2.2 pF] no capacitive load: overshoot vanishes at G > 12.5 - no R_n and C_n needed on master - 50k and 0.01-0.07n on slave - 40k and 0.02-0.10n on slave - 30k and 0.03-0.15n on slave - 20k and 0.04-0.20n on slave with piezo: [C_f = 0.5 pF, C_c = 2.2 pF] no capacitive load: overshoot vanishes at G > 4.0 - 70k and 3-30p - 50k and 7-40p - 20k and 30-1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"
- note added: "impact of C_c, C_f on slew rate into piezo: TODO"
- note added: "quantification of voltage noise: (5 / 10 / 20 kHz, peak-peak) DAC: 54 / 70 / 94 μV op amp input: 212 / 300 / 425 μV modeling all relevant variables (mechanical Q = 100, G_master = 50) R_n = 50k, C_n = 0.255 nF: 4.9 / 9.4 / 16.7 pm R_n = 50k, C_n = 0.127 nF: 3.8 / 6.8 / 13.2 pm R_n = 50k, C_n = 0.076 nF: 3.3 / 5.5 / 10.3 pm R_n = 50k, C_n = 0.051 nF: 3.1 / 4.8 / 8.5 pm all of this optimization eff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"
- note added: "what elements to add to stabilize the slave, with -1 gain? resistor: 40k (application note formula) 20-60k (C_f = 0.01 pF) 20-60k (C_f = 0.05 pF) 30-90k (C_f = 0.1 pF) 45-110k (C_f = 0.2 pF) capacitor (50k, C_f = 0.05 pF) 0.07 nF (simulation) capacitor (50k, C_f = 0.2 pF) 0.05 nF (simulation)"
- note removed: "TNPW0805 (200k) 150 V rating <0.3 pF parasitic capacitance 0.1%, 25 ppm/°C Rf = 2x 200k in series [probably not needed, but let's be conservative regarding R_f C_f cutoff, in case the SPICE simulation is wrong]"
- note removed: "master: input resistors: YAGEO MFP-25 0.5-1.5 pF parasitic capacitance [not required with board design that has replaceable amplifiers] slave: input resistor: same as Rf"
- note removed: "what elements to add to stabilize the slave, with -1 gain? resistor: 39k (application note formula) 23k (simulation, C_f = 0.05 pF) 38k (simulation, C_f = 0.3 pF) 20k (decision) capacitor (20k, C_f = 0.05 pF) 1.6 nF (application note formula) 4.5 nF (simulation) capacitor (20k, C_f = 0.3 pF) 1.6 nF (application note formula) 3.0 nF (simulation) 10.0 nF (decision) effect on input-output Bode plot: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"
- moved on the sheet: C1, C2, C6, C7, C8, R1, R2, R7, R8, R9, V1, V2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

Commit message: Pick this back up when I return to it
Parts:
- removed C4: 10n, symbol Device:C
- removed R17: 50k, symbol Device:R_US
- C4: renamed from C5; value 0.5p -> 0.3p
- C5: renamed from C6; value 0.5p -> 0.3p
- C6: renamed from C7; value 100n -> 0.1n
- C7: renamed from C8; value 0.5p -> 0.3p
- R3: value 40k -> 30.6k
- renumbered R5 to R4, R6 to R5, R7 to R6, R8 to R7, R9 to R8, R10 to R9, V4 to V3, V3 to V4
Connections:
- net IN: no longer C3.1, R3.1
- new net OPA828/OUT: C3.1, R3.1
Other:
- added sheet OPA828 (OPA828.kicad_sch)
- note added: "close to a decision: power supplies: exactly 170 V target amplitude: 165 V G_pre (OPA828) = 13.5 / 5 = -2.7 G_post (PA97) = 170 / 12.5 = -13.6 fine Z channel in OPA828 passes through -1.0 gain"
- note added: "current limit safe vs. design requirement master: 15 Ω / 6 Ω slave: 12 Ω / 5 Ω start with the safe values for an initial test, upgrade to the smaller resistances afterward, design board to easily replace fried amplifiers"
- note removed: "current limit safe vs. design requirement master: 15 Ω / 6 Ω slave: 12 Ω / 5 Ω the safe limits are to help in a fault condition where the current shorts it will be easier to test with the safe ones first, and once we have experience, replace with more optimized resistors design the board to make broken amplifiers easily replaced only do this modification on the amplifier for the Z axis, or whiche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"
- note removed: "impact of C_c, C_f on slew rate into piezo: TODO"
- note removed: "quantification of voltage noise: (5 / 10 / 20 kHz, peak-peak) DAC: 54 / 70 / 94 μV op amp input: 212 / 300 / 425 μV modeling all relevant variables (mechanical Q = 100, G_master = 50) R_n = 50k, C_n = 0.255 nF: 4.9 / 9.4 / 16.7 pm R_n = 50k, C_n = 0.127 nF: 3.8 / 6.8 / 13.2 pm R_n = 50k, C_n = 0.076 nF: 3.3 / 5.5 / 10.3 pm R_n = 50k, C_n = 0.051 nF: 3.1 / 4.8 / 8.5 pm all of this optimization eff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"
- note removed: "what elements to add to stabilize the slave, with -1 gain? resistor: 40k (application note formula) 20-60k (C_f = 0.01 pF) 20-60k (C_f = 0.05 pF) 30-90k (C_f = 0.1 pF) 45-110k (C_f = 0.2 pF) capacitor (50k, C_f = 0.05 pF) 0.07 nF (simulation) capacitor (50k, C_f = 0.2 pF) 0.05 nF (simulation)"
- moved on the sheet: C1, C2, C3, C4, C5, C6, C7, R1, R2, R3, R4, R5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

Commit message: Save progress
Parts:
- added C32: 10u, symbol Device:C
- added R21: 0.227, symbol Device:R_US
- added V10, V11, V12, V9: ${SIM.PARAMS}, symbol Simulation_SPICE:VDC
Connections:
- net GND: now also C32.2, V10.2, V11.2, V12.2, V9.2
- new net NOISE_DAC_COARSE: V11.1
- new net NOISE_DAC_FINE: V12.1
- new net NOISE_FILTER_OUT: C32.1, R21.2
- new net NOISE_PA79A: R21.1, V9.1
- new net NOISE_PA79B: V10.1
Other:
- note added: "105 nV/sqrt(Hz)"
- note added: "500 nV/sqrt(Hz)"
- note added: "70 kHz 1st-order checks correctness of noise gen"
- note added: "current limit safe vs. design requirement master: 15 Ω / 6 Ω slave: 12 Ω / 5 Ω start with the safe values for an initial test, upgrade to the smaller resistances afterward, design board to easily replace fried amplifiers order the following parts: 15, 10, 6 Ω 12, 8.66, 5 Ω"
- note removed: "current limit safe vs. design requirement master: 15 Ω / 6 Ω slave: 12 Ω / 5 Ω start with the safe values for an initial test, upgrade to the smaller resistances afterward, design board to easily replace fried amplifiers"
- moved on the sheet: V3, V4

Commit message: Save progress
Parts:
- added R22, R23, R24: 0.001, symbol Device:R_US
- C6: value 0.1n -> 10n
Connections:
- net -175V: now also R23.2; no longer C2.2, R2.2, V2.2
- net 175V: now also R22.2; no longer C1.1, R1.1, V1.1
- net GND: now also R24.2; no longer V1.2, V2.1
- new net: C1.1, R1.1, R22.1, V1.1
- new net: R24.1, V1.2, V2.1
- new net: C2.2, R2.2, R23.1, V2.2
Other:
- note added: ".control set controlswait meas tran dynamic_tfall TRIG v(/piezo/pos_unfiltered) VAL=60.2 FALL=1 TARG v(/piezo/pos_unfiltered) VAL=-37.7 FALL=1 meas tran dynamic_trise TRIG v(/piezo/pos_unfiltered) VAL=-60.3 RISE=1 TARG v(/piezo/pos_unfiltered) VAL=37.6 RISE=1 meas tran Vmin min v(/piezo/pos_unfiltered) from=1u to=60u meas tran Vmax max v(/piezo/pos_unfiltered) from=1u to=60u .endc"
- note added: "Large C_n here does not degrade circuit performance in any way"

Commit message: Save progress
Other:
- note added: ".control set controlswait meas tran dynamic_tfall5 TRIG v(/piezo/pos_unfiltered) VAL=142.1 FALL=1 TARG v(/piezo/pos_unfiltered) VAL=-86.4 FALL=1 meas tran dynamic_trise5 TRIG v(/piezo/pos_unfiltered) VAL=-139.1 RISE=1 TARG v(/piezo/pos_unfiltered) VAL=89.4 RISE=1 meas tran Vmin min v(/piezo/pos_unfiltered) from=1u to=60u meas tran Vmax max v(/piezo/pos_unfiltered) from=1u to=60u .endc"
- note removed: ".control set controlswait meas tran dynamic_tfall TRIG v(/piezo/pos_unfiltered) VAL=60.2 FALL=1 TARG v(/piezo/pos_unfiltered) VAL=-37.7 FALL=1 meas tran dynamic_trise TRIG v(/piezo/pos_unfiltered) VAL=-60.3 RISE=1 TARG v(/piezo/pos_unfiltered) VAL=37.6 RISE=1 meas tran Vmin min v(/piezo/pos_unfiltered) from=1u to=60u meas tran Vmax max v(/piezo/pos_unfiltered) from=1u to=60u .endc"
Changed lines of the file:
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@@
 		)
 	)
-	(text ".control\nset controlswait\n\nmeas tran dynamic_tfall TRIG v(/piezo/pos_unfiltered) VAL=60.2 FALL=1 TARG v(/piezo/pos_unfiltered) VAL=-37.7 FALL=1\nmeas tran dynamic_trise TRIG v(/piezo/pos_unfiltered) VAL=-60.3 RISE=1 TARG v(/piezo/pos_unfiltered) VAL=37.6 RISE=1\nmeas tran Vmin min v(/piezo/pos_unfiltered) from=1u to=60u\nmeas tran Vmax max v(/piezo/pos_unfiltered) from=1u to=60u\n.endc\n"
+	(text ".control\nset controlswait\n\nmeas tran dynamic_tfall5 TRIG v(/piezo/pos_unfiltered) VAL=142.1 FALL=1 TARG v(/piezo/pos_unfiltered) VAL=-86.4 FALL=1\nmeas tran dynamic_trise5 TRIG v(/piezo/pos_unfiltered) VAL=-139.1 RISE=1 TARG v(/piezo/pos_unfiltered) VAL=89.4 RISE=1\nmeas tran Vmin min v(/piezo/pos_unfiltered) from=1u to=60u\nmeas tran Vmax max v(/piezo/pos_unfiltered) from=1u to=60u\n.endc\n"
 		(exclude_from_sim no)
 		(at 23.368 16.51 0)
