File: Models/HighVoltageBoard2/Simulation/PA79_Single.kicad_sch (KiCad schematic)
At the start: 9 parts, among them IC1 PA79DK

Commit message: Pick this back up when I return to it
Parts:
- renumbered C11 to C10, C12 to C11, C13 to C12, C9 to C8, C10 to C9, R11 to R10, R12 to R11, R13 to R12
Changed lines of the file:
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@@
 		(dnp no)
 		(fields_autoplaced yes)
-		(property "Reference" "C12"
+		(property "Reference" "C11"
 			(at 160.02 106.6799 0)
 			(show_name no)
@@
 			(project "HighVoltageBoard2_Simulation"
 				(path "/9bc71ba4-b324-4c2f-a958-e9450ff9b707/2050f40a-14c6-4f54-9670-197e7dd64f72"
-					(reference "C12")
+					(reference "C11")
 					(unit 1)
 				)
 				(path "/9bc71ba4-b324-4c2f-a958-e9450ff9b707/a06ffbea-e0a1-4134-8518-d5f130694c51"
-					(reference "C17")
+					(reference "C16")
 					(unit 1)
 				)
@@
 		(dnp no)
 		(fields_autoplaced yes)
-		(property "Reference" "#PWR07"
+		(property "Reference" "#PWR06"
 			(at 156.21 72.39 0)
 			(hide yes)
@@
 			(project "HighVoltageBoard2_Simulation"
 				(path "/9bc71ba4-b324-4c2f-a958-e9450ff9b707/2050f40a-14c6-4f54-9670-197e7dd64f72"
-					(reference "#PWR07")
+					(reference "#PWR06")
 					(unit 1)
 				)
 				(path "/9bc71ba4-b324-4c2f-a958-e9450ff9b707/a06ffbea-e0a1-4134-8518-d5f130694c51"
-					(reference "#PWR09")
+					(reference "#PWR08")
 					(unit 1)
 				)
@@
 		(dnp no)
 		(fields_autoplaced yes)
-		(property "Reference" "R12"
+		(property "Reference" "R11"
 			(at 99.06 90.17 90)
 			(show_name no)
@@
 			(project "HighVoltageBoard2_Simulation"
 				(path "/9bc71ba4-b324-4c2f-a958-e9450ff9b707/2050f40a-14c6-4f54-9670-197e7dd64f72"
-					(reference "R12")
+					(reference "R11")
 					(unit 1)
 				)
 				(path "/9bc71ba4-b324-4c2f-a958-e9450ff9b707/a06ffbea-e0a1-4134-8518-d5f130694c51"
-					(reference "R15")
+					(reference "R14")
 					(unit 1)
 				)
@@
 		(dnp no)
 		(fields_autoplaced yes)
-		(property "Reference" "#PWR08"
+		(property "Reference" "#PWR07"
 			(at 156.21 120.65 0)
 			(hide yes)
@@
 			(project "HighVoltageBoard2_Simulation"
 				(path "/9bc71ba4-b324-4c2f-a958-e9450ff9b707/2050f40a-14c6-4f54-9670-197e7dd64f72"
-					(reference "#PWR08")
+					(reference "#PWR07")
 					(unit 1)
 				)
 				(path "/9bc71ba4-b324-4c2f-a958-e9450ff9b707/a06ffbea-e0a1-4134-8518-d5f130694c51"
-					(reference "#PWR010")
+					(reference "#PWR09")
 					(unit 1)
 				)
@@
 		(dnp no)
 		(fields_autoplaced yes)
-		(property "Reference" "R13"
+		(property "Reference" "R12"
 			(at 171.45 83.8199 0)
 			(show_name no)
@@
 			(project "HighVoltageBoard2_Simulation"
 				(path "/9bc71ba4-b324-4c2f-a958-e9450ff9b707/2050f40a-14c6-4f54-9670-197e7dd64f72"
-					(reference "R13")
+					(reference "R12")
 					(unit 1)
 				)
 				(path "/9bc71ba4-b324-4c2f-a958-e9450ff9b707/a06ffbea-e0a1-4134-8518-d5f130694c51"
-					(reference "R16")
+					(reference "R15")
 					(unit 1)
 				)
@@
 		(dnp no)
 		(fields_autoplaced yes)
-		(property "Reference" "C11"
+		(property "Reference" "C10"
 			(at 160.02 83.8199 0)
 			(show_name no)
@@
 			(project "HighVoltageBoard2_Simulation"
 				(path "/9bc71ba4-b324-4c2f-a958-e9450ff9b707/2050f40a-14c6-4f54-9670-197e7dd64f72"
-					(reference "C11")
+					(reference "C10")
 					(unit 1)
 				)
 				(path "/9bc71ba4-b324-4c2f-a958-e9450ff9b707/a06ffbea-e0a1-4134-8518-d5f130694c51"
-					(reference "C16")
+					(reference "C15")
 					(unit 1)
 				)
@@
 		(dnp no)
 		(fields_autoplaced yes)
-		(property "Reference" "C9"
+		(property "Reference" "C8"
 			(at 86.36 76.2 90)
 			(show_name no)
@@
 			(project "HighVoltageBoard2_Simulation"
 				(path "/9bc71ba4-b324-4c2f-a958-e9450ff9b707/2050f40a-14c6-4f54-9670-197e7dd64f72"
-					(reference "C9")
+					(reference "C8")
 					(unit 1)
 				)
 				(path "/9bc71ba4-b324-4c2f-a958-e9450ff9b707/a06ffbea-e0a1-4134-8518-d5f130694c51"
-					(reference "C14")
+					(reference "C13")
 					(unit 1)
 				)
@@
 		(dnp no)
 		(fields_autoplaced yes)
-		(property "Reference" "R11"
+		(property "Reference" "R10"
 			(at 99.06 77.47 90)
 			(show_name no)
@@
 			(project "HighVoltageBoard2_Simulation"
 				(path "/9bc71ba4-b324-4c2f-a958-e9450ff9b707/2050f40a-14c6-4f54-9670-197e7dd64f72"
-					(reference "R11")
+					(reference "R10")
 					(unit 1)
 				)
 				(path "/9bc71ba4-b324-4c2f-a958-e9450ff9b707/a06ffbea-e0a1-4134-8518-d5f130694c51"
-					(reference "R14")
+					(reference "R13")
 					(unit 1)
 				)
@@
 		(dnp no)
 		(fields_autoplaced yes)
-		(property "Reference" "C13"
+		(property "Reference" "C12"
 			(at 172.72 106.6799 0)
 			(show_name no)
@@
 			(project "HighVoltageBoard2_Simulation"
 				(path "/9bc71ba4-b324-4c2f-a958-e9450ff9b707/2050f40a-14c6-4f54-9670-197e7dd64f72"
-					(reference "C13")
+					(reference "C12")
 					(unit 1)
 				)
 				(path "/9bc71ba4-b324-4c2f-a958-e9450ff9b707/a06ffbea-e0a1-4134-8518-d5f130694c51"
-					(reference "C18")
+					(reference "C17")
 					(unit 1)
 				)
@@
 		(dnp no)
 		(fields_autoplaced yes)
-		(property "Reference" "C10"
+		(property "Reference" "C9"
 			(at 86.36 88.9 90)
 			(show_name no)
@@
 			(project "HighVoltageBoard2_Simulation"
 				(path "/9bc71ba4-b324-4c2f-a958-e9450ff9b707/2050f40a-14c6-4f54-9670-197e7dd64f72"
-					(reference "C10")
+					(reference "C9")
 					(unit 1)
 				)
 				(path "/9bc71ba4-b324-4c2f-a958-e9450ff9b707/a06ffbea-e0a1-4134-8518-d5f130694c51"
-					(reference "C15")
-					(unit 1)
-				)
+					(reference "C14")
+					(unit 1)
+				)

Commit message: Save progress
Other:
- note added: "TODO: Revisit C_c and optimize if it limits slew rate Analyze whether reaching a maximum input voltage triumphs over C_c in unlocking maximum current - Test (±1 V, ±2 V, ±3 V, ±4 V, ±5 V) at the DAC w/ respective slew times - Test (5, 7, 10, 15, 20, 30) pF capacitance"
Changed lines of the file:
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@@
 	(generator_version "10.0")
 	(paper "A4")
+	(text "TODO: Revisit C_c and optimize if it limits slew rate\n\nAnalyze whether reaching a maximum input voltage\ntriumphs over C_c in unlocking maximum current\n- Test (±1 V, ±2 V, ±3 V, ±4 V, ±5 V) at the DAC w/ respective slew times\n- Test (5, 7, 10, 15, 20, 30) pF capacitance"
+		(exclude_from_sim no)
+		(at 71.882 36.576 0)
+		(effects
+			(font
+				(size 1.27 1.27)
+			)
+			(justify left top)
+		)
+	)
 	(junction
 		(at 168.91 91.44)

Commit message: Save progress
Parts:
- C8, C9: value 10p -> {capc}
Other:
- note added: ".PARAM capc = 3p"
- note added: ".PARAM cappiezo = 114p"
- note added: ".PARAM sigmag = 3"
- note added: "TODO: Revisit C_c and optimize if it limits slew rate Analyze stability w.r.t: 1. compensation capacitance 2. piezo capacitance (dynamically scale 114 pF) 3. signal magnitude"
- note removed: "TODO: Revisit C_c and optimize if it limits slew rate Analyze whether reaching a maximum input voltage triumphs over C_c in unlocking maximum current - Test (±1 V, ±2 V, ±3 V, ±4 V, ±5 V) at the DAC w/ respective slew times - Test (5, 7, 10, 15, 20, 30) pF capacitance"
Changed lines of the file:
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@@
 	(generator_version "10.0")
 	(paper "A4")
-	(text "TODO: Revisit C_c and optimize if it limits slew rate\n\nAnalyze whether reaching a maximum input voltage\ntriumphs over C_c in unlocking maximum current\n- Test (±1 V, ±2 V, ±3 V, ±4 V, ±5 V) at the DAC w/ respective slew times\n- Test (5, 7, 10, 15, 20, 30) pF capacitance"
+	(text "TODO: Revisit C_c and optimize if it limits slew rate\n\nAnalyze stability w.r.t:\n1. compensation capacitance\n2. piezo capacitance (dynamically scale 114 pF)\n3. signal magnitude"
 		(exclude_from_sim no)
 		(at 71.882 36.576 0)
+		(effects
+			(font
+				(size 1.27 1.27)
+			)
+			(justify left top)
+		)
+	)
+	(text ".PARAM cappiezo = 114p"
+		(exclude_from_sim no)
+		(at 83.312 61.214 0)
+		(effects
+			(font
+				(size 1.27 1.27)
+			)
+			(justify left top)
+		)
+	)
+	(text ".PARAM sigmag = 3"
+		(exclude_from_sim no)
+		(at 83.312 57.404 0)
+		(effects
+			(font
+				(size 1.27 1.27)
+			)
+			(justify left top)
+		)
+	)
+	(text ".PARAM capc = 3p"
+		(exclude_from_sim no)
+		(at 83.312 64.516 0)
 		(effects
 			(font
@@
 			)
 		)
-		(property "Value" "10p"
+		(property "Value" "{capc}"
 			(at 86.36 78.74 90)
 			(show_name no)
@@
 			)
 		)
-		(property "Value" "10p"
+		(property "Value" "{capc}"
 			(at 86.36 91.44 90)
 			(show_name no)

Commit message: Save progress
Other:
- note added: ".PARAM sigmag = 5"
- note added: "order the following parts: 4.7, 6.8, 10, 15, 22 pF Start out with 10 pF. Once we are testing an actual high-capacitance piezo in the small-signal regime, inspect the waveforms on the scope. Remove and replace the SMT bypass caps or solder a new PA79 sub-board with a different value for C_c. Cal-Chip Electronics, CHV, 500V rated, 0805 package, ±0.25pF or 5% tolerance 4 caps/board * $1.034 (sum of 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"
- note added: "ordering PA79: componentstockers.com has in stock Mouser is out of stock until 9/15/2026 $53.80 * 6 = $322.80 + shipping"
- note removed: ".PARAM sigmag = 3"
Changed lines of the file:
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@@
+		)
+	)
+	(text "ordering PA79:\ncomponentstockers.com has in stock\nMouser is out of stock until 9/15/2026\n\n$53.80 * 6 = $322.80 + shipping"
+		(exclude_from_sim no)
+		(at 101.6 127.254 0)
+		(effects
+			(font
+				(size 1.27 1.27)
+			)
+			(justify left top)
+		)
+	)
+	(text "order the following parts:\n4.7, 6.8, 10, 15, 22 pF\n\nStart out with 10 pF. Once we are testing an actual\nhigh-capacitance piezo in the small-signal regime,\ninspect the waveforms on the scope. Remove and replace\nthe SMT bypass caps or solder a new PA79 sub-board with\na different value for C_c.\n\nCal-Chip Electronics, CHV, 500V rated,\n0805 package, ±0.25pF or 5% tolerance\n4 caps/board * $1.034 (sum of costs across 5 variants) * 7 = $28.95"
+		(exclude_from_sim no)
+		(at 144.78 34.036 0)
+		(effects
+			(font
+				(size 1.27 1.27)
+			)
+			(justify left top)
 		)
 	)
@@
 		)
 	)
-	(text ".PARAM sigmag = 3"
+	(text ".PARAM sigmag = 5"
 		(exclude_from_sim no)
 		(at 83.312 57.404 0)
